File: CarMan KiCAD Schematics/GLV_BOBV6/GLV_BOBV6.kicad_pcb (KiCad board)
At the start: 2 copper layers, 87 x 60.3 mm, 26 parts, among them J1 Battery Conn_01x02, J2 Extra 24V Conn_01x02, J3 24V CAN ISO Conn_01x02, J4 Logic Conn_02x02_Odd_Even, J5 TSI Conn_02x02_Odd_Even, J6 Breakers J6, U1 INA226AIDGSR

Commit message: GLV DR Fixes
Parts:
- J1 LSP: renamed from J1 Battery
- J3 CAN ISO: renamed from J3 24V CAN ISO
- moved H3 8.17 mm to (189.9, 22.4)
- moved H4 8.17 mm to (189.9, 69.8)
Connections:
- J6 Breakers pad 1: /BATT+ -> /24V_NOT_BREAKERED
- J6 Breakers pad 2: /BATT+ -> /24V_NOT_BREAKERED
- J6 Breakers pad 3: /BATT+ -> /24V_NOT_BREAKERED
- R1 pad 1: /24V -> /24V_NOT_BREAKERED
- U1 pad 8: /24V -> /24V_NOT_BREAKERED
- U1 pad 9: /24V -> /24V_NOT_BREAKERED
Routing:
- net /BATT+: track 89.5 -> 29.5 mm
- net /24V_NOT_BREAKERED: track 0.00 -> 56.4 mm
- net /24V: track 176.6 -> 167.5 mm
- net /3.3V_NOT_ISO: track 48.4 -> 46.1 mm, vias 0 -> 2
- net /GLV_RTN: track 72.2 -> 74.3 mm
Other:
- board size 87 x 60.3 mm -> 79.5 x 60.3 mm
- board text added: "GLV BOB V6.0 Troy Coleman and Zachary Martin 2/9/21"
- board text removed: "GLV BOB V6 Troy Coleman and Zachary Martin 11/22/20"
- board text removed: "Left Side"
- board text removed: "Right Side"
