File: CarMan KiCAD Schematics/Logic/Logic.sch (KiCad schematic (older format))
At the start: 29 parts, among them J1 MC_CAN, J2 IMU, J3 RTC, J4 GLV_I2C

Commit message: Refactored repo
Parts:
- added J18: PIC program, symbol Connector_Generic:Conn_01x06
- gave numbers to parts that had none: 25
Connections:
- wire segments 243 -> 248
- no-connect marks 34 -> 49
Changed lines of the file:
@@
 $EndComp
 $Comp
-L PYB20-Q24-S5:PYB20-Q24-S5 U?
+L PYB20-Q24-S5:PYB20-Q24-S5 U2
 U 1 1 5F997454
 P 2300 7000
-F 0 "U?" H 2300 7667 50  0000 C CNN
+F 0 "U2" H 2300 7667 50  0000 C CNN
 F 1 "PYB20-Q24-S5" H 2300 7576 50  0000 C CNN
 F 2 "CONV_PYB20-Q24-S5" H 2300 7000 50  0001 L BNN
@@
 $EndComp
 $Comp
-L Lafayette_Electric_Car_Internals:LT1763CS8-3.3PBF U?
+L Lafayette_Electric_Car_Internals:LT1763CS8-3.3PBF U4
 U 1 1 5F997AAE
 P 5000 6900
-F 0 "U?" H 5000 7570 50  0000 C CNN
+F 0 "U4" H 5000 7570 50  0000 C CNN
 F 1 "LT1763CS8-3.3PBF" H 5000 7479 50  0000 C CNN
 F 2 "SOIC127P600X175-8N" H 5000 6900 50  0001 L BNN
@@
 	1150 7300 1450 7300
 $Comp
-L Device:C C?
+L Device:C C1
 U 1 1 5F99E44C
 P 1450 7000
-F 0 "C?" H 1565 7046 50  0000 L CNN
+F 0 "C1" H 1565 7046 50  0000 L CNN
 F 1 "0.1uF" H 1565 6955 50  0000 L CNN
 F 2 "" H 1488 6850 50  0001 C CNN
@@
 	1450 7300 1650 7300
 $Comp
-L Device:C C?
+L Device:C C3
 U 1 1 5F99F0F5
 P 3050 7000
-F 0 "C?" H 3165 7046 50  0000 L CNN
+F 0 "C3" H 3165 7046 50  0000 L CNN
 F 1 "0.1uF" H 3165 6955 50  0000 L CNN
 F 2 "" H 3088 6850 50  0001 C CNN
@@
 	3050 6700 4050 6700
 $Comp
-L Device:C C?
+L Device:C C5
 U 1 1 5F99FFE4
 P 3800 7050
-F 0 "C?" H 3915 7096 50  0000 L CNN
+F 0 "C5" H 3915 7096 50  0000 L CNN
 F 1 "1uF" H 3915 7005 50  0000 L CNN
 F 2 "" H 3838 6900 50  0001 C CNN
@@
 P 10000 4100
 AR Path="/5F9665AE/5F9FC061" Ref="U?"  Part="1"
-AR Path="/5F9FC061" Ref="U?"  Part="1"
-F 0 "U?" H 10025 5315 50  0000 C CNN
+AR Path="/5F9FC061" Ref="U6"  Part="1"
+F 0 "U6" H 10025 5315 50  0000 C CNN
 F 1 "RaspberryPi3" H 10025 5224 50  0000 C CNN
 F 2 "Lafayette_Electric_Car_Footprints:RaspberryPi3" H 10250 5300 50  0001 C CNN
@@
 NoConn ~ 9500 3950
 $Comp
-L Connector_Generic:Conn_01x08 J?
+L Connector_Generic:Conn_01x08 J6
 U 1 1 5FA1FE07
 P 9950 5950
-F 0 "J?" H 10030 5942 50  0000 L CNN
+F 0 "J6" H 10030 5942 50  0000 L CNN
 F 1 "You're Welcome -Ethan" H 10030 5851 50  0000 L CNN
 F 2 "" H 9950 5950 50  0001 C CNN
@@
 	1000 2500 1100 2500
 $Comp
-L Device:R R?
+L Device:R R2
 U 1 1 5FB9034F
 P 1200 2650
-F 0 "R?" V 1100 2650 50  0000 C CNN
+F 0 "R2" V 1100 2650 50  0000 C CNN
 F 1 "10k" V 1200 2650 50  0000 C CNN
 F 2 "" V 1130 2650 50  0001 C CNN
@@
 $EndComp
 $Comp
-L Device:R R?
+L Device:R R1
 U 1 1 5FB90355
 P 1000 2650
-F 0 "R?" V 900 2650 50  0000 C CNN
+F 0 "R1" V 900 2650 50  0000 C CNN
 F 1 "10k" V 1000 2650 50  0000 C CNN
 F 2 "" V 930 2650 50  0001 C CNN
@@
 3.3V_rtn
 $Comp
-L Device:C C?
+L Device:C C2
 U 1 1 5FB9037B
 P 1850 2250
-F 0 "C?" H 1965 2296 50  0000 L CNN
+F 0 "C2" H 1965 2296 50  0000 L CNN
 F 1 "0.1uF" H 1965 2205 50  0000 L CNN
 F 2 "" H 1888 2100 50  0001 C CNN
@@
 	2400 1650 2400 1800
 $Comp
-L Device:R R?
+L Device:R R3
 U 1 1 5FB90383
 P 1850 1950
-F 0 "R?" V 1750 1950 50  0000 C CNN
+F 0 "R3" V 1750 1950 50  0000 C CNN
 F 1 "10k" V 1850 1950 50  0000 C CNN
 F 2 "" V 1780 1950 50  0001 C CNN
@@
 	1900 2100 1850 2100
 $Comp
-L Device:R R?
+L Device:R R4
 U 1 1 5FB9038B
 P 2050 2100
-F 0 "R?" V 1950 2100 50  0000 C CNN
+F 0 "R4" V 1950 2100 50  0000 C CNN
 F 1 "1k" V 2050 2100 50  0000 C CNN
 F 2 "" V 1980 2100 50  0001 C CNN
@@
 	1150 700  1150 1250
 $Comp
-L Sensor_Temperature:MCP9700AT-HTT U?
+L Sensor_Temperature:MCP9700AT-HTT U1
 U 1 1 5FB9039A
 P 1150 1550
-F 0 "U?" H 821 1596 50  0000 R CNN
+F 0 "U1" H 821 1596 50  0000 R CNN
 F 1 "MCP9700AT-HTT" H 1800 1800 50  0000 R CNN
 F 2 "Package_TO_SOT_SMD:SOT-23" H 1150 1150 50  0001 C CNN
@@
 	6700 1600 6800 1600
 $Comp
-L Device:L L?
+L Device:L L1
 U 1 1 5FB903CC
 P 6550 1600
-F 0 "L?" V 6369 1600 50  0000 C CNN
+F 0 "L1" V 6369 1600 50  0000 C CNN
 F 1 "28nH" V 6460 1600 50  0000 C CNN
 F 2 "" H 6550 1600 50  0001 C CNN
@@
 	6350 2100 6800 2100
 $Comp
-L Device:C C?
+L Device:C C10
 U 1 1 5FB903DA
 P 7250 4800
-F 0 "C?" H 7365 4846 50  0000 L CNN
+F 0 "C10" H 7365 4846 50  0000 L CNN
 F 1 "0.1uF" H 7365 4755 50  0000 L CNN
 F 2 "" H 7288 4650 50  0001 C CNN
@@
 	8550 2900 8700 2900
 $Comp
-L Device:C C?
+L Device:C C11
 U 1 1 5FB903EB
 P 8400 2900
-F 0 "C?" H 8285 2854 50  0000 R CNN
+F 0 "C11" H 8285 2854 50  0000 R CNN
 F 1 "0.1uF" H 8285 2945 50  0000 R CNN
 F 2 "" H 8438 2750 50  0001 C CNN
@@
 	8150 2800 8150 2900
 $Comp
-L Device:R R?
+L Device:R R5
 U 1 1 5FB903F4
 P 8150 2650
-F 0 "R?" V 8050 2650 50  0000 C CNN
+F 0 "R5" V 8050 2650 50  0000 C CNN
 F 1 "1k" V 8150 2650 50  0000 C CNN
 F 2 "" V 8080 2650 50  0001 C CNN
@@
 	3300 1650 3300 1500
 $Comp
-L Device:C C?
+L Device:C C9
 U 1 1 5FB90443
 P 5700 1350
-F 0 "C?" V 5815 1396 50  0000 L CNN
+F 0 "C9" V 5815 1396 50  0000 L CNN
 F 1 "0.1u" V 5815 1305 50  0000 R CNN
 F 2 "" H 5738 1200 50  0001 C CNN
@@
 $EndComp
 $Comp
-L Device:C C?
+L Device:C C8
 U 1 1 5FB90449
 P 5100 1350
-F 0 "C?" V 5215 1396 50  0000 L CNN
+F 0 "C8" V 5215 1396 50  0000 L CNN
 F 1 "0.1u" V 5215 1305 50  0000 R CNN
 F 2 "" H 5138 1200 50  0001 C CNN
@@
 $EndComp
 $Comp
-L Device:C C?
+L Device:C C7
 U 1 1 5FB9044F
 P 4500 1350
-F 0 "C?" V 4615 1396 50  0000 L CNN
+F 0 "C7" V 4615 1396 50  0000 L CNN
 F 1 "0.1u" V 4615 1305 50  0000 R CNN
 F 2 "" H 4538 1200 50  0001 C CNN
@@
 $EndComp
 $Comp
-L Device:C C?
+L Device:C C6
 U 1 1 5FB90455
 P 3900 1350
-F 0 "C?" V 4015 1396 50  0000 L CNN
+F 0 "C6" V 4015 1396 50  0000 L CNN
 F 1 "0.1u" V 4015 1305 50  0000 R CNN
 F 2 "" H 3938 1200 50  0001 C CNN
@@
 $EndComp
 $Comp
-L Device:C C?
+L Device:C C4
 U 1 1 5FB9045B
 P 3300 1350
-F 0 "C?" V 3415 1396 50  0000 L CNN
+F 0 "C4" V 3415 1396 50  0000 L CNN
 F 1 "0.1u" V 3415 1305 50  0000 R CNN
 F 2 "" H 3338 1200 50  0001 C CNN
@@
 	5700 1700 5700 1650
 $Comp
-L PIC32MZ2048EFM064-I_PT:PIC32MZ2048EFM064-I_PT U?
+L PIC32MZ2048EFM064-I_PT:PIC32MZ2048EFM064-I_PT U3
 U 1 1 5FB90468
 P 4500 3600
-F 0 "U?" H 3000 5350 50  0000 C CNN
+F 0 "U3" H 3000 5350 50  0000 C CNN
 F 1 "PIC32MZ2048EFM064-I_PT" H 3450 1850 50  0000 C CNN
 F 2 "QFP50P1200X1200X120-64N" H 4500 3600 50  0001 L BNN
@@
 P 7950 1850
 AR Path="/5F9673C9/5FB90407" Ref="U?"  Part="1"
-AR Path="/5FB90407" Ref="U?"  Part="1"
-F 0 "U?" H 8300 2200 50  0000 C CNN
+AR Path="/5FB90407" Ref="U5"  Part="1"
+F 0 "U5" H 8300 2200 50  0000 C CNN
 F 1 "MCP2551-I-SN" H 7500 2200 50  0000 C CNN
 F 2 "Package_SO:SOIC-8_3.9x4.9mm_P1.27mm" H 7950 1350 50  0001 C CIN
@@
 3.3V
 $Comp
-L Connector_Generic:Conn_02x10_Counter_Clockwise J?
+L Connector_Generic:Conn_02x10_Counter_Clockwise J5
 U 1 1 5FAE9EF7
 P 6450 6300
-F 0 "J?" V 6454 6780 50  0000 L CNN
+F 0 "J5" V 6454 6780 50  0000 L CNN
 F 1 "Conn to TSI Board" V 6545 6780 50  0000 L CNN
 F 2 "" H 6450 6300 50  0001 C CNN
@@
 Wire Wire Line
 	6850 6600 6850 7400
+NoConn ~ 6350 2500
+NoConn ~ 6350 2600
+NoConn ~ 6350 2900
+NoConn ~ 6350 3400
+NoConn ~ 6350 3500
+NoConn ~ 6350 3600
+NoConn ~ 6350 3800
+NoConn ~ 6350 3900
+NoConn ~ 6350 4000
+NoConn ~ 6350 4100
+NoConn ~ 6350 4300
+NoConn ~ 6350 4400
+NoConn ~ 6350 4700
+NoConn ~ 6350 4800
+$Comp
+L Connector_Generic:Conn_01x06 J18
+U 1 1 5FDCB4A9
+P 750 3950
+F 0 "J18" H 668 4367 50  0000 C CNN
+F 1 "PIC program" H 668 4276 50  0000 C CNN
+F 2 "" H 750 3950 50  0001 C CNN
+F 3 "~" H 750 3950 50  0001 C CNN
+	1    750  3950
+	-1   0    0    -1
+$EndComp
+Wire Wire Line
+	950  3750 1400 3750
+Wire Wire Line
+	950  3850 1400 3850
+Wire Wire Line
+	950  3950 1400 3950
+Wire Wire Line
+	950  4050 1400 4050
+Wire Wire Line
+	950  4150 1400 4150
+NoConn ~ 950  4250
+Text Label 1050 3850 0    50   ~ 0
+3.3V
+Text Label 1050 3750 0    50   ~ 0
+~MCLR~
+Text Label 1050 3950 0    50   ~ 0
+3.3V_rtn
+Text Label 1050 4050 0    50   ~ 0
+PGEC
+Text Label 1050 4150 0    50   ~ 0
+PGED
 $EndSCHEMATC

Commit message: Updated Logic to run off of 5V not 24V
Parts:
- removed C1: 0.1uF, symbol Device:C
- removed U2: PYB20-Q24-S5, CONV_PYB20-Q24-S5, symbol PYB20-Q24-S5:PYB20-Q24-S5
Connections:
- net labels added: 5V_iso, 5V_iso_rtn, D_LED_CTRL
- net labels removed: 24V_iso, 24V_iso_rtn
- wire segments 248 -> 237
- no-connect marks 49 -> 46
Changed lines of the file:
@@
-$EndComp
-$Comp
-L PYB20-Q24-S5:PYB20-Q24-S5 U2
-U 1 1 5F997454
-P 2300 7000
-F 0 "U2" H 2300 7667 50  0000 C CNN
-F 1 "PYB20-Q24-S5" H 2300 7576 50  0000 C CNN
-F 2 "CONV_PYB20-Q24-S5" H 2300 7000 50  0001 L BNN
-F 3 "CUI Inc" H 2300 7000 50  0001 L BNN
-F 4 "1.04" H 2300 7000 50  0001 L BNN "Field4"
-F 5 "Manufacturer Recommendations" H 2300 7000 50  0001 L BNN "Field5"
-	1    2300 7000
-	1    0    0    -1
 $EndComp
 $Comp
@@
 	1    0    0    -1
 $EndComp
-NoConn ~ 1700 6900
-Wire Wire Line
-	850  6800 1150 6800
-Text Label 850  6700 0    50   ~ 0
-24V_iso
-Text Label 850  6800 0    50   ~ 0
-24V_iso_rtn
-Wire Wire Line
-	850  6700 1450 6700
-Wire Wire Line
-	1150 6800 1150 7300
-Wire Wire Line
-	2900 7300 2900 7600
-Wire Wire Line
-	1650 7600 1650 7300
-NoConn ~ 2900 7100
-Connection ~ 2900 7300
 Text Label 3150 6700 0    50   ~ 0
 5V
@@
 Connection ~ 4200 7300
 Wire Wire Line
-	2900 7300 3050 7300
-Wire Wire Line
 	4050 7000 4050 6700
 Wire Wire Line
 	4050 6600 4300 6600
-Wire Wire Line
-	2900 6700 3050 6700
 Connection ~ 4050 6700
 Wire Wire Line
@@
 Wire Wire Line
 	4200 6800 4300 6800
-Connection ~ 1650 7300
-Wire Wire Line
-	1650 7300 1700 7300
-Wire Wire Line
-	1150 7300 1450 7300
-$Comp
-L Device:C C1
-U 1 1 5F99E44C
-P 1450 7000
-F 0 "C1" H 1565 7046 50  0000 L CNN
-F 1 "0.1uF" H 1565 6955 50  0000 L CNN
-F 2 "" H 1488 6850 50  0001 C CNN
-F 3 "~" H 1450 7000 50  0001 C CNN
-	1    1450 7000
-	1    0    0    -1
-$EndComp
-Wire Wire Line
-	1450 6850 1450 6700
-Connection ~ 1450 6700
-Wire Wire Line
-	1450 6700 1700 6700
-Wire Wire Line
-	1450 7150 1450 7300
-Connection ~ 1450 7300
-Wire Wire Line
-	1450 7300 1650 7300
 $Comp
 L Device:C C3
@@
 Wire Wire Line
 	3050 7150 3050 7300
-Connection ~ 3050 7300
 Wire Wire Line
 	3050 6850 3050 6700
-Connection ~ 3050 6700
 Wire Wire Line
 	3050 6700 4050 6700
@@
 Wire Wire Line
 	550  3000 1200 3000
-Wire Wire Line
-	2900 7600 1650 7600
 $Sheet
 S 7900 3900 900  500
@@
 	5950 6900 5950 6600
 Text Label 6850 6050 1    50   ~ 0
-24V_iso
+5V_iso
 Text Label 6750 6050 1    50   ~ 0
-24V_iso_rtn
+5V_iso_rtn
 Text Label 6650 6050 1    50   ~ 0
 SCL_uc
@@
 Text Label 6250 6650 3    50   ~ 0
 PC_ready
-Text Label 6350 6650 3    50   ~ 0
-PC_ready
 Text Label 6450 6650 3    50   ~ 0
 Flowrate
@@
 NoConn ~ 6350 3400
 NoConn ~ 6350 3500
-NoConn ~ 6350 3600
 NoConn ~ 6350 3800
 NoConn ~ 6350 3900
@@
 Text Label 1050 4150 0    50   ~ 0
 PGED
+Wire Wire Line
+	6350 3600 6850 3600
+Text Label 6500 3600 0    50   ~ 0
+D_LED_CTRL
+Text Label 6350 6650 3    50   ~ 0
+D_LED_CTRL
+Wire Wire Line
+	3050 6700 2600 6700
+Connection ~ 3050 6700
+Wire Wire Line
+	3050 7300 2600 7300
+Connection ~ 3050 7300
+Text Label 2600 7300 0    50   ~ 0
+5V_iso_rtn
+Text Label 2600 6700 0    50   ~ 0
+5V_iso
 $EndSCHEMATC

Commit message: Added isolation to CANBUS
Parts:
- removed J5: Conn to TSI Board, symbol Connector_Generic:Conn_02x10_Counter_Clockwise
- added J5: Conn to TSI Board, symbol Connector_Generic:Conn_02x12_Counter_Clockwise
Connections:
- net labels added: 5V_non_iso, GLV_rtn
- wire segments 237 -> 243
- no-connect marks 46 -> 47
Other:
- moved on the sheet: C3, C5, U4

Commit message: Actually isolated things this time
Parts:
- removed R5: 1k, symbol Device:R
- removed U5: MCP2551-I-SN, Package_SO:SOIC-8_3.9x4.9mm_P1.27mm, symbol Interface_CAN_LIN:MCP2551-I-SN
- added C12: 0.1uF, symbol Device:C
- added U5: ISO1050DUB, Package_SO:SOP-8_6.62x9.15mm_P2.54mm, symbol Interface_CAN_LIN:ISO1050DUB
Connections:
- wire segments 243 -> 244
- no-connect marks 47 -> 46
Changed lines of the file:
@@
 Wire Wire Line
 	6550 5150 7050 5150
-Text Label 8150 3050 3    50   ~ 0
+Wire Wire Line
+	6800 3100 6800 2850
+Wire Wire Line
+	6350 3100 6800 3100
+Wire Wire Line
+	6700 2750 6700 3000
+Text Label 7650 2600 1    50   ~ 0
 5V_rtn
-Text Label 8700 2900 2    50   ~ 0
-5V
-Wire Wire Line
-	8150 3050 8150 2900
-Wire Wire Line
-	8550 2900 8700 2900
-$Comp
-L Device:C C11
-U 1 1 5FB903EB
-P 8400 2900
-F 0 "C11" H 8285 2854 50  0000 R CNN
-F 1 "0.1uF" H 8285 2945 50  0000 R CNN
-F 2 "" H 8438 2750 50  0001 C CNN
-F 3 "~" H 8400 2900 50  0001 C CNN
-	1    8400 2900
-	0    1    1    0
-$EndComp
-Wire Wire Line
-	8150 2900 8250 2900
-Connection ~ 8150 2900
-Wire Wire Line
-	8150 2800 8150 2900
-$Comp
-L Device:R R5
-U 1 1 5FB903F4
-P 8150 2650
-F 0 "R5" V 8050 2650 50  0000 C CNN
-F 1 "1k" V 8150 2650 50  0000 C CNN
-F 2 "" V 8080 2650 50  0001 C CNN
-F 3 "~" H 8150 2650 50  0001 C CNN
-	1    8150 2650
-	-1   0    0    1
-$EndComp
-Wire Wire Line
-	8150 2350 8150 2500
-NoConn ~ 8050 2350
-Wire Wire Line
-	6800 3100 6800 2850
-Wire Wire Line
-	6350 3100 6800 3100
-Wire Wire Line
-	6700 2750 6700 3000
-Text Label 8600 1850 2    50   ~ 0
-5V_rtn
-Wire Wire Line
-	8350 1850 8600 1850
-Text Label 7000 1850 2    50   ~ 0
-5V
+Wire Wire Line
+	7650 2350 7650 2600
 Wire Wire Line
 	6350 3000 6700 3000
@@
 	1650 1550 1550 1550
 Wire Wire Line
-	7000 1850 7550 1850
-$Comp
-L Interface_CAN_LIN:MCP2551-I-SN U?
-U 1 1 5FB90407
-P 7950 1850
-AR Path="/5F9673C9/5FB90407" Ref="U?"  Part="1"
-AR Path="/5FB90407" Ref="U5"  Part="1"
-F 0 "U5" H 8300 2200 50  0000 C CNN
-F 1 "MCP2551-I-SN" H 7500 2200 50  0000 C CNN
-F 2 "Package_SO:SOIC-8_3.9x4.9mm_P1.27mm" H 7950 1350 50  0001 C CIN
-F 3 "http://ww1.microchip.com/downloads/en/devicedoc/21667d.pdf" H 7950 1850 50  0001 C CNN
-	1    7950 1850
-	0    -1   -1   0
-$EndComp
-Wire Wire Line
 	6700 2750 7750 2750
 Wire Wire Line
 	7750 2750 7750 2350
 Wire Wire Line
-	6800 2850 7850 2850
-Wire Wire Line
-	7850 2850 7850 2350
-Wire Wire Line
-	8050 1350 8050 850
-Wire Wire Line
-	7850 850  7850 1350
+	7750 1550 7750 1050
 Wire Wire Line
 	1200 5700 1550 5700
 Wire Wire Line
 	1200 5800 1550 5800
-Text Label 7850 1150 1    50   ~ 0
-CAN_H
-Text Label 8050 1150 1    50   ~ 0
+Text Label 7750 1350 1    50   ~ 0
 CAN_L
 Text Label 2550 1650 0    50   ~ 0
@@
 Text Label 5600 7000 3    50   ~ 0
 CAN-
-Wire Wire Line
-	5500 6500 5500 7300
-Wire Wire Line
-	5600 6500 5600 7300
 NoConn ~ 6350 2500
 NoConn ~ 6350 2600
@@
 Text Label 7850 4500 2    50   ~ 0
 GLV_rtn
+Wire Wire Line
+	5500 6500 5500 7550
+Wire Wire Line
+	5600 6500 5600 7550
+Text Label 5500 7300 3    50   ~ 0
+CAN_H
+Text Label 5600 7300 3    50   ~ 0
+CAN_L
+$Comp
+L Interface_CAN_LIN:ISO1050DUB U5
+U 1 1 5F9EC23F
+P 7850 1950
+F 0 "U5" V 7896 2180 50  0000 L CNN
+F 1 "ISO1050DUB" V 7805 2180 50  0000 L CNN
+F 2 "Package_SO:SOP-8_6.62x9.15mm_P2.54mm" H 7850 1600 50  0001 C CIN
+F 3 "http://www.ti.com/lit/ds/symlink/iso1050.pdf" H 7850 1900 50  0001 C CNN
+	1    7850 1950
+	0    1    -1   0
+$EndComp
+$Comp
+L Device:C C?
+U 1 1 5FA132AF
+P 8100 2650
+AR Path="/5F9A7CF0/5FA132AF" Ref="C?"  Part="1"
+AR Path="/5FA132AF" Ref="C11"  Part="1"
+F 0 "C11" H 8215 2696 50  0000 L CNN
+F 1 "0.1uF" H 8215 2605 50  0000 L CNN
+F 2 "" H 8138 2500 50  0001 C CNN
+F 3 "~" H 8100 2650 50  0001 C CNN
+	1    8100 2650
+	0    -1   -1   0
+$EndComp
+Wire Wire Line
+	8250 2650 8300 2650
+Wire Wire Line
+	8300 2650 8300 2550
+Text Label 8300 2550 1    50   ~ 0
+5V_rtn
+Text Label 7950 2550 1    50   ~ 0
+5V
+Wire Wire Line
+	7950 2650 7950 2350
+Wire Wire Line
+	7850 2850 7850 2350
+Wire Wire Line
+	6800 2850 7850 2850
+Text Label 7850 1350 1    50   ~ 0
+CAN_H
+Wire Wire Line
+	7850 1050 7850 1550
+$Comp
+L Device:C C?
+U 1 1 5FADD500
+P 8150 1450
+AR Path="/5F9A7CF0/5FADD500" Ref="C?"  Part="1"
+AR Path="/5FADD500" Ref="C12"  Part="1"
+F 0 "C12" H 8265 1496 50  0000 L CNN
+F 1 "0.1uF" H 8265 1405 50  0000 L CNN
+F 2 "" H 8188 1300 50  0001 C CNN
+F 3 "~" H 8150 1450 50  0001 C CNN
+	1    8150 1450
+	0    1    1    0
+$EndComp
+Wire Wire Line
+	8000 1450 7950 1450
+Wire Wire Line
+	7950 1450 7950 1550
+Text Label 8300 1550 3    50   ~ 0
+GLV_rtn
+Text Label 7950 1550 1    50   ~ 0
+5V_non_iso
+Wire Wire Line
+	8300 1450 8300 1750
+Text Label 7650 1450 1    50   ~ 0
+GLV_rtn
+Wire Wire Line
+	7650 1550 7650 1250
 $EndSCHEMATC

Commit message: Fixed Logic library issue, added I2C translator to Logic, matched I2C names for TSI-Logic
Parts:
- added 200K: R, symbol Device:R
- added U?: PCA9306DCTR, DCT8, symbol CarMan_KiCAD_Library:PCA9306DCTR
- U3: symbol PIC32MZ2048EFM064-I_PT:PIC32MZ2048EFM064-I_PT -> Logic-rescue:PIC32MZ2048EFM064-I_PT-PIC32MZ2048EFM064-I_PT
Connections:
- net labels added: SCL_pi_3.3V, SDA_pi_3.3V
- wire segments 244 -> 246
Other:
- note added: "I2C translator from 5V logic to 3.3V"
- moved on the sheet: C3, C5, U4

Commit message: Fixed Logic Board
Parts:
- removed 200K: R, symbol Device:R
- removed U?: PCA9306DCTR, DCT8, symbol CarMan_KiCAD_Library:PCA9306DCTR
- added D1, D2: LED, symbol Device:LED
- added R5, R6: 10k, symbol Device:R
- C12, C2, C3, C4, C5, C6, C7, C8, C9: symbol Device:C -> Logic-rescue:C-Device-Logic-rescue
- J1: symbol Connector_Generic:Conn_01x04 -> Logic-rescue:Conn_01x04-Connector_Generic-Logic-rescue
- J3: renamed from J2; symbol Connector_Generic:Conn_01x04 -> Logic-rescue:Conn_01x04-Connector_Generic-Logic-rescue
- J4: renamed from J3; symbol Connector_Generic:Conn_01x04 -> Logic-rescue:Conn_01x04-Connector_Generic-Logic-rescue
- J5: symbol Connector_Generic:Conn_02x12_Counter_Clockwise -> Logic-rescue:Conn_02x12_Counter_Clockwise-Connector_Generic-Logic-rescue
- J6: symbol Connector_Generic:Conn_01x08 -> Logic-rescue:Conn_01x08-Connector_Generic-Logic-rescue
- J7: renamed from J4; symbol Connector_Generic:Conn_01x04 -> Logic-rescue:Conn_01x04-Connector_Generic-Logic-rescue
- J8: renamed from J18; symbol Connector_Generic:Conn_01x06 -> Logic-rescue:Conn_01x06-Connector_Generic-Logic-rescue
- L1: symbol Device:L -> Logic-rescue:L-Device-Logic-rescue
- R1, R2, R3, R4: symbol Device:R -> Logic-rescue:R-Device-Logic-rescue
- U1: symbol Sensor_Temperature:MCP9700AT-HTT -> Logic-rescue:MCP9700AT-HTT-Sensor_Temperature-Logic-rescue
- U3: symbol Logic-rescue:PIC32MZ2048EFM064-I_PT-PIC32MZ2048EFM064-I_PT -> PIC32MZ2048EFM064-I_PT:PIC32MZ2048EFM064-I_PT
Connections:
- net labels removed: SCL_pi_3.3V, SDA_pi_3.3V
- wire segments 246 -> 250
Other:
- note removed: "I2C translator from 5V logic to 3.3V"

Commit message: changed logic isolation
Parts:
- removed C3: 0.1uF, symbol Logic-rescue:C-Device-Logic-rescue
- removed C5: 1uF, symbol Logic-rescue:C-Device-Logic-rescue
- removed J7: GLV_I2C, symbol Logic-rescue:Conn_01x04-Connector_Generic-Logic-rescue
- removed U4: LT1763CS8-3.3PBF, SOIC127P600X175-8N, symbol Lafayette_Electric_Car_Internals:LT1763CS8-3.3PBF
- added C18: 0.1uF, symbol Device:C
- added J7: GLV_I2C, symbol Connector_Generic:Conn_01x02
- added R8: 2k, symbol Device:R
- added R9: 3.88k, symbol Device:R
- added U9: ISO1541DR, D8_TEX, symbol CarMan_KiCAD_Library:ISO1541DR
Connections:
- net labels added: 24V, 24V_rtn, 3.3V_non_iso, GLV_SCL, GLV_SDA
- net labels removed: 5V_iso, 5V_iso_rtn, GPIO_I2C_rtn
- wire segments 250 -> 245
- no-connect marks 46 -> 45

Commit message: Added 24v to connection between GLV and Logic and updated headers accordingly
Parts:
- removed J7: GLV_I2C, symbol Connector_Generic:Conn_01x02
- added J7: RTC, symbol Logic-rescue:Conn_01x04-Connector_Generic-Logic-rescue
- U3: symbol PIC32MZ2048EFM064-I_PT:PIC32MZ2048EFM064-I_PT -> Logic-rescue:PIC32MZ2048EFM064-I_PT-PIC32MZ2048EFM064-I_PT
Connections:
- wire segments 245 -> 247
Changed lines of the file:
@@
 EESchema Schematic File Version 4
-EELAYER 30 0
+LIBS:Logic-cache
+EELAYER 29 0
 EELAYER END
 $Descr A4 11693 8268
@@
 	6350 2100 6800 2100
 $Comp
-L PIC32MZ2048EFM064-I_PT:PIC32MZ2048EFM064-I_PT U3
+L Logic-rescue:PIC32MZ2048EFM064-I_PT-PIC32MZ2048EFM064-I_PT U3
 U 1 1 5FB90468
 P 4500 3600
@@
 Text Label 2050 7350 0    50   ~ 0
 3.3V_rtn
-$Comp
-L Connector_Generic:Conn_01x02 J7
-U 1 1 5FB70592
-P 9450 2600
-F 0 "J7" H 9368 2275 50  0000 C CNN
-F 1 "GLV_I2C" H 9368 2366 50  0000 C CNN
-F 2 "" H 9450 2600 50  0001 C CNN
-F 3 "~" H 9450 2600 50  0001 C CNN
-	1    9450 2600
-	-1   0    0    1
-$EndComp
-Wire Wire Line
-	9650 2600 10050 2600
-Wire Wire Line
-	9650 2500 10050 2500
-Text Label 9750 2500 0    50   ~ 0
-GLV_SCL
-Text Label 9750 2600 0    50   ~ 0
-GLV_SDA
 $Sheet
 S 1000 6750 850  850
@@
 	0    -1   -1   0
 $EndComp
+$Comp
+L Logic-rescue:Conn_01x04-Connector_Generic-Logic-rescue J7
+U 1 1 5FB30D0C
+P 9350 2550
+F 0 "J7" H 9430 2542 50  0000 L CNN
+F 1 "RTC" H 9430 2451 50  0000 L CNN
+F 2 "" H 9350 2550 50  0001 C CNN
+F 3 "~" H 9350 2550 50  0001 C CNN
+	1    9350 2550
+	-1   0    0    1
+$EndComp
+Text Label 9550 2650 0    50   ~ 0
+GLV_SCL
+Text Label 9550 2550 0    50   ~ 0
+GLV_SDA
+Text Label 9550 2450 0    50   ~ 0
+GLV_rtn
+Text Label 9550 2350 0    50   ~ 0
+24V
+Wire Wire Line
+	9550 2350 10000 2350
+Wire Wire Line
+	9550 2450 10000 2450
+Wire Wire Line
+	9550 2550 10000 2550
+Wire Wire Line
+	9550 2650 10000 2650
 $EndSCHEMATC
