File: CarMan KiCAD Schematics/Logic/Logic.sch (KiCad schematic (older format))
At the start: 50 parts, among them J1 Motor Controller Can Line, J10 Motor Controller Can Line, J2 IMU PS, J3 Insulation Monitoring Unit, J4 Real Time Clock, J5.1 Conn_01x06, J5.2 Conn_01x06, J6 You're Welcome -Ethan, J7 GLV BOB, J8 PIC program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

Commit message: Logic update
Other:
- note added: "IMU Addressing Pins"
- note removed: "IMU PS"
Changed lines of the file:
@@
 Wire Wire Line
 	7825 10375 8575 10375
-Text Notes 11475 1425 0    50   ~ 0
-IMU PS
+Text Notes 11450 1375 0    50   ~ 0
+IMU Addressing Pins
 Text Notes 13325 1500 0    50   ~ 0
 RTC

Commit message: routed TSI board
Parts:
- gave numbers to parts that had none: 6
Changed lines of the file:
@@
 NoConn ~ 6725 3575
 $Comp
-L Device:LED D?
+L Device:LED D7
 U 1 1 6074CAEC
 P 1400 8675
-F 0 "D?" V 1439 8557 50  0000 R CNN
+F 0 "D7" V 1439 8557 50  0000 R CNN
 F 1 "LED" V 1348 8557 50  0000 R CNN
 F 2 "CarMan General Footprints:VAOL-S8GT4" H 1400 8675 50  0001 C CNN
@@
 $EndComp
 $Comp
-L Device:LED D?
+L Device:LED D8
 U 1 1 6074CAF2
 P 2050 8675
-F 0 "D?" V 2089 8557 50  0000 R CNN
+F 0 "D8" V 2089 8557 50  0000 R CNN
 F 1 "LED" V 1998 8557 50  0000 R CNN
 F 2 "CarMan General Footprints:VAOL-S8GT4" H 2050 8675 50  0001 C CNN
@@
 ISO_RTN
 $Comp
-L Device:R R?
+L Device:R R9
 U 1 1 6074CAFB
 P 1400 8375
-F 0 "R?" H 1470 8421 50  0000 L CNN
+F 0 "R9" H 1470 8421 50  0000 L CNN
 F 1 "10k" H 1470 8330 50  0000 L CNN
 F 2 "Resistor_SMD:R_0805_2012Metric_Pad1.15x1.40mm_HandSolder" V 1330 8375 50  0001 C CNN
@@
 $EndComp
 $Comp
-L Device:R R?
+L Device:R R11
 U 1 1 6074CB01
 P 2050 8375
-F 0 "R?" H 2120 8421 50  0000 L CNN
+F 0 "R11" H 2120 8421 50  0000 L CNN
 F 1 "10k" H 2120 8330 50  0000 L CNN
 F 2 "Resistor_SMD:R_0805_2012Metric_Pad1.15x1.40mm_HandSolder" V 1980 8375 50  0001 C CNN
@@
 	2050 8225 2050 8125
 $Comp
-L Device:LED D?
+L Device:LED D4
 U 1 1 6074CB0B
 P 750 8675
-F 0 "D?" V 789 8557 50  0000 R CNN
+F 0 "D4" V 789 8557 50  0000 R CNN
 F 1 "LED" V 698 8557 50  0000 R CNN
 F 2 "CarMan General Footprints:VAOL-S8GT4" H 750 8675 50  0001 C CNN
@@
 	750  8825 750  9025
 $Comp
-L Device:R R?
+L Device:R R8
 U 1 1 6074CB12
 P 750 8375
-F 0 "R?" H 820 8421 50  0000 L CNN
+F 0 "R8" H 820 8421 50  0000 L CNN
 F 1 "10k" H 820 8330 50  0000 L CNN
 F 2 "Resistor_SMD:R_0805_2012Metric_Pad1.15x1.40mm_HandSolder" V 680 8375 50  0001 C CNN

Commit message: Balls balls balls
Parts:
- removed J5.1: Conn_01x06, Connector_PinSocket_2.54mm:PinSocket_1x06_P2.54mm_Vertical, symbol Connector_Generic:Conn_01x06
- removed J5.2: Conn_01x06, Connector_PinSocket_2.54mm:PinSocket_1x08_P2.54mm_Vertical, symbol Connector_Generic:Conn_01x06
- added J5: Conn_02x06_Odd_Even, Connector_PinSocket_2.54mm:PinSocket_2x06_P2.54mm_Vertical, symbol Connector_Generic:Conn_02x06_Odd_Even
Changed lines of the file:
@@
 Text Label 3550 6875 0    50   ~ 0
 GLV_RTN
-Text Label 12575 2225 2    50   ~ 0
+Text Label 12475 2225 2    50   ~ 0
 CAN_H
-Text Label 12575 2125 2    50   ~ 0
+Text Label 12475 2125 2    50   ~ 0
 CAN_L
 Text Label 13250 5900 0    50   ~ 0
@@
 NoConn ~ 3075 3775
 NoConn ~ 6725 4875
-$Comp
-L Connector_Generic:Conn_01x06 J5.2
-U 1 1 5FB98586
-P 11625 2125
-F 0 "J5.2" H 11525 2425 50  0000 L CNN
-F 1 "Conn_01x06" H 11705 2026 50  0001 L CNN
-F 2 "Connector_PinSocket_2.54mm:PinSocket_1x08_P2.54mm_Vertical" H 11625 2125 50  0001 C CNN
-F 3 "~" H 11625 2125 50  0001 C CNN
-	1    11625 2125
-	-1   0    0    -1
-$EndComp
-$Comp
-L Connector_Generic:Conn_01x06 J5.1
-U 1 1 5FB8432E
-P 11425 2125
-F 0 "J5.1" H 11325 2425 50  0000 L CNN
-F 1 "Conn_01x06" H 11505 2026 50  0001 L CNN
-F 2 "Connector_PinSocket_2.54mm:PinSocket_1x06_P2.54mm_Vertical" H 11425 2125 50  0001 C CNN
-F 3 "~" H 11425 2125 50  0001 C CNN
-	1    11425 2125
-	1    0    0    -1
-$EndComp
-Text Label 12575 2325 2    50   ~ 0
+Text Label 12475 2325 2    50   ~ 0
 ISO_RTN
 Text Label 10475 1925 0    50   ~ 0
@@
 Text Label 15300 9275 2    50   ~ 0
 SDA_TSI_GLV
-Text Label 12575 1925 2    50   ~ 0
+Text Label 12475 1925 2    50   ~ 0
 SDA_TSI_GLV
-Text Label 12575 2025 2    50   ~ 0
+Text Label 12475 2025 2    50   ~ 0
 SCL_TSI_GLV
 $Comp
@@
 	3475 10950 3825 10950
 Wire Wire Line
-	11825 2025 12575 2025
-Wire Wire Line
-	11825 1925 12575 1925
-Wire Wire Line
-	12575 2325 11825 2325
+	11725 2025 12475 2025
+Wire Wire Line
+	11725 1925 12475 1925
+Wire Wire Line
+	12475 2325 11725 2325
 Wire Wire Line
 	10475 1925 11225 1925
@@
 NoConn ~ 3075 3375
 Wire Wire Line
-	12575 2225 11825 2225
-Wire Wire Line
-	11825 2125 12575 2125
-Text Label 11875 2225 0    50   ~ 0
+	12475 2225 11725 2225
+Wire Wire Line
+	11725 2125 12475 2125
+Text Label 11775 2225 0    50   ~ 0
 BP_CAN+
-Text Label 11875 2125 0    50   ~ 0
+Text Label 11775 2125 0    50   ~ 0
 BP_CAN-
 NoConn ~ 3075 3575
@@
 Text Label 2400 4575 0    50   ~ 0
 FlowRate
-Text Label 12575 2425 2    50   ~ 0
+Text Label 12475 2425 2    50   ~ 0
 3.3V_ISO
 Wire Wire Line
-	12575 2425 11825 2425
+	12475 2425 11725 2425
 Text Label 10475 2425 0    50   ~ 0
 ADC_RTN
@@
 Wire Wire Line
 	2400 4775 2400 4875
+$Comp
+L Connector_Generic:Conn_02x06_Odd_Even J5
+U 1 1 607A60D6
+P 11425 2125
+F 0 "J5" H 11475 2450 50  0000 C CNN
+F 1 "Conn_02x06_Odd_Even" H 11475 2451 50  0001 C CNN
+F 2 "Connector_PinSocket_2.54mm:PinSocket_2x06_P2.54mm_Vertical" H 11425 2125 50  0001 C CNN
+F 3 "~" H 11425 2125 50  0001 C CNN
+	1    11425 2125
+	1    0    0    -1
+$EndComp
 $EndSCHEMATC

Commit message: TSI Logic Changes
Parts:
- removed J2: IMU PS, Connector_PinHeader_2.54mm:PinHeader_1x02_P2.54mm_Vertical, symbol Connector_Generic:Conn_01x02
- removed J3: Insulation Monitoring Unit, Connector_PinHeader_2.54mm:PinHeader_1x05_P2.54mm_Vertical, symbol Logic-rescue:Conn_01x04-Connector_Generic-Logic-rescue
- added U10: BNO_055, CarMan General Footprints:BNO_055, symbol CarMan_KiCAD_Library:BNO_055
Connections:
- net 3.3V_ISO: now also U10.1 (Vin)
- net ISO_RTN: now also U10.3 (GND), U10.6 (PS1), U10.7 (PS0)
- net SCL_ISO_PI: now also U10.4 (SCL)
- net SDA_ISO_PI: now also U10.5 (SDA)
- no-connect marks 49 -> 50
Other:
- note removed: "IMU Addressing Pins"
Changed lines of the file:
@@
 $EndDescr
-$Comp
-L Logic-rescue:Conn_01x04-Connector_Generic-Logic-rescue J3
-U 1 1 5F95B303
-P 12400 1250
-F 0 "J3" H 12350 950 50  0000 L CNN
-F 1 "Insulation Monitoring Unit" H 12325 1450 50  0001 L CNN
-F 2 "Connector_PinHeader_2.54mm:PinHeader_1x05_P2.54mm_Vertical" H 12400 1250 50  0001 C CNN
-F 3 "~" H 12400 1250 50  0001 C CNN
-	1    12400 1250
-	-1   0    0    1
-$EndComp
 $Comp
 L Logic-rescue:Conn_01x04-Connector_Generic-Logic-rescue J4
@@
 NoConn ~ 10900 1025
 Wire Wire Line
-	12600 1350 13050 1350
-Wire Wire Line
 	13575 1250 14025 1250
 Wire Wire Line
@@
 Text Label 14025 1150 2    50   ~ 0
 SDA_ISO_PI
-Text Label 13050 1050 2    50   ~ 0
+Text Label 11650 1250 0    50   ~ 0
 SCL_ISO_PI
-Text Label 13050 1150 2    50   ~ 0
+Text Label 11650 1350 0    50   ~ 0
 SDA_ISO_PI
-Text Label 13050 1250 2    50   ~ 0
-ISO_RTN
-Text Label 13050 1350 2    50   ~ 0
-3.3V_ISO
+Text Label 11650 1150 0    50   ~ 0
+ISO_RTN
 Text Label 10575 8575 2    50   ~ 0
 5V_ISO
@@
 	5475 1975 5475 1925
 Wire Wire Line
-	12600 1050 13050 1050
-Wire Wire Line
-	12600 1150 13050 1150
+	12100 1250 11650 1250
+Wire Wire Line
+	12100 1350 11650 1350
 Wire Wire Line
 	13575 1050 14025 1050
@@
 Wire Wire Line
 	1400 10825 2050 10825
-$Comp
-L Connector_Generic:Conn_01x02 J2
-U 1 1 6025C7CF
-P 11625 1075
-F 0 "J2" H 11575 1175 50  0000 L CNN
-F 1 "IMU PS" H 11475 850 50  0001 L CNN
-F 2 "Connector_PinHeader_2.54mm:PinHeader_1x02_P2.54mm_Vertical" H 11625 1075 50  0001 C CNN
-F 3 "~" H 11625 1075 50  0001 C CNN
-	1    11625 1075
-	-1   0    0    -1
-$EndComp
 Wire Wire Line
 	14150 2000 14850 2000
@@
 Text Notes 11150 2575 0    50   ~ 0
 Logic-TSI Connector
-Text Label 12150 1075 2    50   ~ 0
-ISO_RTN
-Wire Wire Line
-	12600 1250 13050 1250
+Text Label 13025 1150 2    50   ~ 0
+ISO_RTN
+Wire Wire Line
+	12100 1150 11650 1150
 Wire Wire Line
 	14150 2100 14850 2100
@@
 Text Label 11350 1225 2    50   ~ 0
 CAN_L
-Text Notes 12325 1475 0    47   ~ 0
+Text Notes 12325 1525 0    47   ~ 0
 IMU
 Wire Wire Line
@@
 	10900 1325 11350 1325
 Wire Wire Line
-	11825 1075 12150 1075
-Wire Wire Line
-	12150 1075 12150 1175
-Wire Wire Line
-	12150 1175 11825 1175
+	12700 1150 13025 1150
+Wire Wire Line
+	13025 1150 13025 1250
+Wire Wire Line
+	13025 1250 12700 1250
 Wire Wire Line
 	7825 9875 8575 9875
@@
 Wire Wire Line
 	7825 10375 8575 10375
-Text Notes 11450 1375 0    50   ~ 0
-IMU Addressing Pins
 Text Notes 13325 1500 0    50   ~ 0
 RTC
@@
 	1    0    0    -1
 $EndComp
+$Comp
+L CarMan_KiCAD_Library:BNO_055 U10
+U 1 1 6081110B
+P 12400 1150
+F 0 "U10" V 11981 1150 47  0000 C CNN
+F 1 "BNO_055" V 12068 1150 47  0000 C CNN
+F 2 "CarMan General Footprints:BNO_055" H 12400 1150 47  0001 C CNN
+F 3 "" H 12400 1150 47  0001 C CNN
+	1    12400 1150
+	0    1    1    0
+$EndComp
+Text Label 11650 950  0    50   ~ 0
+3.3V_ISO
+Wire Wire Line
+	12100 950  11650 950
+NoConn ~ 12100 1050
 $EndSCHEMATC

Commit message: TSI Logic changes the 2nd
Parts:
- removed J5: Conn_02x06_Odd_Even, Connector_PinSocket_2.54mm:PinSocket_2x06_P2.54mm_Vertical, symbol Connector_Generic:Conn_02x06_Odd_Even
- added J14: Conn_02x05_Odd_Even, Connector_PinSocket_2.54mm:PinSocket_2x05_P2.54mm_Vertical, symbol Connector_Generic:Conn_02x05_Odd_Even
Connections:
- net 3.3V_ISO: now also J14.7 (Pin_7)
- net BP_CAN+: now also J14.8 (Pin_8)
- net BP_CAN-: now also J14.6 (Pin_6)
- net Cooling_CTRL: now also J14.1 (Pin_1)
- net FlowRate: now also J14.9 (Pin_9)
- net ISO_RTN: now also J14.5 (Pin_5)
- net SCL_TSI_GLV: now also J14.4 (Pin_4)
- net SDA_TSI_GLV: now also J14.2 (Pin_2)
- net SR_CTRL: now also J14.3 (Pin_3)
- net ADC_RTN: no longer names the net of U3.23 (TMS/CVREFOUT/AN5/RPB10/PMA13/RB10)
- net ADC_RTN: no longer U3.24 (TDO/AN6/PMA12/RB11)
- net APPS: no longer names the net of U3.11 (AN45/C1INA/RPB5/RB5)
- net CoolTemp: no longer names the net of U3.17 (PGEC2/AN46/RPB6/RB6)
- no-connect marks 50 -> 55
Changed lines of the file:
@@
 NoConn ~ 3075 3775
 NoConn ~ 6725 4875
-Text Label 12475 2325 2    50   ~ 0
+Text Label 10475 2125 0    50   ~ 0
 ISO_RTN
 Text Label 10475 1925 0    50   ~ 0
@@
 Wire Wire Line
 	11725 1925 12475 1925
-Wire Wire Line
-	12475 2325 11725 2325
 Wire Wire Line
 	10475 1925 11225 1925
@@
 Wire Wire Line
 	14775 9475 15500 9475
-Text Label 10475 2225 0    50   ~ 0
-CoolTemp
-Wire Wire Line
-	10475 2225 11225 2225
 Text Label 10475 2325 0    50   ~ 0
 FlowRate
 Wire Wire Line
 	10475 2325 11225 2325
-Text Label 10475 2125 0    50   ~ 0
-APPS
-Wire Wire Line
-	10475 2125 11225 2125
 NoConn ~ 9625 9275
 NoConn ~ 3075 3975
@@
 Wire Notes Line
 	2550 7650 2550 9300
-Text Label 7400 3875 2    47   ~ 0
-STATE_OUT_1
-Wire Wire Line
-	7400 3875 6725 3875
-Text Label 7400 3975 2    47   ~ 0
-STATE_OUT_2
-Wire Wire Line
-	7400 3975 6725 3975
-Text Label 7400 4075 2    47   ~ 0
-STATE_OUT_3
-Wire Wire Line
-	7400 4075 6725 4075
 Text Label 1400 8125 0    50   ~ 0
 STATE_OUT_2
@@
 NoConn ~ 3075 2675
 NoConn ~ 3075 2575
-Text Label 2400 3875 0    50   ~ 0
-APPS
-Wire Wire Line
-	2400 3875 3075 3875
-Wire Wire Line
-	2400 4475 3075 4475
 Wire Wire Line
 	2400 4575 3075 4575
-Text Label 2400 4475 0    50   ~ 0
-CoolTemp
 Text Label 2400 4575 0    50   ~ 0
 FlowRate
-Text Label 12475 2425 2    50   ~ 0
+Text Label 10475 2225 0    50   ~ 0
 3.3V_ISO
-Wire Wire Line
-	12475 2425 11725 2425
-Text Label 10475 2425 0    50   ~ 0
-ADC_RTN
-Wire Wire Line
-	10475 2425 11225 2425
-Wire Wire Line
-	2400 4775 3075 4775
-Wire Wire Line
-	2400 4875 3075 4875
-Text Label 2400 4775 0    50   ~ 0
-ADC_RTN
-Wire Wire Line
-	2400 4775 2400 4875
-$Comp
-L Connector_Generic:Conn_02x06_Odd_Even J5
-U 1 1 607A60D6
-P 11425 2125
-F 0 "J5" H 11475 2450 50  0000 C CNN
-F 1 "Conn_02x06_Odd_Even" H 11475 2451 50  0001 C CNN
-F 2 "Connector_PinSocket_2.54mm:PinSocket_2x06_P2.54mm_Vertical" H 11425 2125 50  0001 C CNN
-F 3 "~" H 11425 2125 50  0001 C CNN
-	1    11425 2125
-	1    0    0    -1
-$EndComp
 $Comp
 L CarMan_KiCAD_Library:BNO_055 U10
@@
 	12100 950  11650 950
 NoConn ~ 12100 1050
+Wire Wire Line
+	7400 4075 6725 4075
+Text Label 7400 4075 2    47   ~ 0
+STATE_OUT_3
+Wire Wire Line
+	7400 3975 6725 3975
+Text Label 7400 3975 2    47   ~ 0
+STATE_OUT_2
+Wire Wire Line
+	7400 3875 6725 3875
+Text Label 7400 3875 2    47   ~ 0
+STATE_OUT_1
+NoConn ~ 11725 2325
+NoConn ~ 3075 4775
+NoConn ~ 3075 4875
+NoConn ~ 3075 4475
+NoConn ~ 3075 3875
+Wire Wire Line
+	10475 2125 11225 2125
+Wire Wire Line
+	10475 2225 11225 2225
+$Comp
+L Connector_Generic:Conn_02x05_Odd_Even J14
+U 1 1 609BCAC7
+P 11425 2125
+F 0 "J14" H 11475 2542 50  0000 C CNN
+F 1 "Conn_02x05_Odd_Even" H 11475 2451 50  0000 C CNN
+F 2 "Connector_PinSocket_2.54mm:PinSocket_2x05_P2.54mm_Vertical" H 11425 2125 50  0001 C CNN
+F 3 "~" H 11425 2125 50  0001 C CNN
+	1    11425 2125
+	1    0    0    -1
+$EndComp
 $EndSCHEMATC

Commit message: Updated TSI Schematic
Parts:
- J2: renamed from J10; value Motor Controller Can Line -> NON-ISO I2C Testing Header
- J3: renamed from J14; value Conn_02x05_Odd_Even -> Logic-TSI Connector
- renumbered J7 to J4, J8 to J5, J4 to J666
Other:
- note added: "Mounted External Components"
- note added: "NON-ISO I2C Testing Header"
- note added: "Needs to be changed"
- note added: "Symbol & Footprint for IMU to\nbe mounted to the Logic board"
- note removed: "IMU"
- note removed: "NON-ISO I2C\nTesting Header"
- moved on the sheet: D3, D5, J1, J2, J3, J4, J5, J6, J666, R13, R15, U1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
