File: CarMan KiCAD Schematics/Logic/LogicPower.sch (KiCad schematic (older format))
At the start: 5 parts, among them U4 PYB20-Q24-S5, U7 LT1763CS8-3.3PBF

Commit message: Aesthetics
Parts:
- U7: symbol Lafayette_Electric_Car_Internals:LT1763CS8-3.3PBF -> Logic-rescue:LT1763CS8-3.3PBF-Lafayette_Electric_Car_Internals
Changed lines of the file:
@@
 	7100 1400 8600 1400
 $Comp
-L Lafayette_Electric_Car_Internals:LT1763CS8-3.3PBF U?
+L Logic-rescue:LT1763CS8-3.3PBF-Lafayette_Electric_Car_Internals U?
 U 1 1 5FAF664A
 P 7900 2250
