File: CarMan KiCAD Schematics/Logic/LogicPower.sch (KiCad schematic (older format))
At the start: 5 parts, among them U4 PYB20-Q24-S5, U7 LT1763CS8-3.3PBF

Commit message: Logic Footprints in General Library, Added Logic LEDs
Parts:
- C13, C3, C5: footprint (none) -> Capacitor_SMD:C_0805_2012Metric_Pad1.15x1.40mm_HandSolder
- U4: footprint CONV_PYB20-Q24-S5 -> CarMan General Footprints:CONV_PYB20-Q24-S5
Changed lines of the file:
@@
 F 0 "C5" H 6065 2396 50  0000 L CNN
 F 1 "0.1uF" H 6065 2305 50  0000 L CNN
-F 2 "" H 5988 2200 50  0001 C CNN
+F 2 "Capacitor_SMD:C_0805_2012Metric_Pad1.15x1.40mm_HandSolder" H 5988 2200 50  0001 C CNN
 F 3 "~" H 5950 2350 50  0001 C CNN
 	1    5950 2350
@@
 F 0 "C13" H 6815 2446 50  0000 L CNN
 F 1 "1uF" H 6815 2355 50  0000 L CNN
-F 2 "" H 6738 2250 50  0001 C CNN
+F 2 "Capacitor_SMD:C_0805_2012Metric_Pad1.15x1.40mm_HandSolder" H 6738 2250 50  0001 C CNN
 F 3 "~" H 6700 2400 50  0001 C CNN
 	1    6700 2400
@@
 F 0 "U4" H 4900 3017 50  0000 C CNN
 F 1 "PYB20-Q24-S5" H 4900 2926 50  0000 C CNN
-F 2 "CONV_PYB20-Q24-S5" H 4900 2350 50  0001 L BNN
+F 2 "CarMan General Footprints:CONV_PYB20-Q24-S5" H 4900 2350 50  0001 L BNN
 F 3 "CUI Inc" H 4900 2350 50  0001 L BNN
 F 4 "Manufacturer Recommendations" H 4900 2350 50  0001 L BNN "Field4"
@@
 F 0 "C3" H 3915 2396 50  0000 L CNN
 F 1 "0.1uF" H 3915 2305 50  0000 L CNN
-F 2 "" H 3838 2200 50  0001 C CNN
+F 2 "Capacitor_SMD:C_0805_2012Metric_Pad1.15x1.40mm_HandSolder" H 3838 2200 50  0001 C CNN
 F 3 "~" H 3800 2350 50  0001 C CNN
 	1    3800 2350

Commit message: Logic PCB started, Pi 3B footprint fixed
Parts:
- U7: footprint SOIC127P600X175-8N -> CarMan General Footprints:LT1763CS8-3-PBF
Changed lines of the file:
@@
 F 0 "U7" H 7900 2920 50  0000 C CNN
 F 1 "LT1763CS8-3.3PBF" H 7900 2829 50  0000 C CNN
-F 2 "SOIC127P600X175-8N" H 7900 2250 50  0001 L BNN
+F 2 "CarMan General Footprints:LT1763CS8-3-PBF" H 7900 2250 50  0001 L BNN
 F 3 "Voltage stabiliser; LDO, fixed; 3.3V; 500mA; SO8; SMD" H 7900 2250 50  0001 L BNN
 F 4 "Linear Technology/Analog" H 7900 2250 50  0001 L BNN "Field4"

Commit message: - limited shorting wires and clarified ISO connections - Removed 5V_rtn and 3.3V_rtn and changed to ISO_RTN - 3.3V designated as 3.3V_ISO - 5V designated as 5V_ISO
Connections:
- net 24V_rtn renamed GLV_RTN
- net 3.3V renamed 3.3V_ISO
- net 3.3V_rtn renamed ISO_RTN
- net 5V renamed 5V_ISO
Changed lines of the file:
@@
 $EndDescr
 Text Label 6050 2050 0    50   ~ 0
-5V
-Text Label 6050 2650 0    50   ~ 0
-5V_rtn
+5V_ISO
 Wire Wire Line
 	7200 2550 7100 2550
@@
 	6700 2150 7100 2150
 Connection ~ 7100 2150
-Wire Wire Line
-	7100 2750 7100 3100
-Connection ~ 7100 2750
-Text Label 7100 3100 1    50   ~ 0
-3.3V_rtn
+Text Label 6575 2650 2    50   ~ 0
+ISO_RTN
 Text Label 8400 1400 0    50   ~ 0
-3.3V
+3.3V_ISO
 Wire Wire Line
 	5950 2050 5500 2050
@@
 	5950 2650 5500 2650
 Connection ~ 5950 2650
-Wire Wire Line
-	5950 2650 7100 2650
 $Comp
 L power:PWR_FLAG #FLG03
 U 1 1 5FAF663E
-P 7100 3100
-F 0 "#FLG03" H 7100 3175 50  0001 C CNN
-F 1 "PWR_FLAG" V 7100 3228 50  0000 L CNN
-F 2 "" H 7100 3100 50  0001 C CNN
-F 3 "~" H 7100 3100 50  0001 C CNN
-	1    7100 3100
-	0    1    1    0
+P 6150 2875
+F 0 "#FLG03" H 6150 2950 50  0001 C CNN
+F 1 "PWR_FLAG" H 5975 3050 50  0000 L CNN
+F 2 "" H 6150 2875 50  0001 C CNN
+F 3 "~" H 6150 2875 50  0001 C CNN
+	1    6150 2875
+	-1   0    0    1
 $EndComp
 Wire Wire Line
@@
 24V
 Text HLabel 1150 800  0    50   Input ~ 0
-24V_rtn
-Text HLabel 1150 950  0    50   Input ~ 0
-5V
-Text HLabel 1150 1100 0    50   Input ~ 0
-5V_rtn
+GLV_RTN
+Text HLabel 1125 1350 0    50   Output ~ 0
+5V_ISO
 $Comp
 L CarMan_KiCAD_Library:PYB20-Q24-S5 U4
@@
 	1    0    0    -1
 $EndComp
-Text HLabel 1150 1250 0    50   Input ~ 0
-3.3V
-Text HLabel 1150 1400 0    50   Input ~ 0
-3.3V_rtn
+Text HLabel 1125 1450 0    50   Output ~ 0
+3.3V_ISO
+Text HLabel 1125 1550 0    50   Output ~ 0
+ISO_RTN
 Wire Wire Line
 	1150 650  1500 650
@@
 	1150 800  1500 800
 Wire Wire Line
-	1150 950  1500 950
-Wire Wire Line
-	1150 1100 1500 1100
-Wire Wire Line
-	1150 1250 1500 1250
-Wire Wire Line
-	1150 1400 1500 1400
+	1125 1350 1475 1350
+Wire Wire Line
+	1125 1450 1475 1450
+Wire Wire Line
+	1125 1550 1475 1550
 Text Label 1500 650  0    50   ~ 0
 24V
 Text Label 1500 800  0    50   ~ 0
-24V_rtn
-Text Label 1500 950  0    50   ~ 0
-5V
-Text Label 1500 1100 0    50   ~ 0
-5V_rtn
-Text Label 1500 1250 0    50   ~ 0
-3.3V
-Text Label 1500 1400 0    50   ~ 0
-3.3V_rtn
+GLV_RTN
+Text Label 1475 1350 0    50   ~ 0
+5V_ISO
+Text Label 1475 1450 0    50   ~ 0
+3.3V_ISO
+Text Label 1475 1550 0    50   ~ 0
+ISO_RTN
 NoConn ~ 5500 2450
 NoConn ~ 4300 2250
@@
 	3800 2650 4300 2650
 Text Label 3900 2650 0    50   ~ 0
-24V_rtn
+GLV_RTN
 Text Label 3950 2050 0    50   ~ 0
 24V
@@
 $EndComp
 Connection ~ 3800 2650
+Wire Wire Line
+	5950 2650 6150 2650
+Wire Wire Line
+	6150 2650 6150 2875
+Connection ~ 6150 2650
+Wire Wire Line
+	6150 2650 7100 2650
 $EndSCHEMATC

Commit message: Super organized logic
Other:
- note added: "24V -> 5V_ISO & 3.3V_ISO"
- note added: "ISO"
- note added: "NON-ISO"
- note added: "SIGNALS"
- moved on the sheet: C13, C3, C5, U4, U7

Commit message: Logic Update
Other:
- note added: "24V_NON_ISO -> 5V_ISO"
- note added: "5V_ISO -> 3.3V_ISO"
- moved on the sheet: C5
Changed lines of the file:
@@
 L Device:C C5
 U 1 1 5FAF6616
-P 5500 3775
-F 0 "C5" H 5615 3821 50  0000 L CNN
-F 1 "0.1uF" H 5615 3730 50  0000 L CNN
-F 2 "Capacitor_SMD:C_0805_2012Metric_Pad1.15x1.40mm_HandSolder" H 5538 3625 50  0001 C CNN
-F 3 "~" H 5500 3775 50  0001 C CNN
-	1    5500 3775
-	1    0    0    -1
-$EndComp
-Wire Wire Line
-	5500 3925 5500 4075
-Wire Wire Line
-	5500 3625 5500 3475
+P 5700 3775
+F 0 "C5" H 5815 3821 50  0000 L CNN
+F 1 "0.1uF" H 5815 3730 50  0000 L CNN
+F 2 "Capacitor_SMD:C_0805_2012Metric_Pad1.15x1.40mm_HandSolder" H 5738 3625 50  0001 C CNN
+F 3 "~" H 5700 3775 50  0001 C CNN
+	1    5700 3775
+	1    0    0    -1
+$EndComp
+Wire Wire Line
+	5700 3925 5700 4075
+Wire Wire Line
+	5700 3625 5700 3475
 $Comp
 L Logic-rescue:C-Device-Logic-rescue C13
@@
 Text Label 5400 4075 2    50   ~ 0
 ISO_RTN
-Wire Wire Line
-	5500 3475 5050 3475
-Connection ~ 5500 3475
-Wire Wire Line
-	5500 4075 5050 4075
-Connection ~ 5500 4075
 $Comp
 L power:PWR_FLAG #FLG03
@@
 AR Path="/5FAF664A" Ref="U?"  Part="1"
 AR Path="/5FAD1CB8/5FAF664A" Ref="U7"  Part="1"
-F 0 "U7" H 7450 4445 50  0000 C CNN
-F 1 "LT1763CS8-3.3PBF" H 7450 4354 50  0000 C CNN
+F 0 "U7" H 7450 4325 50  0000 C CNN
+F 1 "LT1763CS8-3.3PBF" H 7450 3025 50  0000 C CNN
 F 2 "CarMan General Footprints:LT1763CS8-3-PBF" H 7450 3775 50  0001 L BNN
 F 3 "Voltage stabiliser; LDO, fixed; 3.3V; 500mA; SO8; SMD" H 7450 3775 50  0001 L BNN
@@
 U 1 1 5FAF8405
 P 4450 3775
-F 0 "U4" H 4450 4442 50  0000 C CNN
-F 1 "PYB20-Q24-S5" H 4450 4351 50  0000 C CNN
+F 0 "U4" H 4450 4325 50  0000 C CNN
+F 1 "PYB20-Q24-S5" H 4450 3225 50  0000 C CNN
 F 2 "CarMan General Footprints:CONV_PYB20-Q24-S5" H 4450 3775 50  0001 L BNN
 F 3 "CUI Inc" H 4450 3775 50  0001 L BNN
@@
 	3350 3475 3350 3625
 Wire Wire Line
-	3350 3925 3350 4075
-Wire Wire Line
 	3350 4075 3850 4075
 Text Label 3450 4075 0    50   ~ 0
@@
 L power:PWR_FLAG #FLG01
 U 1 1 5FAFECF7
-P 3350 3475
-F 0 "#FLG01" H 3350 3550 50  0001 C CNN
-F 1 "PWR_FLAG" H 3350 3648 50  0000 C CNN
-F 2 "" H 3350 3475 50  0001 C CNN
-F 3 "~" H 3350 3475 50  0001 C CNN
-	1    3350 3475
-	1    0    0    -1
-$EndComp
-Connection ~ 3350 3475
+P 3350 3250
+F 0 "#FLG01" H 3350 3325 50  0001 C CNN
+F 1 "PWR_FLAG" H 3350 3423 50  0000 C CNN
+F 2 "" H 3350 3250 50  0001 C CNN
+F 3 "~" H 3350 3250 50  0001 C CNN
+	1    3350 3250
+	1    0    0    -1
+$EndComp
 $Comp
 L power:PWR_FLAG #FLG0101
 U 1 1 5FB6EF51
-P 3350 4075
-F 0 "#FLG0101" H 3350 4150 50  0001 C CNN
-F 1 "PWR_FLAG" V 3350 4203 50  0000 L CNN
-F 2 "" H 3350 4075 50  0001 C CNN
-F 3 "~" H 3350 4075 50  0001 C CNN
-	1    3350 4075
+P 3350 4300
+F 0 "#FLG0101" H 3350 4375 50  0001 C CNN
+F 1 "PWR_FLAG" H 3175 4450 50  0000 L CNN
+F 2 "" H 3350 4300 50  0001 C CNN
+F 3 "~" H 3350 4300 50  0001 C CNN
+	1    3350 4300
 	-1   0    0    1
 $EndComp
-Connection ~ 3350 4075
-Wire Wire Line
-	5500 4075 5700 4075
 Wire Wire Line
 	5700 4075 5700 4300
@@
 3.3V_ISO
 Wire Wire Line
-	5500 3475 6625 3475
-Wire Wire Line
 	6625 3475 6625 3875
 Connection ~ 6625 3475
@@
 Text Notes 7125 6925 0    185  ~ 0
 24V -> 5V_ISO & 3.3V_ISO
+Wire Notes Line
+	5975 4625 8975 4625
+Wire Notes Line
+	8975 4625 8975 2825
+Wire Notes Line
+	8975 2825 5975 2825
+Wire Notes Line
+	5975 2825 5975 4625
+Text Notes 6875 3000 0    79   ~ 0
+5V_ISO -> 3.3V_ISO
+Connection ~ 5700 3475
+Wire Wire Line
+	5700 3475 6625 3475
+Wire Wire Line
+	5050 3475 5700 3475
+Wire Wire Line
+	5050 4075 5700 4075
+Wire Notes Line
+	5475 4625 5475 2800
+Wire Notes Line
+	5475 2800 2875 2800
+Wire Notes Line
+	5475 4625 2875 4625
+Wire Notes Line
+	2875 2800 2875 4625
+Wire Wire Line
+	3350 4075 3350 4300
+Wire Wire Line
+	3350 3925 3350 4075
+Connection ~ 3350 4075
+Wire Wire Line
+	3350 3250 3350 3475
+Text Notes 3450 2975 0    79   ~ 0
+24V_NON_ISO -> 5V_ISO
 $EndSCHEMATC
