File: CarMan KiCAD Schematics/Logic/LogicPower.sch (KiCad schematic (older format))
At the start: 5 parts, among them U4 PYB20-Q24-S5, U7 LT1763CS8-3.3PBF

Commit message: - Removed 5V_NON_ISO -> 3.3V_NON_ISO voltage divider, apparently voltage div put res in // with bi directional transceiver
Parts:
- C13: value 1uF -> 0.01uF
- C5: value 0.1uF -> 1uF
Changed lines of the file:
@@
 U 1 1 5FAF6616
 P 5700 3775
-F 0 "C5" H 5815 3821 50  0000 L CNN
-F 1 "0.1uF" H 5815 3730 50  0000 L CNN
+F 0 "C5" H 5725 3875 50  0000 L CNN
+F 1 "1uF" H 5725 3675 50  0000 L CNN
 F 2 "Capacitor_SMD:C_0805_2012Metric_Pad1.15x1.40mm_HandSolder" H 5738 3625 50  0001 C CNN
 F 3 "~" H 5700 3775 50  0001 C CNN
@@
 P 6175 3825
 F 0 "C13" H 6290 3871 50  0000 L CNN
-F 1 "1uF" H 6290 3780 50  0000 L CNN
+F 1 "0.01uF" H 6290 3780 50  0000 L CNN
 F 2 "Capacitor_SMD:C_0805_2012Metric_Pad1.15x1.40mm_HandSolder" H 6213 3675 50  0001 C CNN
 F 3 "~" H 6175 3825 50  0001 C CNN
@@
 F 1 "LT1763CS8-3.3PBF" H 7450 3025 50  0000 C CNN
 F 2 "CarMan General Footprints:LT1763CS8-3-PBF" H 7450 3775 50  0001 L BNN
-F 3 "Voltage stabiliser; LDO, fixed; 3.3V; 500mA; SO8; SMD" H 7450 3775 50  0001 L BNN
+F 3 "https://www.analog.com/media/en/technical-documentation/data-sheets/1763fh.pdf" H 7450 3775 50  0001 L BNN
 F 4 "Linear Technology/Analog" H 7450 3775 50  0001 L BNN "Field4"
 F 5 "SOIC-8 Linear Technology" H 7450 3775 50  0001 L BNN "Field5"

Commit message: Updated the wiring on the schematic according to the errata update from Marwa
Parts:
- U4: symbol CarMan_KiCAD_Library:PYB20-Q24-S5 -> Logic-rescue:PYB20-Q24-S5-CarMan_KiCAD_Library
Changed lines of the file:
@@
 5V_ISO
 $Comp
-L CarMan_KiCAD_Library:PYB20-Q24-S5 U4
+L Logic-rescue:PYB20-Q24-S5-CarMan_KiCAD_Library U4
 U 1 1 5FAF8405
 P 4450 3775
