File: CarMan KiCAD Schematics/Logic/PiHat.sch (KiCad schematic (older format))
At the start: 11 parts, among them J7 Conn_01x02_Male, U2 ISO1050DUB, U8 MCP2515-xSO, Y1 16MHz

Commit message: Added AIRS monitor signal to Pi, added all Logic Footprints
Parts:
- J7: footprint (none) -> Connector_PinSocket_2.54mm:PinSocket_1x02_P2.54mm_Vertical
Changed lines of the file:
@@
 F 0 "J9" V 2362 1694 50  0000 L CNN
 F 1 "Conn_01x02_Male" V 2453 1694 50  0000 L CNN
-F 2 "" H 2300 1650 50  0001 C CNN
+F 2 "Connector_PinSocket_2.54mm:PinSocket_1x02_P2.54mm_Vertical" H 2300 1650 50  0001 C CNN
 F 3 "~" H 2300 1650 50  0001 C CNN
 	1    2300 1650
@@
 F 1 "16MHz" V 8195 3481 50  0000 L CNN
 F 2 "" H 8150 3350 50  0001 C CNN
-F 3 "~" H 8150 3350 50  0001 C CNN
+F 3 "https://s3.amazonaws.com/snapeda/datasheet/ECS160205PXTR_ECS_International.pdf" H 8150 3350 50  0001 C CNN
 	1    8150 3350
 	0    1    1    0

Commit message: Logic PCB started, Pi 3B footprint fixed
Parts:
- R10, R7: footprint Resistor_SMD:R_0815_2038Metric_Pad1.53x4.00mm_HandSolder -> Resistor_SMD:R_0805_2012Metric_Pad1.15x1.40mm_HandSolder
- Y1: footprint (none) -> CarMan General Footprints:XTAL_ECS-160-20-5PX-TR
Changed lines of the file:
@@
 F 0 "R7" H 2370 2046 50  0000 L CNN
 F 1 "120" V 2300 1950 50  0000 L CNN
-F 2 "Resistor_SMD:R_0815_2038Metric_Pad1.53x4.00mm_HandSolder" V 2230 2000 50  0001 C CNN
+F 2 "Resistor_SMD:R_0805_2012Metric_Pad1.15x1.40mm_HandSolder" V 2230 2000 50  0001 C CNN
 F 3 "~" H 2300 2000 50  0001 C CNN
 	1    2300 2000
@@
 F 0 "R10" V 5850 3700 50  0000 C CNN
 F 1 "4k7" V 5750 3700 50  0000 C CNN
-F 2 "Resistor_SMD:R_0815_2038Metric_Pad1.53x4.00mm_HandSolder" V 5680 3700 50  0001 C CNN
+F 2 "Resistor_SMD:R_0805_2012Metric_Pad1.15x1.40mm_HandSolder" V 5680 3700 50  0001 C CNN
 F 3 "~" H 5750 3700 50  0001 C CNN
 	1    5750 3700
@@
 F 0 "Y1" V 8104 3481 50  0000 L CNN
 F 1 "16MHz" V 8195 3481 50  0000 L CNN
-F 2 "" H 8150 3350 50  0001 C CNN
+F 2 "CarMan General Footprints:XTAL_ECS-160-20-5PX-TR" H 8150 3350 50  0001 C CNN
 F 3 "https://s3.amazonaws.com/snapeda/datasheet/ECS160205PXTR_ECS_International.pdf" H 8150 3350 50  0001 C CNN
 	1    8150 3350
