File: CarMan KiCAD Schematics/Logic/Logic.kicad_pcb (KiCad board)
At the start: 2 copper layers, 168.3 x 153 mm, 69 parts, among them J1 MC Can MC_CAN, J2 IMU IMU PS, J3 IMU IMU, J4 RTC RTC, J5.1 TSI Conn_01x06, J5.2 TSI Conn_01x06, J6 Extra GPIO You're Welcome -Ethan, J7 GLV BOB GLV BOB, J8 Pic32 Prog PIC program, J9 Conn_01x02_Male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

Commit message: Logic updated
Parts:
- removed D4: LED, CarMan General Footprints:VAOL-S8GT4
- removed G***: LOGO, CarMan General Footprints:Laf_College_Logo
- removed R14: 10k, Resistor_SMD:R_0805_2012Metric_Pad1.15x1.40mm_HandSolder
- removed R8: 2k, Resistor_SMD:R_0805_2012Metric_Pad1.15x1.40mm_HandSolder
- removed R9: 3.88k, Resistor_SMD:R_0805_2012Metric_Pad1.15x1.40mm_HandSolder
- removed REF** (x4): MountingHole_2.5mm_Pad, MountingHole:MountingHole_2.5mm_Pad
- added J10: Motor Controller Can Line, Connector_PinSocket_2.54mm:PinSocket_1x04_P2.54mm_Vertical, F.Cu at (55.2, 98.3)
- added U1: MCP9700AT-HTT-Sensor_Temperature-Logic-rescue, Package_TO_SOT_SMD:SOT-23, F.Cu at (59.7, 98.3)
- C13: value 1uF -> 0.01uF
- C5: value 0.1uF -> 1uF
- J1: renamed from J1 MC Can; value MC_CAN -> Motor Controller Can Line
- J2: renamed from J2 IMU
- J3: renamed from J3 IMU; value IMU -> Insulation Monitoring Unit
- J4: renamed from J4 RTC; value RTC -> Real Time Clock
- J5.1: renamed from J5.1 TSI
- J5.2: renamed from J5.2 TSI
- J6: renamed from J6 Extra GPIO
- J7: renamed from J7 GLV BOB
- J8: renamed from J8 Pic32 Prog
- J9: value Conn_01x02_Male -> IMU PS
- moved J9 82.3 mm to (81.0, 98.3), turned to 0 degrees
Connections:
- net /3.3V renamed /3.3V_ISO
- net /GLV_SCL renamed /SCL_TSI_GLV
- net /GLV_SDA renamed /SDA_TSI_GLV
- net /PiHat.sch/PI_SPI_MISO renamed /PI_SPI_MISO
- net /PiHat.sch/PI_SPI_MOSI renamed /PI_SPI_MOSI
- net /PiHat.sch/PI_SPI_SCLK renamed /PI_SPI_SCLK
- net /SCL_iso renamed /SCL_ISO_PI
- net /SDA_iso renamed /SDA_ISO_PI
- net /Safety_Loop_iso renamed /Safety_Loop_ISO
- net Net-(J6-Pad1) renamed /GPIO_16
- net Net-(J6-Pad2) renamed /GPIO_20
- net Net-(J6-Pad3) renamed /GPIO_21
- net Net-(J6-Pad4) renamed /GPIO_26
- net Net-(J6-Pad5) renamed /GPIO_19
- net Net-(J6-Pad6) renamed /GPIO_13
- net Net-(J6-Pad7) renamed /GPIO_5
- net Net-(J6-Pad8) renamed /GPIO_0
- net Net-(U3-Pad41) renamed /PIC_TXD
- net Net-(U3-Pad42) renamed /PIC_RXD
- C1 pad 1: /5V_non_iso -> /GLV_RTN
- C1 pad 2: /24V_rtn -> /5V_NON_ISO
- C10 pad 2: /3.3V_rtn -> /ISO_RTN
- C11 pad 1: /5V -> /5V_ISO
- C11 pad 2: /3.3V_rtn -> /ISO_RTN
- C12 pad 1: /24V_rtn -> /GLV_RTN
- C12 pad 2: /5V_non_iso -> /5V_NON_ISO
- C14 pad 1: /5V -> /ISO_RTN
- C14 pad 2: /3.3V_rtn -> /5V_ISO
- C15 pad 1: /5V -> /5V_ISO
- C15 pad 2: /3.3V_rtn -> /ISO_RTN
- C16 pad 1: /3.3V_rtn -> /ISO_RTN
- C17 pad 1: /3.3V_rtn -> /ISO_RTN
- C18 pad 2: /3.3V_rtn -> /ISO_RTN
- C19 pad 1: /24V_rtn -> /GLV_RTN
- C19 pad 2: /5V_non_iso -> /5V_NON_ISO
- C2 pad 1: Net-(C2-Pad1) -> /ISO_RTN
- C2 pad 2: /3.3V_rtn -> Net-(C2-Pad2)
- C20 pad 2: /24V_rtn -> /GLV_RTN
- C3 pad 2: /24V_rtn -> /GLV_RTN
- C4 pad 1: /3.3V_rtn -> /ISO_RTN
- C5 pad 1: /5V -> /5V_ISO
- C5 pad 2: /3.3V_rtn -> /ISO_RTN
- C6 pad 1: /3.3V_rtn -> /ISO_RTN
- C7 pad 1: /3.3V_rtn -> /ISO_RTN
- C8 pad 1: /3.3V_rtn -> /ISO_RTN
- C9 pad 1: /3.3V_rtn -> /ISO_RTN
- CR1 pad 1: /5V_non_iso -> /5V_NON_ISO
- CR1 pad 2: /24V_rtn -> /GLV_RTN
- CR1 pad 3: /24V_rtn -> /GLV_RTN
- CR1 pad 6: /24V_rtn -> /GLV_RTN
- CR1 pad 7: /24V_rtn -> /GLV_RTN
- D1 pad 1: /3.3V_rtn -> /ISO_RTN
- D2 pad 1: /3.3V_rtn -> /ISO_RTN
- D3 pad 1: /24V_rtn -> /GLV_RTN
- D5 pad 1: /24V_rtn -> /GLV_RTN
- D6 pad 1: /3.3V_rtn -> /ISO_RTN
- J1 pad 3: /3.3V_rtn -> /ISO_RTN
- J2 pad 1: /3.3V_rtn -> /ISO_RTN
- J2 pad 2: /3.3V_rtn -> /ISO_RTN
- J3 pad 2: /3.3V_rtn -> /ISO_RTN
- J4 pad 2: /3.3V_rtn -> /ISO_RTN
- J5.1 pad 3: /3.3V_rtn -> /ISO_RTN
- J7 pad 3: /24V_rtn -> /GLV_RTN
- J8 pad 3: /3.3V_rtn -> /ISO_RTN
- R10 pad 1: /5V -> /5V_ISO
- R12 pad 2: /5V -> /5V_ISO
- R15 pad 1: /5V_non_iso -> /5V_NON_ISO
- R16 pad 1: /5V -> /5V_ISO
- R3 pad 1: Net-(C2-Pad1) -> Net-(C2-Pad2)
- R4 pad 2: Net-(C2-Pad1) -> Net-(C2-Pad2)
- U10 pad 2: /24V_rtn -> /GLV_RTN
- U10 pad 3: /3.3V_rtn -> /ISO_RTN
- U2 pad 1: /5V -> /5V_ISO
- U2 pad 4: /3.3V_rtn -> /ISO_RTN
- U2 pad 5: /24V_rtn -> /GLV_RTN
- U2 pad 8: /5V_non_iso -> /5V_NON_ISO
- U3 pad 20: /3.3V_rtn -> /ISO_RTN
- U3 pad 25: /3.3V_rtn -> /ISO_RTN
- U3 pad 29: Net-(U3-Pad29) -> /V_OUT_TEMP
- U3 pad 34: /3.3V_rtn -> /ISO_RTN
- U3 pad 35: /3.3V_rtn -> /ISO_RTN
- U3 pad 40: /3.3V_rtn -> /ISO_RTN
- U3 pad 55: /3.3V_rtn -> /ISO_RTN
- U3 pad 59: /3.3V_rtn -> /ISO_RTN
- U3 pad 7: /3.3V_rtn -> /ISO_RTN
- U4 pad 1: /24V_rtn -> /GLV_RTN
- U4 pad 3: /5V -> /5V_ISO
- U4 pad 5: /3.3V_rtn -> /ISO_RTN
- U5 pad 1: /5V -> /5V_ISO
- U5 pad 4: /3.3V_rtn -> /ISO_RTN
- U5 pad 5: /24V_rtn -> /GLV_RTN
- U5 pad 8: /5V_non_iso -> /5V_NON_ISO
- U6 pad 14: /3.3V_rtn -> /ISO_RTN
- U6 pad 2: /5V -> /5V_ISO
- U6 pad 20: /3.3V_rtn -> /ISO_RTN
- U6 pad 25: /3.3V_rtn -> /ISO_RTN
- U6 pad 30: /3.3V_rtn -> /ISO_RTN
- U6 pad 34: /3.3V_rtn -> /ISO_RTN
- U6 pad 39: /3.3V_rtn -> /ISO_RTN
- U6 pad 4: /5V -> /5V_ISO
- U6 pad 6: /3.3V_rtn -> /ISO_RTN
- U6 pad 9: /3.3V_rtn -> /ISO_RTN
- U7 pad 3: /3.3V_rtn -> /ISO_RTN
- U7 pad 5: /5V -> /5V_ISO
- U7 pad 6: /3.3V_rtn -> /ISO_RTN
- U7 pad 7: /3.3V_rtn -> /ISO_RTN
- U7 pad 8: /5V -> /5V_ISO
- U8 pad 18: /5V -> /5V_ISO
- U8 pad 9: /3.3V_rtn -> /ISO_RTN
- U9 pad 1: /3.3V_non_iso -> /5V_NON_ISO
- U9 pad 4: /24V_rtn -> /GLV_RTN
- U9 pad 5: /3.3V_rtn -> /ISO_RTN
Routing:
- net /3.3V_rtn: track 770.2 -> 487.5 mm
- net /5V_NON_ISO: track 0.00 -> 181.3 mm, vias 0 -> 4
- net /3.3V_non_iso: track 181.3 -> 0.00 mm, vias 4 -> 0
- net /24V_rtn: track 301.0 -> 157.9 mm
- net /5V: track 551.2 -> 488.3 mm
- net /5V_non_iso: track 203.7 -> 157.3 mm
- net Net-(C2-Pad1): track 5.92 -> 0.00 mm
- net Net-(U3-Pad29): track 3.70 -> 0.00 mm
- net /V_OUT_TEMP: track 0.00 -> 3.70 mm

Commit message: MEGA UPDATE - Changed PC_Ready isolation from logic ISO rtn to GLV_RTN (U27) because it is sent over GPIO - Changed GPIO pins - Added 24V -> 5V TLP stepdown for AMS_FAULT_LED & IMD_FAULT_LED (U29,U31) - Edited U13 & U11 TLPs (RTDS_CTRL & D_LED_CTRL respectively) to be wrt GLV_RTN because signal coming from GPIO - pins on TSI-Logic header match on both boards - lots of other changes, reorganized drive_btn circuit
Parts:
- removed R11: 1k, Resistor_SMD:R_0805_2012Metric_Pad1.15x1.40mm_HandSolder
- removed R12: 2.4k, Resistor_SMD:R_0805_2012Metric_Pad1.15x1.40mm_HandSolder
- removed U10: TLP293, Package_SO:SOIC-4_4.55x2.6mm_P1.27mm
- added C21: 0.1uF, Capacitor_SMD:C_0805_2012Metric_Pad1.15x1.40mm_HandSolder, F.Cu at (68.6, 83.8)
- J5.2: footprint Connector_PinSocket_2.54mm:PinSocket_1x06_P2.54mm_Vertical -> Connector_PinSocket_2.54mm:PinSocket_1x08_P2.54mm_Vertical
Connections:
- J5.1 pad 1: /SCL_TSI_GLV -> /Cooling_CTRL
- J5.1 pad 2: /SDA_TSI_GLV -> /SR_CTRL
- J5.1 pad 3: /ISO_RTN -> /APPS
- J5.1 pad 4: /Safety_Loop -> /CoolTemp
- J5.1 pad 5: /Cooling_CTRL -> /FlowRate
- J5.1 pad 6: /Throttle_SEL -> Net-(J5.1-Pad6)
- J5.2 pad 1: /AMS_Fault -> /SDA_TSI_GLV
- J5.2 pad 2: /SR_CTRL -> /SCL_TSI_GLV
- J5.2 pad 5: /RTDS_CTRL -> /ISO_RTN
- J5.2 pad 6: /PC_ready -> Net-(J5.2-Pad6)
- U3 pad 21: /Throttle_SEL -> Net-(U3-Pad21)
- U3 pad 4: /Safety_Loop_ISO -> Net-(U3-Pad4)
- U3 pad 43: /PC_ready -> Net-(U3-Pad43)
- U3 pad 48: /PC_ready -> Net-(U3-Pad48)
- U3 pad 58: /RTDS_CTRL -> Net-(U3-Pad58)
- U6 pad 16: /Safety_Loop_ISO -> Net-(U6-Pad16)
- U9 pad 1: /5V_NON_ISO -> /3.3V_ISO
- U9 pad 2: /SDA_TSI_GLV -> /SDA_ISO_PI
- U9 pad 3: /SCL_TSI_GLV -> /SCL_ISO_PI
- U9 pad 4: /GLV_RTN -> /ISO_RTN
- U9 pad 5: /ISO_RTN -> /GLV_RTN
- U9 pad 6: /SCL_ISO_PI -> /SCL_TSI_GLV
- U9 pad 7: /SDA_ISO_PI -> /SDA_TSI_GLV
- U9 pad 8: /3.3V_ISO -> /5V_NON_ISO
Routing:
- net /5V_NON_ISO: track 181.3 -> 0.00 mm, vias 4 -> 0
- net /3.3V_ISO: track 413.3 -> 589.0 mm, vias 11 -> 15
- net /Safety_Loop: track 76.1 -> 0.00 mm, vias 4 -> 0
- net /CoolTemp: track 0.00 -> 76.1 mm, vias 0 -> 4
- net /PC_ready: track 148.0 -> 97.8 mm
- net /RTDS_CTRL: track 151.4 -> 126.8 mm
- net /Cooling_CTRL: track 117.6 -> 104.9 mm
- net /SCL_TSI_GLV: track 175.6 -> 163.1 mm
- net /Throttle_SEL: track 133.5 -> 121.6 mm
- net /SDA_TSI_GLV: track 184.7 -> 173.1 mm
- net /SR_CTRL: track 132.3 -> 122.5 mm
- net /Safety_Loop_ISO: track 162.0 -> 156.1 mm
- net /SCL_ISO_PI: track 306.3 -> 303.3 mm
- net /SDA_ISO_PI: track 297.4 -> 295.7 mm

Commit message: routed TSI board
Parts:
- added D4: LED, CarMan General Footprints:VAOL-S8GT4, F.Cu at (47.2, 42.1)
- added D7: LED, CarMan General Footprints:VAOL-S8GT4, F.Cu at (47.2, 45.0)
- added D8: LED, CarMan General Footprints:VAOL-S8GT4, F.Cu at (52.4, 42.1)
- added R11: 10k, Resistor_SMD:R_0805_2012Metric_Pad1.15x1.40mm_HandSolder, F.Cu at (198.6, 142.7)
- added R8: 10k, Resistor_SMD:R_0805_2012Metric_Pad1.15x1.40mm_HandSolder, F.Cu at (193.9, 142.7)
- added R9: 10k, Resistor_SMD:R_0805_2012Metric_Pad1.15x1.40mm_HandSolder, F.Cu at (193.9, 145.7)
- moved J6 17.2 mm to (243.3, 86.9), turned to 0 degrees
- moved U6 1.89 mm to (200.2, 78.7)
Connections:
- CR1 pad 4: Net-(CR1-Pad4) -> (no net)
- CR1 pad 5: Net-(CR1-Pad5) -> (no net)
- J1 pad 4: Net-(J1-Pad4) -> (no net)
- J5.1 pad 6: Net-(J5.1-Pad6) -> /ADC_RTN
- J5.2 pad 6: Net-(J5.2-Pad6) -> /3.3V_ISO
- J8 pad 6: Net-(J8-Pad6) -> (no net)
- U3 pad 1: Net-(U3-Pad1) -> (no net)
- U3 pad 10: Net-(U3-Pad10) -> (no net)
- U3 pad 11: Net-(U3-Pad11) -> /APPS
- U3 pad 12: Net-(U3-Pad12) -> (no net)
- U3 pad 13: Net-(U3-Pad13) -> (no net)
- U3 pad 14: Net-(U3-Pad14) -> (no net)
- U3 pad 17: Net-(U3-Pad17) -> /CoolTemp
- U3 pad 18: Net-(U3-Pad18) -> /FlowRate
- U3 pad 2: Net-(U3-Pad2) -> (no net)
- U3 pad 21: Net-(U3-Pad21) -> (no net)
- U3 pad 22: Net-(U3-Pad22) -> (no net)
- U3 pad 23: Net-(U3-Pad23) -> /ADC_RTN
- U3 pad 24: Net-(U3-Pad24) -> /ADC_RTN
- U3 pad 27: Net-(U3-Pad27) -> (no net)
- U3 pad 28: Net-(U3-Pad28) -> (no net)
- U3 pad 30: Net-(U3-Pad30) -> (no net)
- U3 pad 31: Net-(U3-Pad31) -> (no net)
- U3 pad 32: Net-(U3-Pad32) -> (no net)
- U3 pad 33: Net-(U3-Pad33) -> (no net)
- U3 pad 36: Net-(U3-Pad36) -> (no net)
- U3 pad 37: Net-(U3-Pad37) -> (no net)
- U3 pad 38: Net-(U3-Pad38) -> (no net)
- U3 pad 4: Net-(U3-Pad4) -> (no net)
- U3 pad 43: Net-(U3-Pad43) -> (no net)
- U3 pad 44: Net-(U3-Pad44) -> (no net)
- U3 pad 45: Net-(U3-Pad45) -> (no net)
- U3 pad 46: Net-(U3-Pad46) -> /STATE_OUT_1
- U3 pad 47: Net-(U3-Pad47) -> (no net)
- U3 pad 48: Net-(U3-Pad48) -> (no net)
- U3 pad 49: Net-(U3-Pad49) -> /STATE_OUT_2
- U3 pad 50: Net-(U3-Pad50) -> /STATE_OUT_3
- U3 pad 51: Net-(U3-Pad51) -> (no net)
- U3 pad 52: Net-(U3-Pad52) -> (no net)
- U3 pad 53: Net-(U3-Pad53) -> (no net)
- U3 pad 56: Net-(U3-Pad56) -> (no net)
- U3 pad 57: Net-(U3-Pad57) -> (no net)
- U3 pad 58: Net-(U3-Pad58) -> (no net)
- U3 pad 61: Net-(U3-Pad61) -> (no net)
- U3 pad 62: Net-(U3-Pad62) -> (no net)
- U3 pad 63: Net-(U3-Pad63) -> (no net)
- U3 pad 64: Net-(U3-Pad64) -> (no net)
- U4 pad 4: Net-(U4-Pad4) -> (no net)
- U4 pad 6: Net-(U4-Pad6) -> (no net)
- U6 pad 1: Net-(U6-Pad1) -> (no net)
- U6 pad 10: Net-(U6-Pad10) -> (no net)
- U6 pad 11: Net-(U6-Pad11) -> (no net)
- U6 pad 12: Net-(U6-Pad12) -> (no net)
- U6 pad 13: Net-(U6-Pad13) -> (no net)
- U6 pad 15: Net-(U6-Pad15) -> (no net)
- U6 pad 16: Net-(U6-Pad16) -> (no net)
- U6 pad 17: Net-(U6-Pad17) -> (no net)
- U6 pad 18: Net-(U6-Pad18) -> (no net)
- U6 pad 26: Net-(U6-Pad26) -> (no net)
- U6 pad 28: Net-(U6-Pad28) -> (no net)
- U6 pad 32: Net-(U6-Pad32) -> (no net)
- U6 pad 7: Net-(U6-Pad7) -> (no net)
- U6 pad 8: Net-(U6-Pad8) -> (no net)
- U8 pad 10: Net-(U8-Pad10) -> (no net)
- U8 pad 11: Net-(U8-Pad11) -> (no net)
- U8 pad 3: Net-(U8-Pad3) -> (no net)
- U8 pad 4: Net-(U8-Pad4) -> (no net)
- U8 pad 5: Net-(U8-Pad5) -> (no net)
- U8 pad 6: Net-(U8-Pad6) -> (no net)
Routing:
- net /3.3V_ISO: track 589.0 -> 0.00 mm, vias 15 -> 0
- net /5V: track 488.3 -> 0.00 mm, vias 13 -> 0
- net /3.3V_rtn: track 487.5 -> 0.00 mm, vias 34 -> 0
- net /SCL_ISO_PI: track 303.3 -> 0.00 mm, vias 13 -> 0
- net /SDA_ISO_PI: track 295.7 -> 0.00 mm, vias 13 -> 0
- net /BP_CAN+: track 262.9 -> 0.00 mm, vias 9 -> 0
- net /BP_CAN-: track 260.9 -> 0.00 mm, vias 7 -> 0
- net /SDA_TSI_GLV: track 173.1 -> 0.00 mm, vias 4 -> 0
- net /SCL_TSI_GLV: track 163.1 -> 0.00 mm, vias 5 -> 0
- net /24V_rtn: track 157.9 -> 0.00 mm, vias 9 -> 0
- net /5V_non_iso: track 157.3 -> 0.00 mm, vias 6 -> 0
- net /Safety_Loop_ISO: track 156.1 -> 0.00 mm, vias 7 -> 0
- net /24V: track 145.1 -> 0.00 mm, vias 2 -> 0
- net /PI_SPI_CEO: track 142.5 -> 0.00 mm, vias 3 -> 0
- net /GPIO25: track 134.5 -> 0.00 mm, vias 3 -> 0
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Other:
- board text added: "Electrical and Computer Engineering Ethan Miller and Zachary (Big Zack) Martin Logic V1.1 2/9/21"
- board text removed: "Electrical and Computer Engineering Ethan Miller and Zachary Martin Logic V1.0 2/9/21"

Commit message: Balls balls balls
Parts:
- removed J5.1: Conn_01x06, Connector_PinSocket_2.54mm:PinSocket_1x06_P2.54mm_Vertical
- removed J5.2: Conn_01x06, Connector_PinSocket_2.54mm:PinSocket_1x08_P2.54mm_Vertical
- removed J6: You're Welcome -Ethan, Connector_PinSocket_2.54mm:PinSocket_1x08_P2.54mm_Vertical
- added J5: Conn_02x06_Odd_Even, Connector_PinSocket_2.54mm:PinSocket_2x06_P2.54mm_Vertical, F.Cu at (182.9, 94.2)
- C10, C4, C6, C7, C8, L1: moved to F.Cu
- moved R11 167.1 mm to (64.3, 43.4)
- moved R8 167.1 mm to (59.5, 43.4)
- moved R9 167.1 mm to (59.5, 46.3)
- moved R6 158.7 mm to (57.4, 65.7)
- moved D2 158.7 mm to (60.6, 65.6)
- moved R5 152.8 mm to (60.6, 57.7)
- moved D1 152.3 mm to (56.1, 57.7)
- moved U1 142.3 mm to (201.9, 97.5), turned to 90 degrees
- moved D3 136.8 mm to (47.6, 49.5)
- moved R13 136.8 mm to (42.5, 49.5)
- moved R15 102.7 mm to (46.0, 59.9)
- moved D5 102.7 mm to (50.4, 60.1)
- moved C19 96.8 mm to (218.2, 90.4), turned to 180 degrees
- moved CR1 92.1 mm to (218.9, 85.6), turned to 90 degrees
- moved J8 91.7 mm to (224.8, 94.7), turned to 180 degrees
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Connections:
- CR1 pad 4: (no net) -> Net-(CR1-Pad4)
- CR1 pad 5: (no net) -> Net-(CR1-Pad5)
- J1 pad 4: (no net) -> Net-(J1-Pad4)
- J8 pad 6: (no net) -> Net-(J8-Pad6)
- U3 pad 1: (no net) -> Net-(U3-Pad1)
- U3 pad 10: (no net) -> Net-(U3-Pad10)
- U3 pad 12: (no net) -> Net-(U3-Pad12)
- U3 pad 13: (no net) -> Net-(U3-Pad13)
- U3 pad 14: (no net) -> Net-(U3-Pad14)
- U3 pad 2: (no net) -> Net-(U3-Pad2)
- U3 pad 21: (no net) -> Net-(U3-Pad21)
- U3 pad 22: (no net) -> Net-(U3-Pad22)
- U3 pad 27: (no net) -> Net-(U3-Pad27)
- U3 pad 28: (no net) -> Net-(U3-Pad28)
- U3 pad 30: (no net) -> Net-(U3-Pad30)
- U3 pad 31: (no net) -> Net-(U3-Pad31)
- U3 pad 32: (no net) -> Net-(U3-Pad32)
- U3 pad 33: (no net) -> Net-(U3-Pad33)
- U3 pad 36: (no net) -> Net-(U3-Pad36)
- U3 pad 37: (no net) -> Net-(U3-Pad37)
- U3 pad 38: (no net) -> Net-(U3-Pad38)
- U3 pad 4: (no net) -> Net-(U3-Pad4)
- U3 pad 43: (no net) -> Net-(U3-Pad43)
- U3 pad 44: (no net) -> Net-(U3-Pad44)
- U3 pad 45: (no net) -> Net-(U3-Pad45)
- U3 pad 47: (no net) -> Net-(U3-Pad47)
- U3 pad 48: (no net) -> Net-(U3-Pad48)
- U3 pad 51: (no net) -> Net-(U3-Pad51)
- U3 pad 52: (no net) -> Net-(U3-Pad52)
- U3 pad 53: (no net) -> Net-(U3-Pad53)
- U3 pad 56: (no net) -> Net-(U3-Pad56)
- U3 pad 57: (no net) -> Net-(U3-Pad57)
- U3 pad 58: (no net) -> Net-(U3-Pad58)
- U3 pad 61: (no net) -> Net-(U3-Pad61)
- U3 pad 62: (no net) -> Net-(U3-Pad62)
- U3 pad 63: (no net) -> Net-(U3-Pad63)
- U3 pad 64: (no net) -> Net-(U3-Pad64)
- U4 pad 4: (no net) -> Net-(U4-Pad4)
- U4 pad 6: (no net) -> Net-(U4-Pad6)
- U6 pad 1: (no net) -> Net-(U6-Pad1)
- U6 pad 10: (no net) -> Net-(U6-Pad10)
- U6 pad 11: (no net) -> Net-(U6-Pad11)
- U6 pad 12: (no net) -> Net-(U6-Pad12)
- U6 pad 13: (no net) -> Net-(U6-Pad13)
- U6 pad 15: (no net) -> Net-(U6-Pad15)
- U6 pad 16: (no net) -> Net-(U6-Pad16)
- U6 pad 17: (no net) -> Net-(U6-Pad17)
- U6 pad 18: (no net) -> Net-(U6-Pad18)
- U6 pad 26: (no net) -> Net-(U6-Pad26)
- U6 pad 28: (no net) -> Net-(U6-Pad28)
- U6 pad 32: (no net) -> Net-(U6-Pad32)
- U6 pad 7: (no net) -> Net-(U6-Pad7)
- U6 pad 8: (no net) -> Net-(U6-Pad8)
- U8 pad 10: (no net) -> Net-(U8-Pad10)
- U8 pad 11: (no net) -> Net-(U8-Pad11)
- U8 pad 3: (no net) -> Net-(U8-Pad3)
- U8 pad 4: (no net) -> Net-(U8-Pad4)
- U8 pad 5: (no net) -> Net-(U8-Pad5)
- U8 pad 6: (no net) -> Net-(U8-Pad6)
Routing:
- net /ISO_RTN: track 0.00 -> 9.25 mm
- net /5V_ISO: track 0.00 -> 7.79 mm
- net /PIC_TXD: track 0.00 -> 6.69 mm
- net /PIC_RXD: track 0.00 -> 6.61 mm
- net /GLV_RTN: track 0.00 -> 4.11 mm
- net Net-(C2-Pad2): track 0.00 -> 4.06 mm
- net /3.3V_ISO: track 0.00 -> 3.89 mm
- net /5V_NON_ISO: track 0.00 -> 3.64 mm
- added copper zone on B.Cu, net /ISO_RTN

Commit message: logic & TSI lay out
Parts:
- C3: moved to F.Cu
- J4, J7, J8, U4: moved to B.Cu
- moved C3 17.4 mm to (195.8, 62.2)
- moved U4 9.27 mm to (196.1, 75.2), turned to 270 degrees
- moved J7 3.81 mm to (224.3, 75.4), turned to 90 degrees
- moved J4 1.05 mm to (225.0, 98.0), turned to 180 degrees
- moved J8 0.80 mm to (225.0, 94.0), turned to 0 degrees

Commit message: TSI Logic Changes
Parts:
- removed J2: IMU PS, Connector_PinHeader_2.54mm:PinHeader_1x02_P2.54mm_Vertical
- removed J3: Insulation Monitoring Unit, Connector_PinHeader_2.54mm:PinHeader_1x05_P2.54mm_Vertical
- added U10: BNO_055, CarMan General Footprints:BNO_055, B.Cu at (182.4, 97.5)
- C1, J1, J5: moved to B.Cu
- C5: moved to F.Cu
- moved C21 147.1 mm to (215.1, 71.4), turned to 270 degrees
- moved Y1 86.1 mm to (206.8, 86.1), turned to 90 degrees
- moved C17 79.0 mm to (202.9, 82.3), turned to 90 degrees
- moved C16 78.8 mm to (202.9, 90.2), turned to 270 degrees
- moved C5 76.7 mm to (200.7, 69.6)
- moved R7 72.3 mm to (85.3, 97.8)
- moved J1 65.4 mm to (224.3, 64.0), turned to 90 degrees
- moved C14 59.4 mm to (185.4, 100.8)
- moved U2 57.6 mm to (192.8, 100.1)
- moved U7 53.5 mm to (194.8, 70.2), turned to 0 degrees
- moved C1 52.7 mm to (200.2, 99.1), turned to 90 degrees
- moved U8 52.3 mm to (194.6, 87.2), turned to 180 degrees
- moved C18 52.3 mm to (204.5, 71.1)
- moved C13 43.8 mm to (189.7, 70.2), turned to 270 degrees
- moved R10 35.7 mm to (185.9, 91.1), turned to 0 degrees
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Routing:
- net /SDA_ISO_PI: track 0.00 -> 66.0 mm
- net /SCL_ISO_PI: track 0.00 -> 57.1 mm
- net /ISO_RTN: track 9.25 -> 54.8 mm
- net /24V: track 0.00 -> 38.1 mm
- net /GLV_RTN: track 4.11 -> 39.5 mm, vias 0 -> 1
- net /PGED: track 0.00 -> 21.3 mm
- net /PGEC: track 0.00 -> 20.5 mm
- net /PI_SPI_CEO: track 0.00 -> 17.8 mm
- net /GPIO25: track 0.00 -> 17.5 mm
- net /PI_SPI_MOSI: track 0.00 -> 16.8 mm, vias 0 -> 1
- net /PI_SPI_MISO: track 0.00 -> 16.0 mm
- net /PI_SPI_SCLK: track 0.00 -> 14.5 mm, vias 0 -> 1
- net /5V_ISO: track 7.79 -> 22.1 mm
- net /3.3V_ISO: track 3.89 -> 17.6 mm
- net /5V_NON_ISO: track 3.64 -> 15.2 mm, vias 0 -> 1
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