File: CarMan KiCAD Schematics/TSI/TSI_Rev.5/Fault_Logic_And_Timing_Circuit.sch (KiCad schematic (older format))
At the start: 26 parts

Commit message: fixed some bullshit
Parts:
- gave numbers to parts that had none: 22
Changed lines of the file:
@@
 AMS_Fault
 $Comp
-L 74xGxx:74LVC1GU04DRL U?
+L 74xGxx:74LVC1GU04DRL U38
 U 1 1 5F9E6A96
 P 5550 3300
-F 0 "U?" H 5600 3300 50  0000 L CNN
+F 0 "U38" H 5600 3300 50  0000 L CNN
 F 1 "74LVC1GU04DRL" H 5600 3150 50  0000 L CNN
 F 2 "Package_TO_SOT_SMD:SOT-553" H 5550 3050 50  0001 C CNN
@@
 	6250 3100 6400 3100
 $Comp
-L 74xGxx:74AHC1G08 U?
+L 74xGxx:74AHC1G08 U44
 U 1 1 5FA0F008
 P 7500 3150
-F 0 "U?" H 7475 3417 50  0000 C CNN
+F 0 "U44" H 7475 3417 50  0000 C CNN
 F 1 "74AHC1G08" H 7475 3326 50  0000 C CNN
 F 2 "" H 7500 3150 50  0001 C CNN
@@
 	4650 3150 4950 3150
 $Comp
-L 74xx:74HC02 U?
+L 74xx:74HC02 U16
 U 1 1 5FA13134
 P 8150 3250
-F 0 "U?" H 8150 3250 50  0000 C CNN
+F 0 "U16" H 8150 3250 50  0000 C CNN
 F 1 "74HC02" H 8150 3050 50  0000 C CNN
 F 2 "" H 8150 3250 50  0001 C CNN
@@
 	8600 3250 8450 3250
 $Comp
-L Device:Q_PMOS_SDG Q?
+L Device:Q_PMOS_SDG Q9
 U 1 1 5FA4FE0D
 P 8800 3250
-F 0 "Q?" H 9005 3204 50  0000 L CNN
+F 0 "Q9" H 9005 3204 50  0000 L CNN
 F 1 "Q_PMOS_SDG" H 9005 3295 50  0000 L CNN
 F 2 "" H 9000 3350 50  0001 C CNN
@@
 24V
 $Comp
-L 74xGxx:74LVC1GU04DRL U?
+L 74xGxx:74LVC1GU04DRL U39
 U 1 1 5FA64C59
 P 5550 4800
-F 0 "U?" H 5600 4800 50  0000 L CNN
+F 0 "U39" H 5600 4800 50  0000 L CNN
 F 1 "74LVC1GU04DRL" H 5600 4650 50  0000 L CNN
 F 2 "Package_TO_SOT_SMD:SOT-553" H 5550 4550 50  0001 C CNN
@@
 RESET_IMD
 $Comp
-L 74xGxx:74AHC1G08 U?
+L 74xGxx:74AHC1G08 U43
 U 1 1 5FA64C68
 P 7400 4650
-F 0 "U?" H 7350 4650 50  0000 C CNN
+F 0 "U43" H 7350 4650 50  0000 C CNN
 F 1 "74AHC1G08" H 7375 4826 50  0000 C CNN
 F 2 "" H 7400 4650 50  0001 C CNN
@@
 	8500 4750 8350 4750
 $Comp
-L Device:Q_PMOS_SDG Q?
+L Device:Q_PMOS_SDG Q8
 U 1 1 5FA64C8B
 P 8700 4750
-F 0 "Q?" H 8905 4704 50  0000 L CNN
+F 0 "Q8" H 8905 4704 50  0000 L CNN
 F 1 "Q_PMOS_SDG" H 8905 4795 50  0000 L CNN
 F 2 "" H 8900 4850 50  0001 C CNN
@@
 	4850 3550 4850 4400
 $Comp
-L Device:R R?
+L Device:R R43
 U 1 1 5FA65EAA
 P 8800 5500
-F 0 "R?" H 8870 5546 50  0000 L CNN
+F 0 "R43" H 8870 5546 50  0000 L CNN
 F 1 "R" H 8870 5455 50  0000 L CNN
 F 2 "" V 8730 5500 50  0001 C CNN
@@
 Safety_Loop
 $Comp
-L CarMan_KiCAD_Library:MC14043BDR2G U?
+L CarMan_KiCAD_Library:MC14043BDR2G U36
 U 1 1 5F9E8EA1
 P 3850 4850
-F 0 "U?" H 4150 7100 50  0000 C CNN
+F 0 "U36" H 4150 7100 50  0000 C CNN
 F 1 "MC14043BDR2G" H 4150 4800 50  0000 C CNN
 F 2 "SO16" H 3850 4850 50  0001 L BNN
@@
 GLV_RTN
 $Comp
-L 74xx:74HC02 U?
+L 74xx:74HC02 U16
 U 2 1 5FA7BC19
 P 6700 3200
-F 0 "U?" H 6700 3525 50  0000 C CNN
+F 0 "U16" H 6700 3525 50  0000 C CNN
 F 1 "74HC02" H 6700 3434 50  0000 C CNN
 F 2 "" H 6700 3200 50  0001 C CNN
@@
 $EndComp
 $Comp
-L 74xx:74HC02 U?
+L 74xx:74HC02 U16
 U 3 1 5FA80025
 P 8050 4750
-F 0 "U?" H 8050 4750 50  0000 C CNN
+F 0 "U16" H 8050 4750 50  0000 C CNN
 F 1 "74HC02" H 8200 4550 50  0000 C CNN
 F 2 "" H 8050 4750 50  0001 C CNN
@@
 $EndComp
 $Comp
-L 74xx:74HC02 U?
+L 74xx:74HC02 U16
 U 4 1 5FA8384A
 P 6600 4700
-F 0 "U?" H 6600 4700 50  0000 C CNN
+F 0 "U16" H 6600 4700 50  0000 C CNN
 F 1 "74HC02" H 6750 4500 50  0000 C CNN
 F 2 "" H 6600 4700 50  0001 C CNN
@@
 $EndComp
 $Comp
-L 74xx:74HC02 U?
+L 74xx:74HC02 U16
 U 5 1 5FA92438
 P 1450 1100
-F 0 "U?" V 1200 1100 50  0000 C CNN
+F 0 "U16" V 1200 1100 50  0000 C CNN
 F 1 "74HC02" V 1700 1100 50  0000 C CNN
 F 2 "" H 1450 1100 50  0001 C CNN
@@
 IMD_FAULT_LED
 $Comp
-L CarMan_KiCAD_Library:SN74LV1T34DCKR U?
+L CarMan_KiCAD_Library:SN74LV1T34DCKR U35
 U 1 1 5FAAC151
 P 3500 6650
-F 0 "U?" H 3500 7300 60  0000 C CNN
+F 0 "U35" H 3500 7300 60  0000 C CNN
 F 1 "SN74LV1T34DCKR" H 3550 6000 60  0000 C CNN
 F 2 "DCK0005A_N" H 3500 6590 60  0001 C CNN
@@
 5V
 $Comp
-L CarMan_KiCAD_Library:74HC00 U?
+L CarMan_KiCAD_Library:74HC00 U19
 U 5 1 5FAC39DC
 P 1450 1750
-F 0 "U?" V 1200 1750 50  0000 C CNN
+F 0 "U19" V 1200 1750 50  0000 C CNN
 F 1 "74HC00" V 1700 1750 50  0000 C CNN
 F 2 "" H 1450 1750 50  0001 C CNN
@@
 	9550 500  9550 1750
 $Comp
-L Device:R R?
+L Device:R R19
 U 1 1 5FB88DEA
 P 4700 900
-F 0 "R?" H 4770 946 50  0000 L CNN
+F 0 "R19" H 4770 946 50  0000 L CNN
 F 1 "1.3M" V 4700 830 50  0000 L CNN
 F 2 "" V 4630 900 50  0001 C CNN
@@
 $EndComp
 $Comp
-L Device:R R?
+L Device:R R36
 U 1 1 5FB89B59
 P 5250 900
-F 0 "R?" H 5320 946 50  0000 L CNN
+F 0 "R36" H 5320 946 50  0000 L CNN
 F 1 "1M" V 5250 850 50  0000 L CNN
 F 2 "" V 5180 900 50  0001 C CNN
@@
 $EndComp
 $Comp
-L pspice:CAP C?
+L pspice:CAP C10
 U 1 1 5FB8A940
 P 4700 1700
-F 0 "C?" H 4750 1800 50  0000 L CNN
+F 0 "C10" H 4750 1800 50  0000 L CNN
 F 1 "200u" H 4750 1600 50  0000 L CNN
 F 2 "" H 4700 1700 50  0001 C CNN
@@
 GLV_RTN
 $Comp
-L Device:Q_NMOS_DSG Q?
+L Device:Q_NMOS_DSG Q6
 U 1 1 5FB94191
 P 5150 1400
-F 0 "Q?" H 5354 1446 50  0000 L CNN
+F 0 "Q6" H 5354 1446 50  0000 L CNN
 F 1 "Q_NMOS_DSG" H 5354 1355 50  0000 L CNN
 F 2 "" H 5350 1500 50  0001 C CNN
@@
 RESET_AMS
 $Comp
-L Device:R R?
+L Device:R R37
 U 1 1 5FBB8BC8
 P 6350 950
-F 0 "R?" H 6420 996 50  0000 L CNN
+F 0 "R37" H 6420 996 50  0000 L CNN
 F 1 "1.3M" V 6350 869 50  0000 L CNN
 F 2 "" V 6280 950 50  0001 C CNN
@@
 $EndComp
 $Comp
-L Device:R R?
+L Device:R R42
 U 1 1 5FBB8BCE
 P 6900 950
-F 0 "R?" H 6970 996 50  0000 L CNN
+F 0 "R42" H 6970 996 50  0000 L CNN
 F 1 "1M" V 6900 900 50  0000 L CNN
 F 2 "" V 6830 950 50  0001 C CNN
@@
 $EndComp
 $Comp
-L pspice:CAP C?
+L pspice:CAP C11
 U 1 1 5FBB8BD4
 P 6350 1750
-F 0 "C?" H 6400 1850 50  0000 L CNN
+F 0 "C11" H 6400 1850 50  0000 L CNN
 F 1 "200u" H 6400 1650 50  0000 L CNN
 F 2 "" H 6350 1750 50  0001 C CNN
@@
 GLV_RTN
 $Comp
-L Device:Q_NMOS_DSG Q?
+L Device:Q_NMOS_DSG Q7
 U 1 1 5FBB8BE4
 P 6800 1450
-F 0 "Q?" H 7004 1496 50  0000 L CNN
+F 0 "Q7" H 7004 1496 50  0000 L CNN
 F 1 "Q_NMOS_DSG" H 7004 1405 50  0000 L CNN
 F 2 "" H 7000 1550 50  0001 C CNN
@@
 AMS_IMD
 $Comp
-L Device:R R?
+L Device:R R44
 U 1 1 5F9E6F79
 P 8900 3600
-F 0 "R?" H 8970 3646 50  0000 L CNN
+F 0 "R44" H 8970 3646 50  0000 L CNN
 F 1 "R" H 8970 3555 50  0000 L CNN
 F 2 "" V 8830 3600 50  0001 C CNN
@@
 FAULT LOGIC \n& TIMING CIRCUIT
 $Comp
-L Device:R R?
+L Device:R R18
 U 1 1 5FB5A4D9
 P 2100 5200
-F 0 "R?" H 2170 5246 50  0000 L CNN
+F 0 "R18" H 2170 5246 50  0000 L CNN
 F 1 "2.9k" V 2100 5119 50  0000 L CNN
 F 2 "" V 2030 5200 50  0001 C CNN
@@
 $EndComp
 $Comp
-L Device:R R?
+L Device:R R17
 U 1 1 5FB59651
 P 1900 4900
-F 0 "R?" H 1970 4946 50  0000 L CNN
+F 0 "R17" H 1970 4946 50  0000 L CNN
 F 1 "10k" V 1900 4800 50  0000 L CNN
 F 2 "" V 1830 4900 50  0001 C CNN
