File: CarMan KiCAD Schematics/TSI/TSI_Rev.5/StatusLights_Cockpit.sch (KiCad schematic (older format))
At the start: 20 parts, among them Q3 ZVP1320F, U1 RDE03110S12, U11 TLP293, U13 TLP293, U27 TLP293

Commit message: TSI Footprints - Res, Caps, Inductor all 0805s - Mounting Holes
Parts:
- C17, C6: footprint (none) -> Capacitor_SMD:C_0805_2012Metric_Pad1.15x1.40mm_HandSolder
- R110, R12, R15, R25, R3, R68, R74, R97: footprint (none) -> Resistor_SMD:R_0805_2012Metric_Pad1.15x1.40mm_HandSolder
Changed lines of the file:
@@
 F 0 "R3" H 10100 1300 50  0000 C CNN
 F 1 "330" V 10200 1300 50  0000 C CNN
-F 2 "" V 10130 1300 50  0001 C CNN
+F 2 "Resistor_SMD:R_0805_2012Metric_Pad1.15x1.40mm_HandSolder" V 10130 1300 50  0001 C CNN
 F 3 "~" H 10200 1300 50  0001 C CNN
 	1    10200 1300
@@
 F 0 "R12" V 3800 1300 50  0000 C CNN
 F 1 "300" V 3900 1300 50  0000 C CNN
-F 2 "" V 3830 1300 50  0001 C CNN
+F 2 "Resistor_SMD:R_0805_2012Metric_Pad1.15x1.40mm_HandSolder" V 3830 1300 50  0001 C CNN
 F 3 "~" H 3900 1300 50  0001 C CNN
 	1    3900 1300
@@
 F 0 "R110" V 5300 1300 50  0000 C CNN
 F 1 "10K" V 5400 1300 50  0000 C CNN
-F 2 "" V 5330 1300 50  0001 C CNN
+F 2 "Resistor_SMD:R_0805_2012Metric_Pad1.15x1.40mm_HandSolder" V 5330 1300 50  0001 C CNN
 F 3 "~" H 5400 1300 50  0001 C CNN
 	1    5400 1300
@@
 F 0 "R74" H 5970 1046 50  0000 L CNN
 F 1 "1M" V 5900 950 50  0000 L CNN
-F 2 "" V 5830 1000 50  0001 C CNN
+F 2 "Resistor_SMD:R_0805_2012Metric_Pad1.15x1.40mm_HandSolder" V 5830 1000 50  0001 C CNN
 F 3 "~" H 5900 1000 50  0001 C CNN
 	1    5900 1000
@@
 F 0 "R15" V 3800 2000 50  0000 C CNN
 F 1 "300" V 3900 2000 50  0000 C CNN
-F 2 "" V 3830 2000 50  0001 C CNN
+F 2 "Resistor_SMD:R_0805_2012Metric_Pad1.15x1.40mm_HandSolder" V 3830 2000 50  0001 C CNN
 F 3 "~" H 3900 2000 50  0001 C CNN
 	1    3900 2000
@@
 F 0 "R25" V 3800 2800 50  0000 C CNN
 F 1 "300" V 3900 2800 50  0000 C CNN
-F 2 "" V 3830 2800 50  0001 C CNN
+F 2 "Resistor_SMD:R_0805_2012Metric_Pad1.15x1.40mm_HandSolder" V 3830 2800 50  0001 C CNN
 F 3 "~" H 3900 2800 50  0001 C CNN
 	1    3900 2800
@@
 F 0 "C17" H 4578 6746 50  0000 L CNN
 F 1 "4.7u" H 4578 6655 50  0000 L CNN
-F 2 "" H 4400 6700 50  0001 C CNN
+F 2 "Capacitor_SMD:C_0805_2012Metric_Pad1.15x1.40mm_HandSolder" H 4400 6700 50  0001 C CNN
 F 3 "~" H 4400 6700 50  0001 C CNN
 	1    4400 6700
@@
 F 0 "R68" V 7650 5000 50  0000 C CNN
 F 1 "10K" V 7750 5000 50  0000 C CNN
-F 2 "" V 7680 5000 50  0001 C CNN
+F 2 "Resistor_SMD:R_0805_2012Metric_Pad1.15x1.40mm_HandSolder" V 7680 5000 50  0001 C CNN
 F 3 "~" H 7750 5000 50  0001 C CNN
 	1    7750 5000
@@
 F 0 "R97" V 7650 5350 50  0000 C CNN
 F 1 "10K" V 7750 5350 50  0000 C CNN
-F 2 "" V 7680 5350 50  0001 C CNN
+F 2 "Resistor_SMD:R_0805_2012Metric_Pad1.15x1.40mm_HandSolder" V 7680 5350 50  0001 C CNN
 F 3 "~" H 7750 5350 50  0001 C CNN
 	1    7750 5350
@@
 F 0 "C6" H 8100 5800 50  0000 L CNN
 F 1 "0.1u" H 8100 5600 50  0000 L CNN
-F 2 "" H 8050 5700 50  0001 C CNN
+F 2 "Capacitor_SMD:C_0805_2012Metric_Pad1.15x1.40mm_HandSolder" H 8050 5700 50  0001 C CNN
 F 3 "~" H 8050 5700 50  0001 C CNN
 	1    8050 5700

Commit message: TSI Footprinting (~80%)  - Added Molex  - Added Current Sensor
Parts:
- TSAL_RTN1: footprint (none) -> TestPoint:TestPoint_Pad_D3.0mm
Changed lines of the file:
@@
 F 0 "TSAL_RTN1" H 4142 7276 50  0000 R CNN
 F 1 "TSAL_RTN" H 4142 7367 50  0000 R CNN
-F 2 "" H 4400 7250 50  0001 C CNN
+F 2 "TestPoint:TestPoint_Pad_D3.0mm" H 4400 7250 50  0001 C CNN
 F 3 "~" H 4400 7250 50  0001 C CNN
 	1    4200 7250
