File: CarMan KiCAD Schematics/TSI/TSI_Rev.5/TSI_Rev.5.sch (KiCad schematic (older format))
At the start: 29 parts, among them J1 J1, J10 J10, J11 J11, J12 J12, J13.1 Conn_01x06, J13.2 Conn_01x06, J14 J14, J15 J15, J16 J16, J17 J17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

Commit message: TSI (~98.5%)
Connections:
- net SL1_In: now also J19.1 (Pin_1); no longer J19.2 (Pin_2)
- net TSAL: now also J19.2 (Pin_2)
- no-connect marks 10 -> 9
Changed lines of the file:
@@
 Text Label 4700 2800 0    50   ~ 0
 SCL
-Text Label 1550 2800 0    50   ~ 0
+Text Label 1550 2700 0    50   ~ 0
 SL1_In
 Text Label 4700 2700 0    50   ~ 0
@@
 	1550 2900 2050 2900
 Wire Wire Line
-	1550 2800 2050 2800
+	1550 2700 2050 2700
 Text Label 1550 3000 0    50   ~ 0
 Throttle_SEL
@@
 Text Notes 1600 3300 0    50   ~ 0
 Left Side\nTesting Connector\n\n
-$Comp
-L Connector_Generic:Conn_01x04 J19
-U 1 1 5FE0EFE1
-P 2250 2800
-F 0 "J19" H 2200 3000 50  0000 L CNN
-F 1 "J19" H 2200 3100 50  0001 L CNN
-F 2 "Connector_PinSocket_2.54mm:PinSocket_1x04_P2.54mm_Vertical" H 2250 2800 50  0001 C CNN
-F 3 "~" H 2250 2800 50  0001 C CNN
-	1    2250 2800
-	1    0    0    -1
-$EndComp
 Text Label 11100 3000 2    50   ~ 0
 24V
@@
 Wire Wire Line
 	3100 3000 2500 3000
-NoConn ~ 2050 2700
+$Comp
+L Connector_Generic:Conn_01x04 J19
+U 1 1 5FE0EFE1
+P 2250 2800
+F 0 "J19" H 2200 3000 50  0000 L CNN
+F 1 "J19" H 2200 3100 50  0001 L CNN
+F 2 "Connector_PinSocket_2.54mm:PinSocket_1x04_P2.54mm_Vertical" H 2250 2800 50  0001 C CNN
+F 3 "~" H 2250 2800 50  0001 C CNN
+	1    2250 2800
+	1    0    0    -1
+$EndComp
+Wire Wire Line
+	1550 2800 2050 2800
+Text Label 1550 2800 0    50   ~ 0
+TSAL
 $EndSCHEMATC
