File: CarMan KiCAD Schematics/TSI/TSI_Rev.5/TSI_Throttle_Plausibility.sch (KiCad schematic (older format))
At the start: 64 parts, among them Q2 MMBF170, SW1 TS5A3159DBVT, U16 TS372CDT, U18 MCP6004, U22 MCP23016-I_SO, U23 DAC5574IDGS, U3 TS912, U30 TLP293, U6 TS912, U7 MCP6004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

Commit message: oopdate
Other:
- note added: "GPIO Expander\n"
Changed lines of the file:
@@
 Wire Notes Line
 	2750 3200 500  3200
+Text Notes 9050 4550 0    79   ~ 0
+GPIO Expander\n
 $EndSCHEMATC

Commit message: organizational update
Connections:
- net labels added: Brake_Light
- wire segments 287 -> 288
Other:
- moved on the sheet: C27
Changed lines of the file:
@@
 Wire Wire Line
 	4100 2250 4250 2250
-Text Label 1000 2600 0    50   ~ 0
+Text Label 1000 2650 0    50   ~ 0
 APPS1_RTN
 Text Label 2150 1200 2    50   ~ 0
 APPS1
-Text Label 1000 2500 0    50   ~ 0
+Text Label 1000 2550 0    50   ~ 0
 APPS1_10V
-Text Label 1000 2900 0    50   ~ 0
+Text Label 1000 2950 0    50   ~ 0
 Throttle_LV
-Text Label 1000 3000 0    50   ~ 0
+Text Label 1000 3050 0    50   ~ 0
 Throttle_PL
 Text Label 2150 1300 2    50   ~ 0
 APPS2
-Text HLabel 1800 3000 2    50   Output ~ 0
+Text HLabel 1800 3050 2    50   Output ~ 0
 Throttle_PL
 Wire Wire Line
@@
 Wire Wire Line
 	14300 8550 14300 8600
-Connection ~ 14300 9000
 Wire Wire Line
 	14300 9000 14300 8900
@@
 	14600 9000 14650 9000
 Wire Notes Line
-	12750 8250 12750 9900
+	12200 8250 12200 9900
 Text Notes 14500 9450 0    50   ~ 0
 Inv. signal\nCurr. Transfer ratio = 100 %
 Wire Wire Line
-	13050 9750 13050 9450
-Wire Wire Line
-	13050 8600 13050 8950
+	12400 9750 12400 9450
+Wire Wire Line
+	12400 8600 12400 8950
 $Comp
 L pspice:CAP C27
 U 1 1 5FDC04B0
-P 13050 9200
-F 0 "C27" H 13150 9050 50  0000 C CNN
-F 1 "0.1u" H 13150 9350 50  0000 C CNN
-F 2 "Capacitor_SMD:C_0805_2012Metric_Pad1.15x1.40mm_HandSolder" H 13050 9200 50  0001 C CNN
-F 3 "~" H 13050 9200 50  0001 C CNN
-	1    13050 9200
+P 12400 9200
+F 0 "C27" H 12500 9050 50  0000 C CNN
+F 1 "0.1u" H 12500 9350 50  0000 C CNN
+F 2 "Capacitor_SMD:C_0805_2012Metric_Pad1.15x1.40mm_HandSolder" H 12400 9200 50  0001 C CNN
+F 3 "~" H 12400 9200 50  0001 C CNN
+	1    12400 9200
 	1    0    0    -1
 $EndComp
@@
 	1    0    0    -1
 $EndComp
-Text Label 13600 9000 0    50   ~ 0
+Text Label 12950 9000 0    50   ~ 0
 BRAKE_OUT
 Text Label 14650 9200 2    50   ~ 0
 GLV_RTN
-Text Label 14800 9750 2    50   ~ 0
-GLV_RTN
-Connection ~ 13600 9750
-Wire Wire Line
-	13050 9750 13600 9750
-Wire Wire Line
-	13050 8600 13600 8600
+Text Label 14150 9750 2    50   ~ 0
+GLV_RTN
+Connection ~ 12950 9750
+Wire Wire Line
+	12400 9750 12950 9750
+Wire Wire Line
+	12400 8600 12950 8600
 Wire Notes Line
 	8450 10850 8450 10100
-Text Notes 13750 8400 0    87   ~ 0
+Text Notes 13475 8400 0    87   ~ 0
 BRAKE PRESSED
 Text Notes 9050 10200 0    59   ~ 0
@@
 Text HLabel 1550 1200 0    50   Input ~ 0
 APPS1
-Text HLabel 1800 2600 2    50   Output ~ 0
+Text HLabel 1800 2650 2    50   Output ~ 0
 APPS1_RTN
-Text HLabel 1800 2500 2    50   Output ~ 0
+Text HLabel 1800 2550 2    50   Output ~ 0
 APPS1_10V
-Text HLabel 1800 2800 2    50   Output ~ 0
+Text HLabel 1800 2850 2    50   Output ~ 0
 APPS2_RTN
 Text HLabel 1550 1300 0    50   Input ~ 0
 APPS2
-Text HLabel 1800 2700 2    50   Output ~ 0
+Text HLabel 1800 2750 2    50   Output ~ 0
 APPS2_5V
 Wire Notes Line
@@
 Wire Notes Line
 	2950 3500 2950 5950
-Text Label 1000 2800 0    50   ~ 0
+Text Label 1000 2850 0    50   ~ 0
 APPS2_RTN
-Text Label 1000 2700 0    50   ~ 0
+Text Label 1000 2750 0    50   ~ 0
 APPS2_5V
 Wire Notes Line
@@
 	15550 2750 15900 2750
 Wire Notes Line
-	13700 8900 13700 8650
-Wire Notes Line
-	13500 8650 13500 8900
-Wire Wire Line
-	13600 9350 13600 9750
-Wire Notes Line
-	13500 9400 13700 9400
-Wire Notes Line
-	13700 9400 13700 9150
-Wire Notes Line
-	13700 9150 13500 9150
-Wire Notes Line
-	13500 9150 13500 9400
-Wire Wire Line
-	13600 9750 14800 9750
-Text Notes 13700 9300 0    31   ~ 0
+	13050 8900 13050 8650
+Wire Notes Line
+	12850 8650 12850 8900
+Wire Wire Line
+	12950 9350 12950 9750
+Wire Notes Line
+	12850 9400 13050 9400
+Wire Notes Line
+	13050 9400 13050 9150
+Wire Notes Line
+	13050 9150 12850 9150
+Wire Notes Line
+	12850 9150 12850 9400
+Wire Wire Line
+	12950 9750 14150 9750
+Text Notes 13050 9300 0    31   ~ 0
 Brake Light & RTDS\n(J17)
 Wire Notes Line
-	13500 8900 13700 8900
-Wire Notes Line
-	13700 8650 13500 8650
-Wire Notes Line
-	12750 9900 16000 9900
-Wire Notes Line
-	12750 8250 16000 8250
+	12850 8900 13050 8900
+Wire Notes Line
+	13050 8650 12850 8650
 Text Label 2150 2200 2    50   ~ 0
 BRAKE_IN
-Text Label 13150 8600 0    50   ~ 0
+Text Label 12500 8600 0    50   ~ 0
 BRAKE_IN
 Wire Wire Line
-	13600 8850 13600 9000
-Wire Wire Line
-	13600 9000 14300 9000
-Connection ~ 13600 9000
-Wire Wire Line
-	13600 9000 13600 9200
-Text Notes 13700 8800 0    31   ~ 0
+	12950 8850 12950 9000
+Connection ~ 12950 9000
+Wire Wire Line
+	12950 9000 12950 9200
+Text Notes 13050 8800 0    31   ~ 0
 Brake & BOT\n(J16)
 Wire Wire Line
@@
 Text HLabel 1550 1700 0    50   Input ~ 0
 BRAKE_OUT
-Text HLabel 1800 2900 2    50   Output ~ 0
+Text HLabel 1800 2950 2    50   Output ~ 0
 Throttle_LV
 Text Label 2150 2300 2    50   ~ 0
@@
 BRAKE_OUT
 Wire Wire Line
-	13600 8700 13600 8600
-Text Label 13750 9750 0    50   ~ 0
+	12950 8700 12950 8600
+Text Label 13100 9750 0    50   ~ 0
 Brake_Light_RTN
-Text Label 1000 3100 0    50   ~ 0
+Text Label 1000 3150 0    50   ~ 0
 Brake_Light_RTN
-Text HLabel 1800 3100 2    50   Output ~ 0
+Text HLabel 1800 3150 2    50   Output ~ 0
 Brake_Light_RTN
 Text Notes 14350 4000 0    51   ~ 0
@@
 	1550 1800 2150 1800
 Wire Wire Line
-	1000 3100 1800 3100
-Wire Wire Line
-	1000 3000 1800 3000
-Wire Wire Line
-	1000 2900 1800 2900
-Wire Wire Line
-	1000 2800 1800 2800
-Wire Wire Line
-	1000 2700 1800 2700
-Wire Wire Line
-	1000 2600 1800 2600
-Wire Wire Line
-	1000 2500 1800 2500
-Wire Notes Line
-	2750 500  2750 3200
-Wire Notes Line
-	500  500  500  3200
-Wire Notes Line
-	2750 3200 500  3200
+	1000 3150 1800 3150
+Wire Wire Line
+	1000 3050 1800 3050
+Wire Wire Line
+	1000 2950 1800 2950
+Wire Wire Line
+	1000 2850 1800 2850
+Wire Wire Line
+	1000 2750 1800 2750
+Wire Wire Line
+	1000 2650 1800 2650
+Wire Wire Line
+	1000 2550 1800 2550
 Text Notes 9050 4550 0    79   ~ 0
 GPIO Expander\n
+Connection ~ 14300 9000
+Text Label 13525 9000 0    50   ~ 0
+Brake_Light
+Wire Notes Line
+	12200 9900 16000 9900
+Wire Notes Line
+	12200 8250 16000 8250
+Text HLabel 1550 2400 0    50   Input ~ 0
+Brake_Light
+Wire Wire Line
+	1550 2400 2150 2400
+Text Label 2150 2400 2    50   ~ 0
+Brake_Light
+Wire Notes Line
+	2750 500  2750 3250
+Wire Notes Line
+	500  3250 2750 3250
+Wire Notes Line
+	500  500  500  3250
+Wire Wire Line
+	12950 9000 14300 9000
 $EndSCHEMATC

Commit message: Small updates
Other:
- note added: "0.24V"
- note added: "4.76V"
- note added: "Voltage Comparator"
Changed lines of the file:
@@
 Wire Wire Line
 	12950 9000 14300 9000
+Text Notes 6575 5425 0    47   ~ 0
+4.76V
+Text Notes 6575 6375 0    47   ~ 0
+0.24V
+Text Notes 6950 2600 0    47   ~ 0
+Voltage Comparator
 $EndSCHEMATC

Commit message: Updated Brake_Pressed_uC Signal
Parts:
- added R98: 1k, Resistor_SMD:R_0805_2012Metric_Pad1.15x1.40mm_HandSolder, symbol Device:R
Connections:
- net labels added: 3.3V
- wire segments 288 -> 292
Other:
- note removed: "Inv. signal\nCurr. Transfer ratio = 100 %"
Changed lines of the file:
@@
 Wire Wire Line
 	4100 2250 4250 2250
-Text Label 1000 2650 0    50   ~ 0
+Text Label 1050 2900 0    50   ~ 0
 APPS1_RTN
 Text Label 2150 1200 2    50   ~ 0
 APPS1
-Text Label 1000 2550 0    50   ~ 0
+Text Label 1050 2800 0    50   ~ 0
 APPS1_10V
-Text Label 1000 2950 0    50   ~ 0
+Text Label 1050 3200 0    50   ~ 0
 Throttle_LV
-Text Label 1000 3050 0    50   ~ 0
+Text Label 1050 3300 0    50   ~ 0
 Throttle_PL
 Text Label 2150 1300 2    50   ~ 0
 APPS2
-Text HLabel 1800 3050 2    50   Output ~ 0
+Text HLabel 1850 3300 2    50   Output ~ 0
 Throttle_PL
 Wire Wire Line
@@
 Wire Notes Line
 	12200 8250 12200 9900
-Text Notes 14500 9450 0    50   ~ 0
-Inv. signal\nCurr. Transfer ratio = 100 %
 Wire Wire Line
 	12400 9750 12400 9450
@@
 	1    0    0    -1
 $EndComp
-Text Label 15300 9200 0    50   ~ 0
-GLV_RTN
-Text Label 15300 9000 0    50   ~ 0
+Text Label 15450 9650 0    50   ~ 0
+GLV_RTN
+Text Label 15950 9200 2    50   ~ 0
 Brake_Pressed_uC
-Wire Wire Line
-	15300 9200 15250 9200
-Wire Wire Line
-	15300 9000 15250 9000
 $Comp
 L TSI_Rev.5-rescue:TLP293-CarMan_KiCAD_Library-TSI_Rev.5-rescue U30
@@
 Text HLabel 1550 1200 0    50   Input ~ 0
 APPS1
-Text HLabel 1800 2650 2    50   Output ~ 0
+Text HLabel 1850 2900 2    50   Output ~ 0
 APPS1_RTN
-Text HLabel 1800 2550 2    50   Output ~ 0
+Text HLabel 1850 2800 2    50   Output ~ 0
 APPS1_10V
-Text HLabel 1800 2850 2    50   Output ~ 0
+Text HLabel 1850 3100 2    50   Output ~ 0
 APPS2_RTN
 Text HLabel 1550 1300 0    50   Input ~ 0
 APPS2
-Text HLabel 1800 2750 2    50   Output ~ 0
+Text HLabel 1850 3000 2    50   Output ~ 0
 APPS2_5V
 Wire Notes Line
@@
 Wire Notes Line
 	2950 3500 2950 5950
-Text Label 1000 2850 0    50   ~ 0
+Text Label 1050 3100 0    50   ~ 0
 APPS2_RTN
-Text Label 1000 2750 0    50   ~ 0
+Text Label 1050 3000 0    50   ~ 0
 APPS2_5V
 Wire Notes Line
@@
 Text HLabel 1550 1700 0    50   Input ~ 0
 BRAKE_OUT
-Text HLabel 1800 2950 2    50   Output ~ 0
+Text HLabel 1850 3200 2    50   Output ~ 0
 Throttle_LV
 Text Label 2150 2300 2    50   ~ 0
@@
 Text Label 13100 9750 0    50   ~ 0
 Brake_Light_RTN
-Text Label 1000 3150 0    50   ~ 0
+Text Label 1050 3400 0    50   ~ 0
 Brake_Light_RTN
-Text HLabel 1800 3150 2    50   Output ~ 0
+Text HLabel 1850 3400 2    50   Output ~ 0
 Brake_Light_RTN
 Text Notes 14350 4000 0    51   ~ 0
@@
 	1550 1800 2150 1800
 Wire Wire Line
-	1000 3150 1800 3150
-Wire Wire Line
-	1000 3050 1800 3050
-Wire Wire Line
-	1000 2950 1800 2950
-Wire Wire Line
-	1000 2850 1800 2850
-Wire Wire Line
-	1000 2750 1800 2750
-Wire Wire Line
-	1000 2650 1800 2650
-Wire Wire Line
-	1000 2550 1800 2550
+	1050 3400 1850 3400
+Wire Wire Line
+	1050 3300 1850 3300
+Wire Wire Line
+	1050 3200 1850 3200
+Wire Wire Line
+	1050 3100 1850 3100
+Wire Wire Line
+	1050 3000 1850 3000
+Wire Wire Line
+	1050 2900 1850 2900
+Wire Wire Line
+	1050 2800 1850 2800
 Text Notes 9050 4550 0    79   ~ 0
 GPIO Expander\n
@@
 Text Label 2150 2400 2    50   ~ 0
 Brake_Light
-Wire Notes Line
-	2750 500  2750 3250
-Wire Notes Line
-	500  3250 2750 3250
-Wire Notes Line
-	500  500  500  3250
 Wire Wire Line
 	12950 9000 14300 9000
@@
 Text Notes 6950 2600 0    47   ~ 0
 Voltage Comparator
+Wire Notes Line
+	2750 500  2750 3450
+Wire Notes Line
+	500  500  500  3450
+Wire Notes Line
+	500  3450 2750 3450
+Text HLabel 1550 2500 0    50   Input ~ 0
+3.3V
+Wire Wire Line
+	1550 2500 2150 2500
+Text Label 2150 2500 2    50   ~ 0
+3.3V
+Wire Wire Line
+	15250 9000 15550 9000
+Text Label 15550 9000 2    50   ~ 0
+3.3V
+Wire Wire Line
+	15250 9200 15300 9200
+Wire Wire Line
+	15300 9200 15300 9350
+Connection ~ 15300 9200
+Wire Wire Line
+	15300 9200 15950 9200
+$Comp
+L Device:R R98
+U 1 1 605CF404
+P 15300 9500
+F 0 "R98" V 15200 9500 50  0000 C CNN
+F 1 "1k" V 15300 9500 50  0000 C CNN
+F 2 "Resistor_SMD:R_0805_2012Metric_Pad1.15x1.40mm_HandSolder" V 15230 9500 50  0001 C CNN
+F 3 "~" H 15300 9500 50  0001 C CNN
+	1    15300 9500
+	1    0    0    -1
+$EndComp
+Wire Wire Line
+	15300 9650 15450 9650
 $EndSCHEMATC

Commit message: TSI Updated & error fixes: added pull down resistors, and 5V_ISO_RTN
Parts:
- removed D4: RED LED TP, LED_SMD:LED_0805_2012Metric_Pad1.15x1.40mm_HandSolder, symbol Device:LED_ALT
- added D4: RED LED TP, LED_SMD:LED_0805_2012Metric_Pad1.15x1.40mm_HandSolder, symbol Device:LED
- R98: value 1k -> 1K
Connections:
- wire segments 292 -> 294
Other:
- note added: "Brake & BOT\n(J17)"
- note added: "Brake Light & RTDS\n(J18)"
- note added: "TP\n(J16)"
- note removed: "Brake & BOT\n(J16)"
- note removed: "Brake Light & RTDS\n(J17)"
- moved on the sheet: C27, R48, R49, R98, U30
Changed lines of the file:
@@
 Text Notes 4650 9000 2    79   ~ 0
 APPS1_b & APPS2_b
-Text Label 14300 8550 0    50   ~ 0
-GLV_RTN
-Wire Wire Line
-	14300 8550 14300 8600
-Wire Wire Line
-	14300 9000 14300 8900
+Text Label 14400 8550 2    50   ~ 0
+GLV_RTN
+Wire Wire Line
+	14050 8550 14050 8600
+Wire Wire Line
+	14050 9000 14050 8900
 $Comp
 L Device:R R48
 U 1 1 609E809D
-P 14300 8750
-F 0 "R48" V 14200 8750 50  0000 C CNN
-F 1 "100K" V 14300 8750 50  0000 C CNN
-F 2 "Resistor_SMD:R_0805_2012Metric_Pad1.15x1.40mm_HandSolder" V 14230 8750 50  0001 C CNN
-F 3 "~" H 14300 8750 50  0001 C CNN
-	1    14300 8750
+P 14050 8750
+F 0 "R48" V 13950 8750 50  0000 C CNN
+F 1 "100K" V 14050 8750 50  0000 C CNN
+F 2 "Resistor_SMD:R_0805_2012Metric_Pad1.15x1.40mm_HandSolder" V 13980 8750 50  0001 C CNN
+F 3 "~" H 14050 8750 50  0001 C CNN
+	1    14050 8750
 	1    0    0    -1
 $EndComp
@@
 L Device:R R49
 U 1 1 60975D89
-P 14450 9000
-F 0 "R49" V 14350 9000 50  0000 C CNN
-F 1 "2.4K" V 14450 9000 50  0000 C CNN
-F 2 "Resistor_SMD:R_0805_2012Metric_Pad1.15x1.40mm_HandSolder" V 14380 9000 50  0001 C CNN
-F 3 "~" H 14450 9000 50  0001 C CNN
-	1    14450 9000
+P 14200 9000
+F 0 "R49" V 14100 9000 50  0000 C CNN
+F 1 "2.4K" V 14200 9000 50  0000 C CNN
+F 2 "Resistor_SMD:R_0805_2012Metric_Pad1.15x1.40mm_HandSolder" V 14130 9000 50  0001 C CNN
+F 3 "~" H 14200 9000 50  0001 C CNN
+	1    14200 9000
 	0    1    1    0
 $EndComp
 Wire Wire Line
-	14600 9000 14650 9000
-Wire Notes Line
-	12200 8250 12200 9900
-Wire Wire Line
-	12400 9750 12400 9450
-Wire Wire Line
-	12400 8600 12400 8950
+	14350 9000 14400 9000
+Wire Notes Line
+	11950 8250 11950 9900
+Wire Wire Line
+	12150 9750 12150 9450
+Wire Wire Line
+	12150 8600 12150 8950
 $Comp
 L pspice:CAP C27
 U 1 1 5FDC04B0
-P 12400 9200
-F 0 "C27" H 12500 9050 50  0000 C CNN
-F 1 "0.1u" H 12500 9350 50  0000 C CNN
-F 2 "Capacitor_SMD:C_0805_2012Metric_Pad1.15x1.40mm_HandSolder" H 12400 9200 50  0001 C CNN
-F 3 "~" H 12400 9200 50  0001 C CNN
-	1    12400 9200
-	1    0    0    -1
-$EndComp
-Text Label 15450 9650 0    50   ~ 0
-GLV_RTN
-Text Label 15950 9200 2    50   ~ 0
+P 12150 9200
+F 0 "C27" H 12250 9050 50  0000 C CNN
+F 1 "0.1u" H 12250 9350 50  0000 C CNN
+F 2 "Capacitor_SMD:C_0805_2012Metric_Pad1.15x1.40mm_HandSolder" H 12150 9200 50  0001 C CNN
+F 3 "~" H 12150 9200 50  0001 C CNN
+	1    12150 9200
+	1    0    0    -1
+$EndComp
+Text Label 15700 9650 2    50   ~ 0
+GLV_RTN
+Text Label 15850 9200 2    50   ~ 0
 Brake_Pressed_uC
 $Comp
 L TSI_Rev.5-rescue:TLP293-CarMan_KiCAD_Library-TSI_Rev.5-rescue U30
 U 1 1 60D50797
-P 14950 9100
-F 0 "U30" H 14950 9425 50  0000 C CNN
-F 1 "TLP293" H 14950 9334 50  0000 C CNN
-F 2 "Package_SO:SOIC-4_4.55x2.6mm_P1.27mm" H 14750 8900 50  0001 L CIN
-F 3 "https://toshiba.semicon-storage.com/info/docget.jsp?did=12884&prodName=TLP291" H 14950 9100 50  0001 L CNN
-	1    14950 9100
-	1    0    0    -1
-$EndComp
-Text Label 12950 9000 0    50   ~ 0
+P 14700 9100
+F 0 "U30" H 14700 9425 50  0000 C CNN
+F 1 "TLP293" H 14700 9334 50  0000 C CNN
+F 2 "Package_SO:SOIC-4_4.55x2.6mm_P1.27mm" H 14500 8900 50  0001 L CIN
+F 3 "https://toshiba.semicon-storage.com/info/docget.jsp?did=12884&prodName=TLP291" H 14700 9100 50  0001 L CNN
+	1    14700 9100
+	1    0    0    -1
+$EndComp
+Text Label 12700 9000 0    50   ~ 0
 BRAKE_OUT
-Text Label 14650 9200 2    50   ~ 0
-GLV_RTN
-Text Label 14150 9750 2    50   ~ 0
-GLV_RTN
-Connection ~ 12950 9750
-Wire Wire Line
-	12400 9750 12950 9750
-Wire Wire Line
-	12400 8600 12950 8600
+Text Label 14050 9200 0    50   ~ 0
+GLV_RTN
+Text Label 13900 9750 2    50   ~ 0
+GLV_RTN
+Connection ~ 12700 9750
+Wire Wire Line
+	12150 9750 12700 9750
+Wire Wire Line
+	12150 8600 12700 8600
 Wire Notes Line
 	8450 10850 8450 10100
-Text Notes 13475 8400 0    87   ~ 0
+Text Notes 13225 8400 0    87   ~ 0
 BRAKE PRESSED
 Text Notes 9050 10200 0    59   ~ 0
 RED LED STATUS LIGHT
-Text Label 10500 10550 0    50   ~ 0
-GLV_RTN
-Wire Wire Line
-	10500 10550 10450 10550
-$Comp
-L Device:LED_ALT D4
-U 1 1 5FE3E975
-P 10300 10550
-F 0 "D4" H 10300 10650 50  0000 C CNN
-F 1 "RED LED TP" H 10300 10400 50  0000 C CNN
-F 2 "LED_SMD:LED_0805_2012Metric_Pad1.15x1.40mm_HandSolder" H 10300 10550 50  0001 C CNN
-F 3 "~" H 10300 10550 50  0001 C CNN
-	1    10300 10550
-	-1   0    0    1
-$EndComp
+Text Label 10850 10550 2    50   ~ 0
+GLV_RTN
 Connection ~ 9850 10550
 $Comp
@@
 Wire Wire Line
 	10250 7000 10250 7100
-Wire Notes Line
-	16000 8250 16000 9900
 $Comp
 L Amplifier_Operational:MCP6004 U7
@@
 	15550 2750 15900 2750
 Wire Notes Line
-	13050 8900 13050 8650
-Wire Notes Line
-	12850 8650 12850 8900
-Wire Wire Line
-	12950 9350 12950 9750
-Wire Notes Line
-	12850 9400 13050 9400
-Wire Notes Line
-	13050 9400 13050 9150
-Wire Notes Line
-	13050 9150 12850 9150
-Wire Notes Line
-	12850 9150 12850 9400
-Wire Wire Line
-	12950 9750 14150 9750
-Text Notes 13050 9300 0    31   ~ 0
-Brake Light & RTDS\n(J17)
-Wire Notes Line
-	12850 8900 13050 8900
-Wire Notes Line
-	13050 8650 12850 8650
+	12800 8900 12800 8650
+Wire Notes Line
+	12600 8650 12600 8900
+Wire Wire Line
+	12700 9350 12700 9750
+Wire Notes Line
+	12600 9400 12800 9400
+Wire Notes Line
+	12800 9400 12800 9150
+Wire Notes Line
+	12800 9150 12600 9150
+Wire Notes Line
+	12600 9150 12600 9400
+Wire Wire Line
+	12700 9750 13900 9750
+Text Notes 12800 9300 0    31   ~ 0
+Brake Light & RTDS\n(J18)
+Wire Notes Line
+	12600 8900 12800 8900
+Wire Notes Line
+	12800 8650 12600 8650
 Text Label 2150 2200 2    50   ~ 0
 BRAKE_IN
-Text Label 12500 8600 0    50   ~ 0
+Text Label 12250 8600 0    50   ~ 0
 BRAKE_IN
 Wire Wire Line
-	12950 8850 12950 9000
-Connection ~ 12950 9000
-Wire Wire Line
-	12950 9000 12950 9200
-Text Notes 13050 8800 0    31   ~ 0
-Brake & BOT\n(J16)
+	12700 8850 12700 9000
+Connection ~ 12700 9000
+Wire Wire Line
+	12700 9000 12700 9200
+Text Notes 12800 8800 0    31   ~ 0
+Brake & BOT\n(J17)
 Wire Wire Line
 	5800 1100 5900 1100
@@
 Wire Notes Line
 	1200 10300 1300 10300
-Text Notes 600  10350 0    31   ~ 0
-Throttle Plausibility\nConnects to pedals:\nAPPS1 2K POT
 Wire Notes Line
 	4500 10450 4500 10100
@@
 BRAKE_OUT
 Wire Wire Line
-	12950 8700 12950 8600
-Text Label 13100 9750 0    50   ~ 0
+	12700 8700 12700 8600
+Text Label 12850 9750 0    50   ~ 0
 Brake_Light_RTN
 Text Label 1050 3400 0    50   ~ 0
@@
 Text Notes 9050 4550 0    79   ~ 0
 GPIO Expander\n
-Connection ~ 14300 9000
-Text Label 13525 9000 0    50   ~ 0
+Connection ~ 14050 9000
+Text Label 13375 9000 0    50   ~ 0
 Brake_Light
-Wire Notes Line
-	12200 9900 16000 9900
-Wire Notes Line
-	12200 8250 16000 8250
 Text HLabel 1550 2400 0    50   Input ~ 0
 Brake_Light
@@
 Brake_Light
 Wire Wire Line
-	12950 9000 14300 9000
+	12700 9000 14050 9000
 Text Notes 6575 5425 0    47   ~ 0
 4.76V
@@
 Text Label 2150 2500 2    50   ~ 0
 3.3V
-Wire Wire Line
-	15250 9000 15550 9000
-Text Label 15550 9000 2    50   ~ 0
+Text Label 15850 9000 2    50   ~ 0
 3.3V
 Wire Wire Line
-	15250 9200 15300 9200
-Wire Wire Line
-	15300 9200 15300 9350
-Connection ~ 15300 9200
-Wire Wire Line
-	15300 9200 15950 9200
+	15000 9200 15050 9200
+Wire Wire Line
+	15050 9200 15050 9350
 $Comp
 L Device:R R98
 U 1 1 605CF404
-P 15300 9500
-F 0 "R98" V 15200 9500 50  0000 C CNN
-F 1 "1k" V 15300 9500 50  0000 C CNN
-F 2 "Resistor_SMD:R_0805_2012Metric_Pad1.15x1.40mm_HandSolder" V 15230 9500 50  0001 C CNN
-F 3 "~" H 15300 9500 50  0001 C CNN
-	1    15300 9500
-	1    0    0    -1
-$EndComp
-Wire Wire Line
-	15300 9650 15450 9650
+P 15050 9500
+F 0 "R98" V 14950 9500 50  0000 C CNN
+F 1 "1K" V 15050 9500 50  0000 C CNN
+F 2 "Resistor_SMD:R_0805_2012Metric_Pad1.15x1.40mm_HandSolder" V 14980 9500 50  0001 C CNN
+F 3 "~" H 15050 9500 50  0001 C CNN
+	1    15050 9500
+	1    0    0    -1
+$EndComp
+Wire Wire Line
+	15050 9650 15700 9650
+Wire Notes Line
+	11950 9900 15950 9900
+Wire Notes Line
+	11950 8250 15950 8250
+Wire Notes Line
+	15950 8250 15950 9900
+Wire Wire Line
+	15050 9200 15850 9200
+Connection ~ 15050 9200
+Wire Wire Line
+	15000 9000 15850 9000
+Wire Wire Line
+	14050 9200 14400 9200
+Wire Wire Line
+	14050 8550 14400 8550
+$Comp
+L Device:LED D?
+U 1 1 60834B36
+P 10300 10550
+AR Path="/5FE1DCBA/60834B36" Ref="D?"  Part="1"
+AR Path="/5FC85F57/60834B36" Ref="D4"  Part="1"
+F 0 "D4" H 10350 10650 50  0000 R CNN
+F 1 "RED LED TP" H 10500 10400 50  0000 R CNN
+F 2 "LED_SMD:LED_0805_2012Metric_Pad1.15x1.40mm_HandSolder" H 10300 10550 50  0001 C CNN
+F 3 "~" H 10300 10550 50  0001 C CNN
+	1    10300 10550
+	-1   0    0    1
+$EndComp
+Wire Wire Line
+	10450 10550 10850 10550
+Text Notes 600  10350 0    31   ~ 0
+Throttle Plausibility\nConnects to pedals:\nAPPS1 2K POT
+Text Notes 4800 10450 0    47   ~ 0
+TP\n(J16)
+Text Notes 1400 10450 0    47   ~ 0
+TP\n(J16)
 $EndSCHEMATC

Commit message: Updated D2 Footprint
Parts:
- D2: footprint Package_SO:MSOP-8_3x3mm_P0.65mm -> Package_SO:SO-8_5.3x6.2mm_P1.27mm
Changed lines of the file:
@@
 F 0 "D2" V 1800 7400 50  0000 R CNN
 F 1 "TL431PS" H 1850 7150 50  0000 R CNN
-F 2 "Package_SO:MSOP-8_3x3mm_P0.65mm" H 1700 7100 50  0001 C CIN
+F 2 "Package_SO:SO-8_5.3x6.2mm_P1.27mm" H 1700 7100 50  0001 C CIN
 F 3 "http://www.ti.com/lit/ds/symlink/tl431.pdf" H 1700 7250 50  0001 C CIN
 	1    1700 7250
