File: CarMan KiCAD Schematics/TSI/TSI_Rev.5/TSI_Throttle_Plausibility.sch (KiCad schematic (older format))
At the start: 65 parts, among them Q2 MMBF170, SW1 TS5A3159DBVT, U16 TS372CDT, U18 MCP6004, U22 MCP23016-I_SO, U23 DAC5574IDGS, U3 TS912, U30 TLP293, U6 TS912, U7 MCP6004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

Commit message: Throttle Plausibility comments
Connections:
- wire segments 294 -> 295
Other:
- note added: "*0-5V Range*"
- note added: "*5-10V Range*"
- note added: "*If the APPS1_ISO and APPS2_b fall \noutside the range of 0.24V-4.76V a \nshort/open is assumed*"
- note added: "*Output is ground if all values are \nhigh and 5V if any values are low*"
- note added: "*Subtracts 5V from APPS1 to bring signal into 0-5V range*\n"
- note added: "*The outputs of the voltage comparator are both high if the differential between APPS1_b and APPS2_b \nis between the 4.44V-5.55V window*"
- note added: "4.44V\n"
- note added: "5.55V"
- note removed: "*Brings 5-10V biases APPS1 signal down to 0-5V*\n"
- moved on the sheet: R44
Changed lines of the file:
@@
 	1    0    0    -1
 $EndComp
-Text Notes 800  5900 0    47   ~ 0
-*Brings 5-10V biases APPS1 signal down to 0-5V*\n
+Text Notes 675  5900 0    47   ~ 0
+*Subtracts 5V from APPS1 to bring signal into 0-5V range*\n
 Wire Notes Line
 	550  3500 550  5950
@@
 Text Label 15900 2750 2    50   ~ 0
 5V
-Text Label 13650 3150 0    50   ~ 0
+Text Label 13475 3150 0    50   ~ 0
 Throttle_LV
 $Comp
@@
 L Device:R R44
 U 1 1 608A2A55
-P 13550 2550
-F 0 "R44" H 13600 2550 50  0000 L BNN
-F 1 "10K" V 13550 2545 50  0000 C CNN
-F 2 "Resistor_SMD:R_0805_2012Metric_Pad1.15x1.40mm_HandSolder" V 13480 2550 50  0001 C CNN
-F 3 "~" H 13550 2550 50  0001 C CNN
-	1    13550 2550
+P 14125 2550
+F 0 "R44" H 14175 2550 50  0000 L BNN
+F 1 "10K" V 14125 2545 50  0000 C CNN
+F 2 "Resistor_SMD:R_0805_2012Metric_Pad1.15x1.40mm_HandSolder" V 14055 2550 50  0001 C CNN
+F 3 "~" H 14125 2550 50  0001 C CNN
+	1    14125 2550
 	-1   0    0    1
 $EndComp
-Text Label 13250 2300 0    50   ~ 0
-GLV_RTN
-Text Label 14100 2950 2    50   ~ 0
+Text Label 13825 2300 0    50   ~ 0
+GLV_RTN
+Text Label 13450 2950 0    50   ~ 0
 Throttle_SEL
 Wire Wire Line
-	13550 2950 14150 2950
-Wire Wire Line
-	13550 2700 13550 2950
+	14125 2700 14125 2950
 Text Notes 14600 2600 0    63   ~ 0
 AUTO TURN\nOFF SWITCH
@@
 NoConn ~ 10250 6700
 Wire Wire Line
-	8550 3200 8550 3350
-Wire Wire Line
-	8550 3350 8550 3450
-Connection ~ 8550 3350
-Wire Wire Line
 	9750 3700 10950 3700
-$Comp
-L TSI_Rev.5-rescue:74ACT11030-74act11030 U?
-U 1 1 604CB1E4
-P 9150 3700
-AR Path="/604CB1E4" Ref="U?"  Part="1"
-AR Path="/5FC85F57/604CB1E4" Ref="U8"  Part="1"
-F 0 "U8" H 9050 3800 50  0000 L CNN
-F 1 "74ACT11030" H 8900 3600 50  0000 L CNN
-F 2 "TSI_Rev_2021_Footprint_Lib:SOIC127P600X175-14N" H 9150 3700 50  0001 C CNN
-F 3 "https://www.snapeda.com/parts/74ACT11030DR/Texas%20Instruments/datasheet/" H 9150 3700 50  0001 C CNN
-	1    9150 3700
-	1    0    0    -1
-$EndComp
 Wire Wire Line
 	5900 1100 5900 1400
@@
 	14900 4550 14600 4550
 Wire Wire Line
-	13250 2300 13550 2300
-Wire Wire Line
-	13550 2300 13550 2400
-Wire Wire Line
-	13650 3150 14150 3150
+	13825 2300 14125 2300
+Wire Wire Line
+	14125 2300 14125 2400
 Wire Wire Line
 	15550 3550 15900 3550
@@
 Text Notes 1400 10450 0    47   ~ 0
 TP\n(J16)
+Text Notes 5925 1875 0    47   ~ 0
+5.55V
+Text Notes 5925 2500 0    47   ~ 0
+4.44V\n
+Text Notes 4200 3150 0    47   ~ 0
+*The outputs of the voltage comparator are both high if the differential between APPS1_b and APPS2_b \nis between the 4.44V-5.55V window*
+Text Notes 3075 10475 0    47   ~ 0
+*5-10V Range*
+Text Notes 6475 10475 0    47   ~ 0
+*0-5V Range*
+Connection ~ 14125 2950
+Wire Wire Line
+	14125 2950 14150 2950
+Wire Wire Line
+	13450 2950 14125 2950
+Wire Wire Line
+	13475 3150 14150 3150
+Text Notes 6200 3675 0    47   ~ 0
+4.76V
+Text Notes 6225 4625 0    47   ~ 0
+0.24V
+Wire Wire Line
+	8550 3200 8550 3350
+Wire Wire Line
+	8550 3350 8550 3450
+Connection ~ 8550 3350
+$Comp
+L TSI_Rev.5-rescue:74ACT11030-74act11030 U?
+U 1 1 604CB1E4
+P 9150 3700
+AR Path="/604CB1E4" Ref="U?"  Part="1"
+AR Path="/5FC85F57/604CB1E4" Ref="U8"  Part="1"
+F 0 "U8" H 9050 3800 50  0000 L CNN
+F 1 "74ACT11030" H 8900 3600 50  0000 L CNN
+F 2 "TSI_Rev_2021_Footprint_Lib:SOIC127P600X175-14N" H 9150 3700 50  0001 C CNN
+F 3 "https://www.snapeda.com/parts/74ACT11030DR/Texas%20Instruments/datasheet/" H 9150 3700 50  0001 C CNN
+	1    9150 3700
+	1    0    0    -1
+$EndComp
+Text Notes 9050 3425 0    47   ~ 0
+*Output is ground if all values are \nhigh and 5V if any values are low*
+Text Notes 5000 6850 0    47   ~ 0
+*If the APPS1_ISO and APPS2_b fall \noutside the range of 0.24V-4.76V a \nshort/open is assumed*
 $EndSCHEMATC
