File: CarMan KiCAD Schematics/Logic_2022/Logic.sch (KiCad schematic (older format))
At the start: 8 parts, among them J2 J2 NI I2C, J4 J4 GLV BOB, U10 BNO_055, U11 Raspberry_Pi_RTC, U6 RaspberryPi3

Commit message: Update the PCB layout with the wiring connected
Parts:
- added C10, C11, C18, C21: 0.1uF, Capacitor_SMD:C_0805_2012Metric_Pad1.15x1.40mm_HandSolder, symbol Device:C
- added C12, C2: 0.1uF, Capacitor_SMD:C_0805_2012Metric_Pad1.15x1.40mm_HandSolder, symbol Logic-rescue:C-Device-Logic-rescue
- added C4, C6, C7, C8, C9: 0.1u, Capacitor_SMD:C_0805_2012Metric_Pad1.15x1.40mm_HandSolder, symbol Logic-rescue:C-Device-Logic-rescue
- added D1: 5V ISO, CarMan General Footprints:VAOL-S8GT4, symbol Device:LED
- added D2: 3.3V ISO, CarMan General Footprints:VAOL-S8GT4, symbol Device:LED
- added D3: SDA ISO, CarMan General Footprints:VAOL-S8GT4, symbol Device:LED
- added D4: STATE_OUT_1, CarMan General Footprints:VAOL-S8GT4, symbol Device:LED
- added D5: STATE_OUT_2, CarMan General Footprints:VAOL-S8GT4, symbol Device:LED
- added D6: STATE_OUT_3, CarMan General Footprints:VAOL-S8GT4, symbol Device:LED
- added D7: 24V, CarMan General Footprints:VAOL-S8GT4, symbol Device:LED
- added D8: 5V NI, CarMan General Footprints:VAOL-S8GT4, symbol Device:LED
- added J1: J1 MC Can Line, CarMan General Footprints:Molex_MiniFit-JR-5556-04A_2x02x4.20mm_Straight, symbol Logic-rescue:Conn_01x04-Connector_Generic-Logic-rescue
- added J3: J3 Logic-TSI, Connector_PinSocket_2.54mm:PinSocket_2x05_P2.54mm_Vertical, symbol Connector_Generic:Conn_02x05_Odd_Even
- added J5: J5 PICKit 3, Connector_PinSocket_2.54mm:PinSocket_1x06_P2.54mm_Vertical, symbol Logic-rescue:Conn_01x06-Connector_Generic-Logic-rescue
- added J6: J6 NI CAN, Connector_PinSocket_2.54mm:PinSocket_1x02_P2.54mm_Vertical, symbol Connector_Generic:Conn_01x02
- added L1: 28nH, Inductor_SMD:L_0805_2012Metric_Pad1.15x1.40mm_HandSolder, symbol Logic-rescue:L-Device-Logic-rescue
- added R1, R2, R3: 10k, Resistor_SMD:R_0805_2012Metric_Pad1.15x1.40mm_HandSolder, symbol Logic-rescue:R-Device-Logic-rescue
- added R11, R12, R13, R14, R15, R8, R9: 10k, Resistor_SMD:R_0805_2012Metric_Pad1.15x1.40mm_HandSolder, symbol Device:R
- added R16: 2K, Resistor_SMD:R_0805_2012Metric_Pad1.15x1.40mm_HandSolder, symbol Device:R
- added R4: 1k, Resistor_SMD:R_0805_2012Metric_Pad1.15x1.40mm_HandSolder, symbol Logic-rescue:R-Device-Logic-rescue
- added R5, R6: 1K, Resistor_SMD:R_0805_2012Metric_Pad1.15x1.40mm_HandSolder, symbol Device:R
- added R7: 120, Resistor_SMD:R_0805_2012Metric_Pad1.15x1.40mm_HandSolder, symbol Logic-rescue:R-Device-Logic-rescue
- added U1: MCP9700AT-HTT-Sensor_Temperature-Logic-rescue, Package_TO_SOT_SMD:SOT-23, symbol Logic-rescue:MCP9700AT-HTT-Sensor_Temperature-Logic-rescue
- added U3: PIC32MZ2048EFM064-I_PT, CarMan General Footprints:QFP50P1200X1200X120-64N, symbol Logic-rescue:PIC32MZ2048EFM064-I_PT-PIC32MZ2048EFM064-I_PT
- added U5: ISO1050DUB, Package_SO:SOP-8_6.62x9.15mm_P2.54mm, symbol Interface_CAN_LIN:ISO1050DUB
- added U9: ISO1541DR, CarMan General Footprints:ISO1541DR, symbol Logic-rescue:ISO1541DR-CarMan_KiCAD_Library
- U6: symbol Logic-rescue:RaspberryPi3-Lafayette_Electric_Car_Internals -> Logic-rescue:RaspberryPi3-Lafayette_Electric_Car_Internals-Logic-rescue
Connections:
- net 24V: now also R13.1
- net 3.3V_ISO: now also C10.1, C18.1, C4.2, C6.2, C7.2, C8.2, C9.2, J3.7 (Pin_7), J5.2 (Pin_2), L1.1, L1.2, R1.2, R2.2, R3.2, R5.1, U3.19 (AVDD), U3.26 (VDD), U3.39 (VDD), U3.54 (VDD), U3.60 (VDD), U3.8 (VDD), U9.1 (VCC1)
- net 5V_ISO: now also C11.1, R16.1, U1.1 (Vdd), U5.1 (VCC1)
- net 5V_NON_ISO: now also C12.2, C21.2, R12.1, R14.1, R15.1, U5.8 (VCC2), U9.8 (VCC2)
- net GLV_RTN: now also C12.1, C21.1, D7.1 (K), D8.1 (K), U5.5 (GND2), U9.5 (GND2)
- net ISO_RTN: now also C10.2, C11.2, C18.2, C2.1, C4.1, C6.1, C7.1, C8.1, C9.1, D1.1 (K), D2.1 (K), D3.1 (K), D4.1 (K), D5.1 (K), D6.1 (K), J1.3 (Pin_3), J3.5 (Pin_5), J5.3 (Pin_3), U1.3 (GND), U3.20 (AVSS), U3.25 (VSS), U3.34 (VUSB3V3), U3.35 (VSS), U3.40 (VSS), U3.55 (VSS), U3.59 (VSS), U3.7 (VSS), U5.4 (GND1), U9.4 (GND1)
- net SCL_ISO_PI: now also R1.1, U3.6 (AN12/C2IND/RPG8/SCL4/PMA3/RG8), U9.3 (SCL1)
- net SCL_TSI_GLV: now also J3.4 (Pin_4), R14.2, U9.6 (SCL2)
- net SDA_ISO_PI: now also R2.1, R6.1, U3.5 (AN13/C1INC/RPG7/SDA4/PMA4/RG7), U9.2 (SDA1)
- net SDA_TSI_GLV: now also J3.2 (Pin_2), R12.2, U9.7 (SDA2)
- net SR_CTRL: now also J3.3 (Pin_3)
- new net: D2.2 (A), R5.2
- new net: D3.2 (A), R6.2
- new net: D8.2 (A), R15.2
- new net: C2.2, R3.1, R4.2
- new net: D7.2 (A), R13.2
- new net: D1.2 (A), R16.2
- new net: D5.2 (A), R9.2
- new net: D6.2 (A), R11.2
- new net: D4.2 (A), R8.2
- new net: J6.1 (Pin_1), R7.1
- new net BP_CAN+: J1.1 (Pin_1), J3.8 (Pin_8), R7.2, U5.7 (CANH)
- new net BP_CAN-: J1.2 (Pin_2), J3.6 (Pin_6), J6.2 (Pin_2), U5.6 (CANL)
- new net Cooling_CTRL: J3.1 (Pin_1), U3.3 (AN15/ETXD1/PMD7/RE7)
- new net FlowRate: J3.9 (Pin_9), U3.18 (PGED2/AN47/RPB7/RB7)
- new net PGEC: J5.5 (Pin_5), U3.15 (PGEC1/VREF-/CVREF-/AN1/RPB1/RB1)
- new net PGED: J5.4 (Pin_4), U3.16 (PGED1/VREF+/CVREF+/AN0/RPB0/PMA6/RB0)
- new net PIC_RXD: U3.42 (RPF5/SCL5/PMA8/RF5), U5.2 (RXD)
- new net PIC_TXD: U3.41 (RPF4/SDA5/PMA9/RF4), U5.3 (TXD)
- new net STATE_OUT_1: R8.1, U3.46 (AERXD1/ETXD3/RPD0/RTCC/INT0/RD0)
- new net STATE_OUT_2: R9.1, U3.49 (EMDIO/AEMDIO/RPD1/SCK1/RD1)
- new net STATE_OUT_3: R11.1, U3.50 (ETXERR/AETXEN/RPD2/SDA3/RD2)
- new net V_OUT_TEMP: U1.2 (Vout), U3.29 (AN9/RPB14/SCK3/PMA1/RB14)
- new net ~MCLR~: J5.1 (Pin_1), R4.1, U3.9 (~MCLR~)
- no-connect marks 25 -> 65
Other:
- note added: "5V & 3.3V have same isolated return"
- note added: "Analog Temperature Sensor"
- note added: "Bi-Directional I2C Isolator"
- note added: "Drive State LEDs"
- note added: "HIERARCHICAL SHEETS"
- note added: "Isolated Can Transceiver"
- note added: "Isolated Status LEDs"
- note added: "LOGIC HEADERS"
- note added: "Logic-TSI Connector"
- note added: "Motor Controller\nCan Line"
- note added: "NON-ISO CAN\nTesting Header"
- note added: "Non-Isolated Voltage LEDs"
- note added: "PICKit Programming Header"
- note removed: "SHIELD HEADERS"
- moved on the sheet: J2, J4, U6
