File: CarMan KiCAD Schematics/Logic_2022/PiShield.sch (KiCad schematic (older format))
At the start: 24 parts, among them J1 J2 NI I2C, J2 J4 GLV BOB, J3 PICAN 2 Connector, J4 Motor Controller Header, J5 TSI Header, J6 PICAN 2 Connector, J7 CAN Testing Header, U1 RaspberryPi3, U10 BNO_055, U11 Raspberry_Pi_RTC

Commit message: Updated the footprints
Parts:
- removed F1, F2: PWR_FLAG, symbol power:PWR_FLAG
- D1: value LED -> D1
- D2: value LED -> D2
- D3: value LED -> D3
- J1: value J2 NI I2C -> I2C Testing Header; footprint Connector_PinSocket_2.54mm:PinSocket_1x04_P2.54mm_Vertical -> Connector_PinHeader_2.54mm:PinHeader_1x04_P2.54mm_Vertical
- J2: value J4 GLV BOB -> J2
- J3: value PICAN 2 Connector -> J3
- J4: value Motor Controller Header -> J4
- J5: value TSI Header -> J5
- J6: value PICAN 2 Connector -> J6
- J7: value CAN Testing Header -> J7
- PS1: value Regulator -> PS1
Other:
- note added: "CAN Testing Header"
- note added: "GPIO Test"
- note added: "Motor Controller Header\n"
- note added: "PICAN 2 Connector"
- note added: "TSI Header\n"
Changed lines of the file:
@@
 P 7010 2770
 F 0 "J2" H 6960 2470 50  0000 L CNN
-F 1 "J4 GLV BOB" H 6835 2995 50  0001 L CNN
+F 1 "J2" H 6835 2995 50  0001 L CNN
 F 2 "CarMan General Footprints:Molex_MiniFit-JR-5556-04A_2x02x4.20mm_Straight" H 7010 2770 50  0001 C CNN
 F 3 "~" H 7010 2770 50  0001 C CNN
@@
 Wire Wire Line
 	2475 5575 3225 5575
-Text Notes 6860 3020 0    50   ~ 0
+Text Notes 6855 3095 0    50   ~ 0
 GLV 24V and I2C to logic
 Wire Wire Line
@@
 P 5745 2660
 F 0 "J1" H 5695 2860 50  0000 L CNN
-F 1 "J2 NI I2C" H 5170 2860 50  0001 L CNN
-F 2 "Connector_PinSocket_2.54mm:PinSocket_1x04_P2.54mm_Vertical" H 5745 2660 50  0001 C CNN
+F 1 "I2C Testing Header" H 5170 2860 50  0001 L CNN
+F 2 "Connector_PinHeader_2.54mm:PinHeader_1x04_P2.54mm_Vertical" H 5745 2660 50  0001 C CNN
 F 3 "~" H 5745 2660 50  0001 C CNN
 	1    5745 2660
 	-1   0    0    -1
 $EndComp
-Text Notes 5700 3035 0    47   ~ 0
+Text Notes 5765 3090 0    47   ~ 0
 I2C Testing Header
 Text Label 6470 2760 2    50   ~ 0
@@
 P 8700 6005
 F 0 "PS1" H 9145 4715 50  0000 L CNN
-F 1 "Regulator" H 9050 6205 50  0000 L CNN
+F 1 "PS1" H 9050 6205 50  0001 L CNN
 F 2 "SamacSys_Parts:P783Q24S5S" H 9550 6105 50  0001 L CNN
 F 3 "https://www.cui.com/product/resource/digikeypdf/p783-s.pdf" H 9550 6005 50  0001 L CNN
@@
 P 11215 5555
 F 0 "D1" V 11254 5437 50  0000 R CNN
-F 1 "LED" V 11163 5437 50  0000 R CNN
+F 1 "D1" V 11163 5437 50  0001 R CNN
 F 2 "CarMan General Footprints:VAOL-S8GT4" H 11215 5555 50  0001 C CNN
 F 3 "~" H 11215 5555 50  0001 C CNN
@@
 P 11630 5565
 F 0 "D2" V 11669 5447 50  0000 R CNN
-F 1 "LED" V 11578 5447 50  0000 R CNN
+F 1 "D2" V 11578 5447 50  0001 R CNN
 F 2 "CarMan General Footprints:VAOL-S8GT4" H 11630 5565 50  0001 C CNN
 F 3 "~" H 11630 5565 50  0001 C CNN
@@
 P 12025 5580
 F 0 "D3" V 12064 5462 50  0000 R CNN
-F 1 "LED" V 11973 5462 50  0000 R CNN
+F 1 "D3" V 11973 5462 50  0001 R CNN
 F 2 "CarMan General Footprints:VAOL-S8GT4" H 12025 5580 50  0001 C CNN
 F 3 "~" H 12025 5580 50  0001 C CNN
@@
 P 2420 2795
 F 0 "J4" H 2338 2370 50  0000 C CNN
-F 1 "Motor Controller Header" H 2330 3045 50  0000 C CNN
+F 1 "J4" H 2330 3045 50  0001 C CNN
 F 2 "CarMan General Footprints:Molex_MiniFit-JR-5556-04A_2x02x4.20mm_Straight" H 2420 2795 50  0001 C CNN
 F 3 "" H 2420 2795 50  0001 C CNN
@@
 P 3735 2800
 F 0 "J5" H 3653 2375 50  0000 C CNN
-F 1 "TSI Header" H 3680 3045 50  0000 C CNN
+F 1 "J5" H 3680 3045 50  0001 C CNN
 F 2 "Connector_PinHeader_2.54mm:PinHeader_2x05_P2.54mm_Vertical" H 3735 2800 50  0001 C CNN
 F 3 "" H 3735 2800 50  0001 C CNN
@@
 P 4800 2805
 F 0 "J6" H 4718 2480 50  0000 C CNN
-F 1 "PICAN 2 Connector" H 4750 2975 50  0000 C CNN
+F 1 "J6" H 4750 2975 50  0001 C CNN
 F 2 "Connector_PinHeader_2.54mm:PinHeader_1x02_P2.54mm_Vertical" H 4800 2805 50  0001 C CNN
 F 3 "~" H 4800 2805 50  0001 C CNN
@@
 P 8435 2740
 F 0 "J3" H 8353 2415 50  0000 C CNN
-F 1 "PICAN 2 Connector" H 8385 2910 50  0000 C CNN
+F 1 "J3" H 8385 2910 50  0001 C CNN
 F 2 "Connector_PinHeader_2.54mm:PinHeader_1x02_P2.54mm_Vertical" H 8435 2740 50  0001 C CNN
 F 3 "~" H 8435 2740 50  0001 C CNN
@@
 P 9385 2740
 F 0 "J7" H 9303 2415 50  0000 C CNN
-F 1 "CAN Testing Header" H 9335 2910 50  0000 C CNN
+F 1 "J7" H 9335 2910 50  0001 C CNN
 F 2 "Connector_PinHeader_2.54mm:PinHeader_1x02_P2.54mm_Vertical" H 9385 2740 50  0001 C CNN
 F 3 "~" H 9385 2740 50  0001 C CNN
@@
 	10620 1715 10620 3370
 $Comp
-L power:PWR_FLAG F1
+L power:PWR_FLAG #F01
 U 1 1 62289588
 P 7810 2570
-F 0 "F1" H 7810 2645 50  0001 C CNN
+F 0 "#F01" H 7810 2645 50  0001 C CNN
 F 1 "PWR_FLAG" V 7810 2698 50  0000 L CNN
 F 2 "" H 7810 2570 50  0001 C CNN
@@
 	7810 2570 7210 2570
 $Comp
-L power:PWR_FLAG F2
+L power:PWR_FLAG #F02
 U 1 1 62298F01
 P 7810 2670
-F 0 "F2" H 7810 2745 50  0001 C CNN
+F 0 "#F02" H 7810 2745 50  0001 C CNN
 F 1 "PWR_FLAG" V 7810 2798 50  0000 L CNN
 F 2 "" H 7810 2670 50  0001 C CNN
@@
 	0    1    1    0
 $EndComp
+Text Notes 2235 3115 0    47   ~ 0
+Motor Controller Header\n
+Text Notes 3790 3130 0    47   ~ 0
+TSI Header\n
+Text Notes 4640 3060 0    47   ~ 0
+PICAN 2 Connector
+Text Notes 8365 3010 0    47   ~ 0
+GPIO Test
+Text Notes 9320 2960 0    47   ~ 0
+CAN Testing Header
 $EndSCHEMATC
