File: CarMan KiCAD Schematics/TSI/TSI_Rev.7/PCDC_Circuit.sch (KiCad schematic (older format))
At the start: 61 parts, among them IC1 TS431ILT, K1 APAN3105, Q1 ZVP1320F, Q3 SI1302DL-T1-E3, U10 MC7805BDTRKG, U12 REF3033, U19 SN74HC00APWR, U21 MCP6004, U27 TLP293, U34 TLP293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

Commit message: TSI Should be final schematic
Parts:
- removed U21, U35: MCP6004, TSI_Rev_2021_Footprint_Lib:SOIC127P600X175-14N, symbol TSI_Rev.5-rescue:MCP6004-Amplifier_Operational
- removed unit 5 of U40
- removed unit 1 of U40
- removed unit 2 of U40
- added U21, U35: TLV2464CDR, CarMan General Footprints:SOIC127P600X175-14N, symbol CarMan_KiCAD_Library:TLV2464CDR
- added unit 1 of U40
- added unit 5 of U40
- added unit 2 of U40
- U40: value MCP6004 -> TLV2464CDR; footprint TSI_Rev_2021_Footprint_Lib:SOIC127P600X175-14N -> CarMan General Footprints:SOIC127P600X175-14N
Connections:
- net 5HV: now also U40.4 (V+)
- net 5V: now also U35.4 (V+)
- net DC_RELAY-: now also U40.11 (V-)
- net GLV_RTN: now also U35.11 (V-)
- net MC_95%: now also U40.7
- net MC_Voltage: now also U21.12 (+)
- net Safety_Loop: now also U35.3 (+)
- net TSV_MIN_REF: now also U40.2 (-)
- net TSV_Ready: now also U40.1
- net TS_Voltage: now also U21.10 (+)
- net at R105.1, R47.1: now also U35.1, U35.2 (-)
- net at RV1.3: now also U21.8, U21.9 (-), U40.3 (+)
- net at RV1.2: now also U40.5 (+)
- new net: U21.13 (-), U21.14, U40.6 (-)
Changed lines of the file:
@@
 $Descr A2 23386 16535
 encoding utf-8
-Sheet 3 7
+Sheet 2 7
 Title ""
 Date ""
@@
 Text Label 6425 6575 0    69   ~ 0
 MC_95%
-$Comp
-L TSI_Rev.5-rescue:MCP6004-Amplifier_Operational U40
-U 2 1 616E5BE5
-P 5150 6575
-F 0 "U40" H 5150 6575 50  0000 C CNN
-F 1 "MCP6004" H 5350 6450 50  0000 C CNN
-F 2 "TSI_Rev_2021_Footprint_Lib:SOIC127P600X175-14N" H 5100 6675 50  0001 C CNN
-F 3 "http://www.ti.com/lit/gpn/sn74hc00" H 5200 6775 50  0001 C CNN
-	2    5150 6575
-	1    0    0    1
-$EndComp
 Wire Wire Line
 	5725 5650 5725 6375
@@
 Text Label 5050 5950 0    50   ~ 0
 IO_Ground
-$Comp
-L TSI_Rev.5-rescue:MCP6004-Amplifier_Operational U40
-U 1 1 616E5BDE
-P 5150 5650
-F 0 "U40" H 5200 5650 50  0000 C CNN
-F 1 "MCP6004" H 5300 5800 50  0000 C CNN
-F 2 "TSI_Rev_2021_Footprint_Lib:SOIC127P600X175-14N" H 5100 5750 50  0001 C CNN
-F 3 "http://www.ti.com/lit/gpn/sn74hc00" H 5200 5850 50  0001 C CNN
-	1    5150 5650
-	1    0    0    -1
-$EndComp
-$Comp
-L TSI_Rev.5-rescue:MCP6004-Amplifier_Operational U40
-U 5 1 616E5BD8
-P 5150 5650
-F 0 "U40" H 5108 5696 50  0001 L CNN
-F 1 "MCP6004" H 5108 5650 50  0001 L CNN
-F 2 "TSI_Rev_2021_Footprint_Lib:SOIC127P600X175-14N" H 5100 5750 50  0001 C CNN
-F 3 "http://www.ti.com/lit/gpn/sn74hc00" H 5200 5850 50  0001 C CNN
-	5    5150 5650
-	1    0    0    -1
-$EndComp
 Text Label 5050 5350 0    50   ~ 0
 5HV
@@
 Text Label 2100 5450 0    79   ~ 0
 TS_Voltage
-$Comp
-L TSI_Rev.5-rescue:MCP6004-Amplifier_Operational U?
-U 3 1 616E5BB2
-P 3250 5550
-AR Path="/5FC85F57/616E5BB2" Ref="U?"  Part="3"
-AR Path="/6196BF15/616E5BB2" Ref="U21"  Part="3"
-F 0 "U21" H 3200 5550 50  0000 C CNN
-F 1 "MCP6004" H 3400 5400 50  0000 C CNN
-F 2 "TSI_Rev_2021_Footprint_Lib:SOIC127P600X175-14N" H 3200 5650 50  0001 C CNN
-F 3 "http://www.ti.com/lit/gpn/sn74hc00" H 3300 5750 50  0001 C CNN
-	3    3250 5550
-	1    0    0    -1
-$EndComp
-$Comp
-L TSI_Rev.5-rescue:MCP6004-Amplifier_Operational U?
-U 4 1 616E5BAC
-P 3250 6675
-AR Path="/5FC85F57/616E5BAC" Ref="U?"  Part="4"
-AR Path="/6196BF15/616E5BAC" Ref="U21"  Part="4"
-F 0 "U21" H 3200 6675 50  0000 C CNN
-F 1 "MCP6004" H 3400 6525 50  0000 C CNN
-F 2 "TSI_Rev_2021_Footprint_Lib:SOIC127P600X175-14N" H 3200 6775 50  0001 C CNN
-F 3 "http://www.ti.com/lit/gpn/sn74hc00" H 3300 6875 50  0001 C CNN
-	4    3250 6675
-	1    0    0    -1
-$EndComp
 Text Notes 15875 6725 0    35   ~ 0
 Flyback\nDiode
@@
 P 15450 8250
 F 0 "U40" H 15450 8250 50  0000 C CNN
-F 1 "MCP6004" H 15450 8526 50  0000 C CNN
-F 2 "TSI_Rev_2021_Footprint_Lib:SOIC127P600X175-14N" H 15400 8350 50  0001 C CNN
-F 3 "http://www.ti.com/lit/gpn/sn74hc00" H 15500 8450 50  0001 C CNN
+F 1 "TLV2464CDR" H 15450 8526 50  0000 C CNN
+F 2 "CarMan General Footprints:SOIC127P600X175-14N" H 15400 8350 50  0001 C CNN
+F 3 "" H 15500 8450 50  0001 C CNN
 	4    15450 8250
 	1    0    0    -1
@@
 Wire Wire Line
 	3900 13000 3600 13000
-$Comp
-L TSI_Rev.5-rescue:MCP6004-Amplifier_Operational U35
-U 1 1 6135E725
-P 3700 12700
-F 0 "U35" H 3700 12700 50  0000 C CNN
-F 1 "MCP6004" H 3900 12850 50  0000 C CNN
-F 2 "TSI_Rev_2021_Footprint_Lib:SOIC127P600X175-14N" H 3650 12800 50  0001 C CNN
-F 3 "http://ww1.microchip.com/downloads/en/DeviceDoc/21733j.pdf" H 3750 12900 50  0001 C CNN
-	1    3700 12700
-	1    0    0    -1
-$EndComp
-$Comp
-L TSI_Rev.5-rescue:MCP6004-Amplifier_Operational U35
-U 5 1 613AB3DB
-P 3700 12700
-F 0 "U35" H 3658 12700 50  0001 L CNN
-F 1 "MCP6004" H 3658 12655 50  0001 L CNN
-F 2 "TSI_Rev_2021_Footprint_Lib:SOIC127P600X175-14N" H 3650 12800 50  0001 C CNN
-F 3 "http://ww1.microchip.com/downloads/en/DeviceDoc/21733j.pdf" H 3750 12900 50  0001 C CNN
-	5    3700 12700
-	1    0    0    -1
-$EndComp
 Connection ~ 4150 12700
 Wire Wire Line
@@
 Text Notes 16100 5775 2    31   ~ 0
 This state is not possible since whenver Safety_Loop_HV is low, the output of U19C must be high
+$Comp
+L CarMan_KiCAD_Library:TLV2464CDR U?
+U 1 1 62FA2AD2
+P 5150 5650
+AR Path="/5FC85F57/62FA2AD2" Ref="U?"  Part="1"
+AR Path="/6196BF15/62FA2AD2" Ref="U40"  Part="1"
+F 0 "U40" H 5150 5650 50  0000 C CNN
+F 1 "TLV2464CDR" H 5300 5900 50  0001 C CNN
+F 2 "CarMan General Footprints:SOIC127P600X175-14N" H 5100 5750 50  0001 C CNN
+F 3 "" H 5200 5850 50  0001 C CNN
+	1    5150 5650
+	1    0    0    -1
+$EndComp
+$Comp
+L CarMan_KiCAD_Library:TLV2464CDR U?
+U 5 1 62FA2AD8
+P 5150 5650
+AR Path="/5FC85F57/62FA2AD8" Ref="U?"  Part="5"
+AR Path="/6196BF15/62FA2AD8" Ref="U40"  Part="5"
+F 0 "U40" H 5100 6100 50  0001 L CNN
+F 1 "TLV2464CDR" H 5150 5500 50  0000 L CNN
+F 2 "CarMan General Footprints:SOIC127P600X175-14N" H 5100 5750 50  0001 C CNN
+F 3 "" H 5200 5850 50  0001 C CNN
+	5    5150 5650
+	1    0    0    -1
+$EndComp
+$Comp
+L CarMan_KiCAD_Library:TLV2464CDR U?
+U 2 1 62FA2ADE
+P 5150 6575
+AR Path="/5FC85F57/62FA2ADE" Ref="U?"  Part="2"
+AR Path="/6196BF15/62FA2ADE" Ref="U40"  Part="2"
+F 0 "U40" H 5150 6575 50  0000 C CNN
+F 1 "TLV2464CDR" H 5250 6375 50  0000 C CNN
+F 2 "CarMan General Footprints:SOIC127P600X175-14N" H 5100 6675 50  0001 C CNN
+F 3 "" H 5200 6775 50  0001 C CNN
+	2    5150 6575
+	1    0    0    -1
+$EndComp
+$Comp
+L CarMan_KiCAD_Library:TLV2464CDR U?
+U 3 1 62FA2AE4
+P 3250 5550
+AR Path="/5FC85F57/62FA2AE4" Ref="U?"  Part="3"
+AR Path="/6196BF15/62FA2AE4" Ref="U21"  Part="3"
+F 0 "U21" H 3250 5550 50  0000 C CNN
+F 1 "TLV2464CDR" H 3400 5350 50  0000 C CNN
+F 2 "CarMan General Footprints:SOIC127P600X175-14N" H 3200 5650 50  0001 C CNN
+F 3 "" H 3300 5750 50  0001 C CNN
+	3    3250 5550
+	1    0    0    -1
+$EndComp
+$Comp
+L CarMan_KiCAD_Library:TLV2464CDR U?
+U 4 1 62FA2AEA
+P 3250 6675
+AR Path="/5FC85F57/62FA2AEA" Ref="U?"  Part="4"
+AR Path="/6196BF15/62FA2AEA" Ref="U21"  Part="4"
+F 0 "U21" H 3250 6675 50  0000 C CNN
+F 1 "TLV2464CDR" H 3400 6475 50  0000 C CNN
+F 2 "CarMan General Footprints:SOIC127P600X175-14N" H 3200 6775 50  0001 C CNN
+F 3 "" H 3300 6875 50  0001 C CNN
+	4    3250 6675
+	1    0    0    -1
+$EndComp
+$Comp
+L CarMan_KiCAD_Library:TLV2464CDR U?
+U 1 1 631E6F5A
+P 3700 12700
+AR Path="/5FC85F57/631E6F5A" Ref="U?"  Part="1"
+AR Path="/6196BF15/631E6F5A" Ref="U35"  Part="1"
+F 0 "U35" H 3700 12700 50  0000 C CNN
+F 1 "TLV2464CDR" H 3850 12950 50  0001 C CNN
+F 2 "CarMan General Footprints:SOIC127P600X175-14N" H 3650 12800 50  0001 C CNN
+F 3 "" H 3750 12900 50  0001 C CNN
+	1    3700 12700
+	1    0    0    -1
+$EndComp
+$Comp
+L CarMan_KiCAD_Library:TLV2464CDR U?
+U 5 1 631E6F60
+P 3700 12700
+AR Path="/5FC85F57/631E6F60" Ref="U?"  Part="5"
+AR Path="/6196BF15/631E6F60" Ref="U35"  Part="5"
+F 0 "U35" H 3650 13150 50  0001 L CNN
+F 1 "TLV2464CDR" H 3700 12550 50  0000 L CNN
+F 2 "CarMan General Footprints:SOIC127P600X175-14N" H 3650 12800 50  0001 C CNN
+F 3 "" H 3750 12900 50  0001 C CNN
+	5    3700 12700
+	1    0    0    -1
+$EndComp
 $EndSCHEMATC

Commit message: Pre-review_schematic
Parts:
- C1, C12, C2, C37, C38, C42, C5: footprint Capacitor_SMD:C_0805_2012Metric_Pad1.15x1.40mm_HandSolder -> Capacitor_SMD:C_0805_2012Metric_Pad1.18x1.45mm_HandSolder
- R100, R101, R102, R105, R106, R107, R108, R115, R116, R117, R4, R46, R47, R56, R67, R69, R72, R73: footprint Resistor_SMD:R_0805_2012Metric_Pad1.15x1.40mm_HandSolder -> Resistor_SMD:R_0805_2012Metric_Pad1.20x1.40mm_HandSolder
Changed lines of the file:
@@
 F 0 "R106" V 6350 11325 50  0000 L CNN
 F 1 "10K" V 6250 11375 50  0000 L CNN
-F 2 "Resistor_SMD:R_0805_2012Metric_Pad1.15x1.40mm_HandSolder" V 6180 11425 50  0001 C CNN
+F 2 "Resistor_SMD:R_0805_2012Metric_Pad1.20x1.40mm_HandSolder" V 6180 11425 50  0001 C CNN
 F 3 "~" H 6250 11425 50  0001 C CNN
 	1    6250 11425
@@
 F 0 "R107" V 6900 11075 50  0000 L CNN
 F 1 "1M" V 6800 11125 50  0000 L CNN
-F 2 "Resistor_SMD:R_0805_2012Metric_Pad1.15x1.40mm_HandSolder" V 6730 11175 50  0001 C CNN
+F 2 "Resistor_SMD:R_0805_2012Metric_Pad1.20x1.40mm_HandSolder" V 6730 11175 50  0001 C CNN
 F 3 "~" H 6800 11175 50  0001 C CNN
 	1    6800 11175
@@
 F 0 "C12" H 21325 13675 50  0000 C CNN
 F 1 "0.33u" H 21325 13875 50  0000 C CNN
-F 2 "Capacitor_SMD:C_0805_2012Metric_Pad1.15x1.40mm_HandSolder" H 21225 13775 50  0001 C CNN
+F 2 "Capacitor_SMD:C_0805_2012Metric_Pad1.18x1.45mm_HandSolder" H 21225 13775 50  0001 C CNN
 F 3 "~" H 21225 13775 50  0001 C CNN
 	1    21225 13775
@@
 F 0 "R46" V 19200 11925 50  0000 L CNN
 F 1 "1K" V 19100 11975 50  0000 L CNN
-F 2 "Resistor_SMD:R_0805_2012Metric_Pad1.15x1.40mm_HandSolder" V 19030 12025 50  0001 C CNN
+F 2 "Resistor_SMD:R_0805_2012Metric_Pad1.20x1.40mm_HandSolder" V 19030 12025 50  0001 C CNN
 F 3 "~" H 19100 12025 50  0001 C CNN
 	1    19100 12025
@@
 F 0 "R101" V 21000 12125 50  0000 L CNN
 F 1 "10K" V 20900 12175 50  0000 L CNN
-F 2 "Resistor_SMD:R_0805_2012Metric_Pad1.15x1.40mm_HandSolder" V 20830 12225 50  0001 C CNN
+F 2 "Resistor_SMD:R_0805_2012Metric_Pad1.20x1.40mm_HandSolder" V 20830 12225 50  0001 C CNN
 F 3 "~" H 20900 12225 50  0001 C CNN
 	1    20900 12225
@@
 F 0 "C1" H 17725 13650 50  0000 C CNN
 F 1 "0.47u" H 17725 13850 50  0000 C CNN
-F 2 "Capacitor_SMD:C_0805_2012Metric_Pad1.15x1.40mm_HandSolder" H 17625 13750 50  0001 C CNN
+F 2 "Capacitor_SMD:C_0805_2012Metric_Pad1.18x1.45mm_HandSolder" H 17625 13750 50  0001 C CNN
 F 3 "~" H 17625 13750 50  0001 C CNN
 	1    17625 13750
@@
 F 0 "R108" V 5200 11325 50  0000 L CNN
 F 1 "2.4K" V 5100 11325 50  0000 L CNN
-F 2 "Resistor_SMD:R_0805_2012Metric_Pad1.15x1.40mm_HandSolder" V 5030 11425 50  0001 C CNN
+F 2 "Resistor_SMD:R_0805_2012Metric_Pad1.20x1.40mm_HandSolder" V 5030 11425 50  0001 C CNN
 F 3 "~" H 5100 11425 50  0001 C CNN
 	1    5100 11425
@@
 F 0 "R100" V 5425 15550 50  0000 L CNN
 F 1 "5K" V 5325 15600 50  0000 L CNN
-F 2 "Resistor_SMD:R_0805_2012Metric_Pad1.15x1.40mm_HandSolder" V 5255 15650 50  0001 C CNN
+F 2 "Resistor_SMD:R_0805_2012Metric_Pad1.20x1.40mm_HandSolder" V 5255 15650 50  0001 C CNN
 F 3 "~" H 5325 15650 50  0001 C CNN
 	1    5325 15650
@@
 F 0 "R73" V 6350 13000 50  0000 L CNN
 F 1 "5K" V 6250 13050 50  0000 L CNN
-F 2 "Resistor_SMD:R_0805_2012Metric_Pad1.15x1.40mm_HandSolder" V 6180 13100 50  0001 C CNN
+F 2 "Resistor_SMD:R_0805_2012Metric_Pad1.20x1.40mm_HandSolder" V 6180 13100 50  0001 C CNN
 F 3 "~" H 6250 13100 50  0001 C CNN
 	1    6250 13100
@@
 F 0 "R105" V 4700 12250 50  0000 L CNN
 F 1 "330" V 4600 12275 50  0000 L CNN
-F 2 "Resistor_SMD:R_0805_2012Metric_Pad1.15x1.40mm_HandSolder" V 4530 12350 50  0001 C CNN
+F 2 "Resistor_SMD:R_0805_2012Metric_Pad1.20x1.40mm_HandSolder" V 4530 12350 50  0001 C CNN
 F 3 "~" H 4600 12350 50  0001 C CNN
 	1    4600 12350
@@
 F 0 "R47" V 5200 12600 50  0000 L CNN
 F 1 "499" V 5100 12625 50  0000 L CNN
-F 2 "Resistor_SMD:R_0805_2012Metric_Pad1.15x1.40mm_HandSolder" V 5030 12700 50  0001 C CNN
+F 2 "Resistor_SMD:R_0805_2012Metric_Pad1.20x1.40mm_HandSolder" V 5030 12700 50  0001 C CNN
 F 3 "~" H 5100 12700 50  0001 C CNN
 	1    5100 12700
@@
 F 0 "C2" H 4575 14100 50  0000 C CNN
 F 1 "4.7u" H 4575 14300 50  0000 C CNN
-F 2 "Capacitor_SMD:C_0805_2012Metric_Pad1.15x1.40mm_HandSolder" H 4475 14200 50  0001 C CNN
+F 2 "Capacitor_SMD:C_0805_2012Metric_Pad1.18x1.45mm_HandSolder" H 4475 14200 50  0001 C CNN
 F 3 "~" H 4475 14200 50  0001 C CNN
 	1    4475 14200
@@
 F 0 "R72" V 3550 6200 50  0000 L CNN
 F 1 "95K" V 3650 6200 50  0000 L CNN
-F 2 "Resistor_SMD:R_0805_2012Metric_Pad1.15x1.40mm_HandSolder" V 3580 6275 50  0001 C CNN
+F 2 "Resistor_SMD:R_0805_2012Metric_Pad1.20x1.40mm_HandSolder" V 3580 6275 50  0001 C CNN
 F 3 "~" H 3650 6275 50  0001 C CNN
 	1    3650 6275
@@
 F 0 "R69" V 17400 7350 50  0000 C CNN
 F 1 "499" V 17500 7350 50  0000 C CNN
-F 2 "Resistor_SMD:R_0805_2012Metric_Pad1.15x1.40mm_HandSolder" V 17430 7350 50  0001 C CNN
+F 2 "Resistor_SMD:R_0805_2012Metric_Pad1.20x1.40mm_HandSolder" V 17430 7350 50  0001 C CNN
 F 3 "~" H 17500 7350 50  0001 C CNN
 	1    17500 7350
@@
 F 0 "C38" H 14500 8350 50  0000 C CNN
 F 1 "15u" H 14500 8550 50  0000 C CNN
-F 2 "Capacitor_SMD:C_0805_2012Metric_Pad1.15x1.40mm_HandSolder" H 14400 8450 50  0001 C CNN
+F 2 "Capacitor_SMD:C_0805_2012Metric_Pad1.18x1.45mm_HandSolder" H 14400 8450 50  0001 C CNN
 F 3 "~" H 14400 8450 50  0001 C CNN
 	1    14400 8450
@@
 F 0 "R56" V 14300 7950 50  0000 C CNN
 F 1 "56K" V 14400 7950 50  0000 C CNN
-F 2 "Resistor_SMD:R_0805_2012Metric_Pad1.15x1.40mm_HandSolder" V 14330 7950 50  0001 C CNN
+F 2 "Resistor_SMD:R_0805_2012Metric_Pad1.20x1.40mm_HandSolder" V 14330 7950 50  0001 C CNN
 F 3 "~" H 14400 7950 50  0001 C CNN
 	1    14400 7950
@@
 F 0 "R4" V 14650 7150 50  0000 C CNN
 F 1 "5K" V 14750 7150 50  0000 C CNN
-F 2 "Resistor_SMD:R_0805_2012Metric_Pad1.15x1.40mm_HandSolder" V 14680 7150 50  0001 C CNN
+F 2 "Resistor_SMD:R_0805_2012Metric_Pad1.20x1.40mm_HandSolder" V 14680 7150 50  0001 C CNN
 F 3 "~" H 14750 7150 50  0001 C CNN
 	1    14750 7150
@@
 F 0 "C5" V 19000 2425 50  0000 C CNN
 F 1 "0.1u" V 19000 2125 50  0000 C CNN
-F 2 "Capacitor_SMD:C_0805_2012Metric_Pad1.15x1.40mm_HandSolder" H 19100 2275 50  0001 C CNN
+F 2 "Capacitor_SMD:C_0805_2012Metric_Pad1.18x1.45mm_HandSolder" H 19100 2275 50  0001 C CNN
 F 3 "~" H 19100 2275 50  0001 C CNN
 	1    19100 2275
@@
 F 0 "C42" V 20100 3550 50  0000 C CNN
 F 1 "0.1u" V 20100 3250 50  0000 C CNN
-F 2 "Capacitor_SMD:C_0805_2012Metric_Pad1.15x1.40mm_HandSolder" H 20200 3400 50  0001 C CNN
+F 2 "Capacitor_SMD:C_0805_2012Metric_Pad1.18x1.45mm_HandSolder" H 20200 3400 50  0001 C CNN
 F 3 "~" H 20200 3400 50  0001 C CNN
 	1    20200 3400
@@
 F 0 "C37" V 21025 2450 50  0000 C CNN
 F 1 "0.1u" V 21025 2150 50  0000 C CNN
-F 2 "Capacitor_SMD:C_0805_2012Metric_Pad1.15x1.40mm_HandSolder" H 21125 2300 50  0001 C CNN
+F 2 "Capacitor_SMD:C_0805_2012Metric_Pad1.18x1.45mm_HandSolder" H 21125 2300 50  0001 C CNN
 F 3 "~" H 21125 2300 50  0001 C CNN
 	1    21125 2300
@@
 F 0 "R67" V 15550 6250 50  0000 L CNN
 F 1 "2.4K" V 15450 6250 50  0000 L CNN
-F 2 "Resistor_SMD:R_0805_2012Metric_Pad1.15x1.40mm_HandSolder" V 15380 6325 50  0001 C CNN
+F 2 "Resistor_SMD:R_0805_2012Metric_Pad1.20x1.40mm_HandSolder" V 15380 6325 50  0001 C CNN
 F 3 "~" H 15450 6325 50  0001 C CNN
 	1    15450 6325
@@
 F 0 "R102" V 6350 15175 50  0000 L CNN
 F 1 "2.4K" V 6250 15175 50  0000 L CNN
-F 2 "Resistor_SMD:R_0805_2012Metric_Pad1.15x1.40mm_HandSolder" V 6180 15275 50  0001 C CNN
+F 2 "Resistor_SMD:R_0805_2012Metric_Pad1.20x1.40mm_HandSolder" V 6180 15275 50  0001 C CNN
 F 3 "~" H 6250 15275 50  0001 C CNN
 	1    6250 15275
@@
 F 0 "R117" V 6550 7175 50  0000 C CNN
 F 1 "2.4K" V 6625 7175 50  0000 C CNN
-F 2 "Resistor_SMD:R_0805_2012Metric_Pad1.15x1.40mm_HandSolder" V 6555 7175 50  0001 C CNN
+F 2 "Resistor_SMD:R_0805_2012Metric_Pad1.20x1.40mm_HandSolder" V 6555 7175 50  0001 C CNN
 F 3 "~" H 6625 7175 50  0001 C CNN
 	1    6625 7175
@@
 F 0 "R116" V 6275 7175 50  0000 C CNN
 F 1 "2.4K" V 6350 7175 50  0000 C CNN
-F 2 "Resistor_SMD:R_0805_2012Metric_Pad1.15x1.40mm_HandSolder" V 6280 7175 50  0001 C CNN
+F 2 "Resistor_SMD:R_0805_2012Metric_Pad1.20x1.40mm_HandSolder" V 6280 7175 50  0001 C CNN
 F 3 "~" H 6350 7175 50  0001 C CNN
 	1    6350 7175
@@
 F 0 "R115" V 6000 7175 50  0000 C CNN
 F 1 "2.4K" V 6100 7175 50  0000 C CNN
-F 2 "Resistor_SMD:R_0805_2012Metric_Pad1.15x1.40mm_HandSolder" V 6030 7175 50  0001 C CNN
+F 2 "Resistor_SMD:R_0805_2012Metric_Pad1.20x1.40mm_HandSolder" V 6030 7175 50  0001 C CNN
 F 3 "~" H 6100 7175 50  0001 C CNN
 	1    6100 7175

Commit message: removed u41 power
Parts:
- removed C42: 0.1u, Capacitor_SMD:C_0805_2012Metric_Pad1.18x1.45mm_HandSolder, symbol TSI_Rev.5-rescue:CAP-pspice
- removed U41: SN74HC00APWR, Package_SO:TSSOP-14_4.4x5mm_P0.65mm, symbol TSI_Rev.5-rescue:74HC00-74xx
Changed lines of the file:
@@
 	0    1    1    0
 $EndComp
-Text Label 19300 3000 0    47   ~ 0
-IO_Ground
 Text Label 18175 1850 0    47   ~ 0
 IO_Ground
@@
 	21625 1850 21625 2300
 Connection ~ 21625 1850
-Wire Wire Line
-	19700 3400 19950 3400
 $Comp
 L TSI_Rev.5-rescue:TestPoint-Connector TP?
@@
 Wire Wire Line
 	4600 15850 5325 15850
-Wire Wire Line
-	20700 3000 20700 3400
-Wire Wire Line
-	20700 3400 20450 3400
-Wire Wire Line
-	20700 3000 21000 3000
-$Comp
-L TSI_Rev.5-rescue:CAP-pspice C?
-U 1 1 63EC1341
-P 20200 3400
-AR Path="/5FC85F57/63EC1341" Ref="C?"  Part="1"
-AR Path="/6196BF15/63EC1341" Ref="C42"  Part="1"
-F 0 "C42" V 20100 3550 50  0000 C CNN
-F 1 "0.1u" V 20100 3250 50  0000 C CNN
-F 2 "Capacitor_SMD:C_0805_2012Metric_Pad1.18x1.45mm_HandSolder" H 20200 3400 50  0001 C CNN
-F 3 "~" H 20200 3400 50  0001 C CNN
-	1    20200 3400
-	0    -1   -1   0
-$EndComp
-Text Label 21000 3000 2    47   ~ 0
-5HV
 Text Notes 19250 1325 0    79   ~ 0
 NAND Package Power Supplies
@@
 Text Notes 7575 5475 0    197  ~ 0
 PRE-CHARGE LOGIC CIRCUIT
-Wire Notes Line
-	18075 3600 22100 3600
 Wire Notes Line
 	22100 3600 22100 1150
@@
 Wire Wire Line
 	6350 7925 6700 7925
-Connection ~ 20700 3000
-Wire Wire Line
-	19700 3000 19300 3000
-$Comp
-L TSI_Rev.5-rescue:74HC00-74xx U41
-U 5 1 63EC134F
-P 20200 3000
-AR Path="/63EC134F" Ref="U41"  Part="5"
-AR Path="/6196BF15/63EC134F" Ref="U41"  Part="5"
-F 0 "U41" V 20350 3000 50  0000 C CNN
-F 1 "SN74HC00APWR" V 19950 3000 50  0000 C CNN
-F 2 "Package_SO:TSSOP-14_4.4x5mm_P0.65mm" H 20200 3000 50  0001 C CNN
-F 3 "http://www.ti.com/lit/gpn/sn74hc00" H 20200 3000 50  0001 C CNN
-	5    20200 3000
-	0    1    1    0
-$EndComp
-Wire Wire Line
-	19700 3000 19700 3400
-Connection ~ 19700 3000
 Text Label 7100 15275 2    59   ~ 0
 PC_Control
@@
 	1    0    0    -1
 $EndComp
+Wire Notes Line
+	18075 3600 22100 3600
 $EndSCHEMATC

Commit message: TSI Post-Nadovich
Parts:
- R100: value 5K -> 10K
- R105: value 330 -> 2.4K
Connections:
- net 3.3V: now also U27.4
- net 5V: no longer U27.4
Changed lines of the file:
@@
 P 5325 15650
 F 0 "R100" V 5425 15550 50  0000 L CNN
-F 1 "5K" V 5325 15600 50  0000 L CNN
+F 1 "10K" V 5325 15575 50  0000 L CNN
 F 2 "Resistor_SMD:R_0805_2012Metric_Pad1.20x1.40mm_HandSolder" V 5255 15650 50  0001 C CNN
 F 3 "~" H 5325 15650 50  0001 C CNN
@@
 P 4600 12350
 F 0 "R105" V 4700 12250 50  0000 L CNN
-F 1 "330" V 4600 12275 50  0000 L CNN
+F 1 "2.4K" V 4600 12275 50  0000 L CNN
 F 2 "Resistor_SMD:R_0805_2012Metric_Pad1.20x1.40mm_HandSolder" V 4530 12350 50  0001 C CNN
 F 3 "~" H 4600 12350 50  0001 C CNN
@@
 	14400 8900 13900 8900
 Text Label 4600 15275 0    49   ~ 0
-5V
+3.3V
 Text Label 1850 11050 2    50   ~ 0
 5V
