File: CarMan KiCAD Schematics/TSI/TSI_Rev.7/TSI_Rev.7.kicad_pcb (KiCad board)
At the start: 2 copper layers, 203.2 x 165.1 mm, 292 parts, among them IC1 TS431ILT, IC2 TS431ILT, J1 J1 TSV, J10 J10 COOL PWR, J11 J11 GLV PWR, J12 J12 DASH/EPAL, J13 J13 BP SL, J14 J14 RSP SL, J15 J15 TSI-Logic, J16 J16 ROLL TSAL, J17 J17 THROTTLE PLAUS., J18 J18 BRAKES, J19 J19 RTDS & BRK LIGHT, J2 J2 MC, J20 J20 COOL SENSORS, J21 J21 LSP, J22 J22 I2C, J3 J3 MC Direction Switch, J4 J4 PC Relay, J5 J5 DC Relay, J6 J6 Current_Sensor, J7 J7 IMD, J8 J8 BP CAN & PWR, J9 J9 COCKPIT, K1 APAN3105, K2 G5LE-1-E, K3 SFS2-DC24V, K4 SFS2-DC24V, Q1 ZVP1320F, Q2 MMBF170, Q3 SI1302DL-T1-E3, SW1 TS5A3159DBVT, SW2 IMD RST, SW3 AMS RST, SW4 RTDS Test, U1 RDE03110S12, U10 MC7805BDTRKG, U11 TLP293, U12 REF3033, U13 TLP293, U14 Bottom Left, U15 Top Left, U16 TS372CDT, U17 Top Right, U18 MCP6004, U19 SN74HC00APWR, U2 Bottom Right, U20 TLP293, U21 MCP6004, U22 MCP23016-I_SO, U23 DAC5574IDGS, U24 TLP293, U25 NCD9830DBR2G, U26 MCP6004, U27 TLP293, U28 TLP293, U29 TLP293, U3 TS912, U30 TLP293, U31 TLP293, U32 TLP293, U33 TLP293, U34 TLP293, U35 MCP6004, U36 LT1763CS8-3.3PBF, U37 TLP293, U38 PDQ10-Q24-D5-D, U39 TLP293, U4 ACPL-C870, U40 MCP6004, U41 SN74HC00APWR, U42 SN74HC00APWR, U43 NCD9830DBR2G, U5 SI8600AB-B-IS, U6 TS912, U7 MCP6004, U8 74ACT11030, U9 STN3NF06L

Commit message: PCB_Progress
Parts:
- removed C10, C11, C15, C16, C21, C22, C24, C27, C3, C35, C37, C5, C7, C8: 0.1u, Capacitor_SMD:C_0805_2012Metric_Pad1.15x1.40mm_HandSolder
- removed C18: 10u, Capacitor_SMD:C_0805_2012Metric_Pad1.15x1.40mm_HandSolder
- removed C2: 4.7u, Capacitor_SMD:C_0805_2012Metric_Pad1.15x1.40mm_HandSolder
- removed C23: 33p, Capacitor_SMD:C_0805_2012Metric_Pad1.15x1.40mm_HandSolder
- removed C41: 100p, Capacitor_SMD:C_0805_2012Metric_Pad1.15x1.40mm_HandSolder
- removed D2: TL431PS, Package_SO:SO-8_5.3x6.2mm_P1.27mm
- removed D3: MMSZ5231B-7-F, Diode_SMD:D_SOD-123
- removed IC1: TS431ILT, TSI_Rev_2021_Footprint_Lib:SOT95P280X145-5N
- removed Q1: ZVP1320F, TSI_Rev_2021_Footprint_Lib:SOT23
- removed R1, R54, R98: 1K, Resistor_SMD:R_0805_2012Metric_Pad1.15x1.40mm_HandSolder
- removed R107: 1M, Resistor_SMD:R_0805_2012Metric_Pad1.15x1.40mm_HandSolder
- removed R109, R110: 1.5K, Resistor_SMD:R_0805_2012Metric_Pad1.15x1.40mm_HandSolder
- removed R113: 500, Resistor_SMD:R_0805_2012Metric_Pad1.15x1.40mm_HandSolder
- removed R114, R17, R18, R19, R20, R22, R23, R24, R26, R36, R37, R40, R5, R52, R62, R63, R74, R75, R8, R90, R91, R93, R94, R95, R96: 10K, Resistor_SMD:R_0805_2012Metric_Pad1.15x1.40mm_HandSolder
- removed R12, R92: 120, Resistor_SMD:R_0805_2012Metric_Pad1.15x1.40mm_HandSolder
- removed R14: 2.2K, Resistor_SMD:R_0805_2012Metric_Pad1.15x1.40mm_HandSolder
- removed R2, R33, R49, R79: 2.4K, Resistor_SMD:R_0805_2012Metric_Pad1.15x1.40mm_HandSolder
- removed R21, R27, R48: 100K, Resistor_SMD:R_0805_2012Metric_Pad1.15x1.40mm_HandSolder
- removed R28, R29: 4K, Resistor_SMD:R_0805_2012Metric_Pad1.15x1.40mm_HandSolder
- removed R30, R34: 9.31K, Resistor_SMD:R_0805_2012Metric_Pad1.15x1.40mm_HandSolder
- removed R31, R32, R35, R60: 499, Resistor_SMD:R_0805_2012Metric_Pad1.15x1.40mm_HandSolder
- removed R39: 2K, Resistor_SMD:R_0805_2012Metric_Pad1.15x1.40mm_HandSolder
- removed R41: 3.9K, Resistor_SMD:R_0805_2012Metric_Pad1.15x1.40mm_HandSolder
- removed R43: 3K, Resistor_SMD:R_0805_2012Metric_Pad1.15x1.40mm_HandSolder
- removed R57: 40K, Resistor_SMD:R_0805_2012Metric_Pad1.15x1.40mm_HandSolder
- removed R64: 24.9K, Resistor_SMD:R_0805_2012Metric_Pad1.15x1.40mm_HandSolder
- removed R71: 2.1K, Resistor_SMD:R_0805_2012Metric_Pad1.15x1.40mm_HandSolder
- removed RV2: 1K, TSI_Rev_2021_Footprint_Lib:Potentiometer
- removed U13, U28, U29, U30, U31, U32, U33, U39: TLP293, Package_SO:SOIC-4_4.55x2.6mm_P1.27mm
- removed U16: TS372CDT, TSI_Rev_2021_Footprint_Lib:SOIC127P600X175-8N
- removed U19, U41, U42: SN74HC00APWR, Package_SO:TSSOP-14_4.4x5mm_P0.65mm
- removed U21, U7: MCP6004, TSI_Rev_2021_Footprint_Lib:SOIC127P600X175-14N
- removed U22: MCP23016-I_SO, TSI_Rev_2021_Footprint_Lib:SOIC127P1030X265-28N
- removed U3, U6: TS912, TSI_Rev_2021_Footprint_Lib:SOIC127P600X175-8N
- C1, C12, C17, C19, C20, C25, C26, C28, C29, C30, C31, C32, C33, C34, C36, C38, C40, C43, C6: footprint Capacitor_SMD:C_0805_2012Metric_Pad1.15x1.40mm_HandSolder -> Capacitor_SMD:C_0805_2012Metric_Pad1.18x1.45mm_HandSolder
- J15: value J15 TSI-Logic -> J15 Testing Header
- K1: footprint TSI_Rev_2021_Footprint_Lib:RELAY_APAN3105 -> RELAY_APAN3105
- R10, R100, R101, R102, R103, R104, R105, R106, R108, R11, R115, R116, R117, R118, R119, R13, R15, R16, R25, R3, R38, R4, R42, R44, R45, R46, R47, R50, R51, R53, R55, R56, R58, R59, R6, R61, R65, R66, R67, R68, R69, R7, R70, R72, R73, R76, R77, R78, R80, R81, R82, R83, R84, R85, R86, R87, R88, R89, R9, R97, R99: footprint Resistor_SMD:R_0805_2012Metric_Pad1.15x1.40mm_HandSolder -> Resistor_SMD:R_0805_2012Metric_Pad1.20x1.40mm_HandSolder
- R111, R112: value 10K -> 10k; footprint Resistor_SMD:R_0805_2012Metric_Pad1.15x1.40mm_HandSolder -> Resistor_SMD:R_0805_2012Metric_Pad1.20x1.40mm_HandSolder
- SW1: footprint TSI_Rev_2021_Footprint_Lib:SOT95P280X145-6N -> SOT95P280X145-6N
- U18, U26, U35, U40: value MCP6004 -> TLV2464CDR; footprint TSI_Rev_2021_Footprint_Lib:SOIC127P600X175-14N -> CarMan General Footprints:SOIC127P600X175-14N
- U23: footprint TSI_Rev_2021_Footprint_Lib:DAC5574IDGS -> CarMan General Footprints:SOP50P490X110-10N
Connections:
- net /Throttle_Plausibility/Throttle_PL renamed /Throttle_PL
- net /Throttle_Plausibility/Throttle_SEL renamed /Throttle_EN
- C43 pad 1: /IO_Ground -> /AIRS-
- C43 pad 2: /5HV -> /3.3V
- IC2 pad 1: (no net) -> Net-(IC2-Pad1)
- IC2 pad 2: (no net) -> Net-(IC2-Pad2)
- J12 pad 8: (no net) -> Net-(J12-Pad8)
- J14 pad 4: (no net) -> Net-(J14-Pad4)
- J15 pad 1: /Cooling_CTRL -> /Test_Pin0
- J15 pad 10: (no net) -> /Test_Pin9
- J15 pad 2: /SDA -> /Test_Pin1
- J15 pad 3: /SR_CTRL -> /Test_Pin2
- J15 pad 4: /SCL -> /Test_Pin3
- J15 pad 5: /BP_CAN- -> /Test_Pin4
- J15 pad 6: /3.3V_ISO -> /Test_Pin5
- J15 pad 7: /BP_CAN+ -> /Test_Pin6
- J15 pad 8: /LOGIC_ISO_RTN -> /Test_Pin7
- J15 pad 9: /Flowrate_LOGIC -> /Test_Pin8
- J2 pad 4: (no net) -> Net-(J2-Pad4)
- J2 pad 8: (no net) -> Net-(J2-Pad8)
- J20 pad 4: /CoolTemp -> /CoolTemp_In
- J20 pad 5: /CoolTemp_In -> /AIRS-
- J20 pad 6: /AIRS- -> Net-(J20-Pad6)
- J3 pad 4: (no net) -> Net-(J3-Pad4)
- J6 pad 1: (no net) -> Net-(J6-Pad1)
- J6 pad 6: (no net) -> Net-(J6-Pad6)
- J7 pad 6: (no net) -> Net-(J7-Pad6)
- J7 pad 7: (no net) -> Net-(J7-Pad7)
- J9 pad 4: (no net) -> Net-(J9-Pad4)
- JP1 pad 1: Net-(JP1-Pad1) -> /Throttle_Plausibility/APPS2_b
- JP1 pad 3: /Throttle_Plausibility/Pedal_Out -> /Throttle_LOGIC
- JP9 pad 2: /Relays_Cooling_Voltage_Refs/Cooling_power -> /Cooling_CTRL
- K2 pad 3: (no net) -> Net-(K2-Pad3)
- K3 pad 3: (no net) -> Net-(K3-Pad3)
- K3 pad 4: (no net) -> Net-(K3-Pad4)
- K4 pad 3: (no net) -> Net-(K4-Pad3)
- K4 pad 4: (no net) -> Net-(K4-Pad4)
- PS1 pad 4: (no net) -> Net-(PS1-Pad4)
- PS1 pad 6: (no net) -> Net-(PS1-Pad6)
- PS2 pad 2: /Relays_Cooling_Voltage_Refs/Cooling_power -> /Cooling_CTRL
- PS2 pad 6: (no net) -> Net-(PS2-Pad6)
- R111 pad 2: /SDA -> /SCL
- R112 pad 1: /SCL -> /5V
- R112 pad 2: /5V -> /SDA
- RV3 pad 3: (no net) -> Net-(RV3-Pad3)
- SW1 pad 1: Net-(JP1-Pad2) -> /Throttle_Plausibility/Pedal_Out
- U18 pad 12: (no net) -> Net-(U18-Pad12)
- U18 pad 13: (no net) -> Net-(R126-Pad1)
- U18 pad 14: (no net) -> /Throttle_LOGIC
- U18 pad 9: Net-(R103-Pad2) -> Net-(R124-Pad2)
- U23 pad 1: Net-(JP1-Pad1) -> Net-(U18-Pad12)
- U23 pad 2: (no net) -> Net-(U23-Pad2)
- U23 pad 4: (no net) -> Net-(U23-Pad4)
- U23 pad 5: (no net) -> Net-(U23-Pad5)
- U23 pad 8: /5V -> /3.3V
- U23 pad 9: /5V -> /3.3V
- U25 pad 1: (no net) -> Net-(U25-Pad1)
- U25 pad 2: (no net) -> Net-(U25-Pad2)
- U25 pad 3: (no net) -> Net-(U25-Pad3)
- U25 pad 6: (no net) -> Net-(U25-Pad6)
- U35 pad 4: /3.3V -> /5V
- U38 pad 6: (no net) -> Net-(U38-Pad6)
- U40 pad 5: Net-(U21-Pad13) -> Net-(RV1-Pad2)
- U40 pad 6: Net-(RV1-Pad2) -> Net-(U21-Pad13)
- U43 pad 14: /SCL -> /Status_Lights_TSAL_RTDS/SCL_5V
- U43 pad 15: /SDA -> /Status_Lights_TSAL_RTDS/SDA_5V
- U43 pad 3: (no net) -> Net-(U43-Pad3)
- U43 pad 4: (no net) -> Net-(U43-Pad4)
- U43 pad 5: (no net) -> Net-(U43-Pad5)
- U43 pad 6: (no net) -> Net-(U43-Pad6)
- U43 pad 7: (no net) -> Net-(U43-Pad7)
- U43 pad 8: (no net) -> Net-(U43-Pad8)
- U5 pad 8: /5V -> /3.3V
- U8 pad 12: /Throttle_Plausibility/U8_Pin12 -> /APPS1_ISO_NG
- U8 pad 13: /Throttle_Plausibility/U8_Pin13 -> /APPS2_ISO_NS
- U8 pad 14: /Throttle_Plausibility/U8_Pin14 -> /APPS2_ISO_NG
- U8 pad 3: /Throttle_Plausibility/U8_Pin3 -> /APPS_WIN1
- U8 pad 8: /Throttle_Plausibility/U8_Pin8 -> /APPS_WIN2
- U8 pad 9: /Throttle_Plausibility/U8_Pin9 -> /APPS1_ISO_NS
Routing:
- net /5V: track 732.3 -> 433.8 mm, vias 23 -> 9
- net /SDA: track 364.7 -> 78.0 mm, vias 9 -> 1
- net /SCL: track 367.0 -> 85.2 mm, vias 5 -> 2
- net /LOGIC_ISO_RTN: track 276.3 -> 0.00 mm, vias 5 -> 0
- net /AIRS-: track 409.3 -> 179.3 mm, vias 88 -> 33
- net /24V: track 546.7 -> 331.9 mm, vias 4 -> 0
- net /10V: track 256.7 -> 63.7 mm, vias 9 -> 1
- net /Throttle_Plausibility/Brake_Pressed_uC: track 155.4 -> 0.00 mm, vias 2 -> 0
- net /Throttle_Plausibility/APPS1_b: track 192.2 -> 40.1 mm, vias 10 -> 2
- net /Throttle_Plausibility/AMS_FAULT: track 144.0 -> 0.00 mm, vias 4 -> 0
- net /SR_CTRL: track 251.3 -> 113.2 mm, vias 8 -> 1
- net /Throttle_Plausibility/IMD_FAULT: track 136.0 -> 0.00 mm, vias 2 -> 0
- net /APPS2: track 133.2 -> 0.00 mm
- net /Flowrate: track 133.8 -> 1.89 mm
- net /APPS1: track 117.8 -> 9.66 mm, vias 2 -> 0
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Other:
- board text removed: "5V->3.3V"
- board text removed: "AMS 24V->5V"
- board text removed: "Flowrate Iso"
- board text removed: "GPIO"
- board text removed: "IMD 24V->5V"
- board text removed: "NAND"
- board text removed: "Precharge State Logic"
- board text removed: "SLOOP EPAL"
- board text removed: "SR Control"
- board text removed: "Shield/Chassis"
