File: CarMan KiCAD Schematics/TSI/TSI_Rev.7/TSI_Rev.7.kicad_pcb (KiCad board)
At the start: 2 copper layers, 203.2 x 165.1 mm, 292 parts, among them IC1 TS431ILT, IC2 TS431ILT, J1 J1 TSV, J10 J10 COOL PWR, J11 J11 GLV PWR, J12 J12 DASH/EPAL, J13 J13 BP SL, J14 J14 RSP SL, J15 J15 TSI-Logic, J16 J16 ROLL TSAL, J17 J17 THROTTLE PLAUS., J18 J18 BRAKES, J19 J19 RTDS & BRK LIGHT, J2 J2 MC, J20 J20 COOL SENSORS, J21 J21 LSP, J22 J22 I2C, J3 J3 MC Direction Switch, J4 J4 PC Relay, J5 J5 DC Relay, J6 J6 Current_Sensor, J7 J7 IMD, J8 J8 BP CAN & PWR, J9 J9 COCKPIT, K1 APAN3105, K2 G5LE-1-E, K3 SFS2-DC24V, K4 SFS2-DC24V, Q1 ZVP1320F, Q2 MMBF170, Q3 SI1302DL-T1-E3, SW1 TS5A3159DBVT, SW2 IMD RST, SW3 AMS RST, SW4 RTDS Test, U1 RDE03110S12, U10 MC7805BDTRKG, U11 TLP293, U12 REF3033, U13 TLP293, U14 Bottom Left, U15 Top Left, U16 TS372CDT, U17 Top Right, U18 MCP6004, U19 SN74HC00APWR, U2 Bottom Right, U20 TLP293, U21 MCP6004, U22 MCP23016-I_SO, U23 DAC5574IDGS, U24 TLP293, U25 NCD9830DBR2G, U26 MCP6004, U27 TLP293, U28 TLP293, U29 TLP293, U3 TS912, U30 TLP293, U31 TLP293, U32 TLP293, U33 TLP293, U34 TLP293, U35 MCP6004, U36 LT1763CS8-3.3PBF, U37 TLP293, U38 PDQ10-Q24-D5-D, U39 TLP293, U4 ACPL-C870, U40 MCP6004, U41 SN74HC00APWR, U42 SN74HC00APWR, U43 NCD9830DBR2G, U5 SI8600AB-B-IS, U6 TS912, U7 MCP6004, U8 74ACT11030, U9 STN3NF06L

Commit message: Updated Schematic and removed extra footprints from PCB. Ready to begin routing new elements in.
Parts:
- removed C23: 33p, Capacitor_SMD:C_0805_2012Metric_Pad1.15x1.40mm_HandSolder
- removed C24: 0.1u, Capacitor_SMD:C_0805_2012Metric_Pad1.15x1.40mm_HandSolder
- removed JP1: Jumper_NC_Dual, Connector_PinHeader_2.54mm:PinHeader_1x03_P2.54mm_Vertical
- removed R109, R110: 1.5K, Resistor_SMD:R_0805_2012Metric_Pad1.15x1.40mm_HandSolder
- removed R2, R79: 2.4K, Resistor_SMD:R_0805_2012Metric_Pad1.15x1.40mm_HandSolder
- removed R30: 9.31K, Resistor_SMD:R_0805_2012Metric_Pad1.15x1.40mm_HandSolder
- removed R31, R60: 499, Resistor_SMD:R_0805_2012Metric_Pad1.15x1.40mm_HandSolder
- removed R41: 3.9K, Resistor_SMD:R_0805_2012Metric_Pad1.15x1.40mm_HandSolder
- removed R48: 100K, Resistor_SMD:R_0805_2012Metric_Pad1.15x1.40mm_HandSolder
- removed R57: 40K, Resistor_SMD:R_0805_2012Metric_Pad1.15x1.40mm_HandSolder
- removed R71: 2.1K, Resistor_SMD:R_0805_2012Metric_Pad1.15x1.40mm_HandSolder
- removed R75: 10K, Resistor_SMD:R_0805_2012Metric_Pad1.15x1.40mm_HandSolder
- removed TP12: TSAL_LV, TestPoint:TestPoint_Pad_D3.0mm
- removed TP18: Pedal Out, TestPoint:TestPoint_Pad_D3.0mm
- removed TP19: PC_Control, TestPoint:TestPoint_Pad_D3.0mm
- removed TP4: TSV_Ready, TestPoint:TestPoint_Pad_D3.0mm
- removed TP5: MC_95%, TestPoint:TestPoint_Pad_D3.0mm
- removed TP6: SLOOP_HV, TestPoint:TestPoint_Pad_D3.0mm
- removed U22: MCP23016-I_SO, TSI_Rev_2021_Footprint_Lib:SOIC127P1030X265-28N
- removed U23: DAC5574IDGS, TSI_Rev_2021_Footprint_Lib:DAC5574IDGS
- removed U29, U31, U33, U39: TLP293, Package_SO:SOIC-4_4.55x2.6mm_P1.27mm
- removed U41: SN74HC00APWR, Package_SO:TSSOP-14_4.4x5mm_P0.65mm
- added C39: 0.1u, Capacitor_SMD:C_0805_2012Metric_Pad1.18x1.45mm_HandSolder, F.Cu at (385.7, 109.8)
- added C44: 0.1u, Capacitor_SMD:C_0805_2012Metric_Pad1.18x1.45mm_HandSolder, F.Cu at (338.8, 117.2)
- added C45: 0.1u, Capacitor_SMD:C_0805_2012Metric_Pad1.18x1.45mm_HandSolder, F.Cu at (353.3, 108.8)
- added C46: 0.1u, Capacitor_SMD:C_0805_2012Metric_Pad1.18x1.45mm_HandSolder, F.Cu at (343.6, 117.2)
- added C47: 0.1u, Capacitor_SMD:C_0805_2012Metric_Pad1.18x1.45mm_HandSolder, F.Cu at (361.2, 102.6)
- added C48: 0.1u, Capacitor_SMD:C_0805_2012Metric_Pad1.18x1.45mm_HandSolder, F.Cu at (353.3, 111.8)
- added C49: 0.1u, Capacitor_SMD:C_0805_2012Metric_Pad1.18x1.45mm_HandSolder, F.Cu at (358.1, 108.8)
- added C50: 0.1u, Capacitor_SMD:C_0805_2012Metric_Pad1.18x1.45mm_HandSolder, F.Cu at (343.9, 194.9)
- added C51: 0.1u, Capacitor_SMD:C_0805_2012Metric_Pad1.18x1.45mm_HandSolder, F.Cu at (418.9, 76.7)
- added C52: 0.1u, Capacitor_SMD:C_0805_2012Metric_Pad1.18x1.45mm_HandSolder, F.Cu at (397.3, 102.0)
- added C53: 0.1u, Capacitor_SMD:C_0805_2012Metric_Pad1.18x1.45mm_HandSolder, F.Cu at (405.3, 95.8)
- added J23: J23 Pickit Programming, Connector_PinHeader_2.54mm:PinHeader_1x05_P2.54mm_Vertical, F.Cu at (340.1, 78.5)
- added J24: J24 UART, Connector_PinHeader_2.54mm:PinHeader_1x03_P2.54mm_Vertical, F.Cu at (398.6, 108.7)
- added J25: J25 PI SHIELD, TSI_Rev_2021_Footprint_Lib:Molex_MiniFit-JR-5556-04A_2x02x4.20mm_Straight, F.Cu at (363.3, 78.5)
- added J27: CAN 120 Terminator, Connector_PinHeader_2.54mm:PinHeader_1x02_P2.54mm_Vertical, F.Cu at (355.9, 78.5)
- added J28: J28 TSAL & Pedal_Out TP, Connector_PinHeader_2.54mm:PinHeader_1x03_P2.54mm_Vertical, F.Cu at (384.5, 123.3)
- added J29: PC Test Points, Connector_PinHeader_2.54mm:PinHeader_1x05_P2.54mm_Vertical, F.Cu at (85.5, 181.2)
- added L1: 28nH, Inductor_SMD:L_0805_2012Metric_Pad1.15x1.40mm_HandSolder, F.Cu at (362.9, 108.6)
- added R120: 10K, Resistor_SMD:R_0805_2012Metric_Pad1.20x1.40mm_HandSolder, F.Cu at (358.1, 111.8)
- added R121: 1K, Resistor_SMD:R_0805_2012Metric_Pad1.20x1.40mm_HandSolder, F.Cu at (353.3, 114.8)
- added R122: 120, Resistor_SMD:R_0805_2012Metric_Pad1.20x1.40mm_HandSolder, F.Cu at (338.7, 89.8)
- added R123: 1K, Resistor_SMD:R_0805_2012Metric_Pad1.20x1.40mm_HandSolder, F.Cu at (366.0, 102.6)
- added R124: 1.8K, Resistor_SMD:R_0805_2012Metric_Pad1.20x1.40mm_HandSolder, F.Cu at (380.0, 116.3)
- added R125: 3.3K, Resistor_SMD:R_0805_2012Metric_Pad1.20x1.40mm_HandSolder, F.Cu at (375.3, 116.3)
- added R126: 1.8K, Resistor_SMD:R_0805_2012Metric_Pad1.20x1.40mm_HandSolder, F.Cu at (348.4, 117.2)
- added R127: 3.3K, Resistor_SMD:R_0805_2012Metric_Pad1.20x1.40mm_HandSolder, F.Cu at (361.2, 105.6)
- added U44: PIC32MZ2048EFM064-I_PT, QFP50P1200X1200X120-64N, F.Cu at (343.6, 108.4)
- added U45: MCP2551-I_SN, SOIC127P600X175-8N, F.Cu at (354.9, 104.2)
- added U46: SI8600AB-B-IS, TSI_Rev_2021_Footprint_Lib:SOIC127P600X175-8N, F.Cu at (398.9, 97.4)
- added U47: MCP23008-ESS, Package_SO:SSOP-20_5.3x7.2mm_P0.65mm, F.Cu at (370.7, 126.2)
- C1, C10, C11, C12, C15, C16, C17, C18, C19, C2, C20, C21, C22, C25, C26, C27, C28, C29, C3, C30, C31, C32, C33, C34, C35, C36, C37, C38, C40, C41, C43, C5, C6, C7, C8: footprint Capacitor_SMD:C_0805_2012Metric_Pad1.15x1.40mm_HandSolder -> Capacitor_SMD:C_0805_2012Metric_Pad1.18x1.45mm_HandSolder
- D2: footprint Package_SO:SO-8_5.3x6.2mm_P1.27mm -> Package_SO:MSOP-8_3x3mm_P0.65mm
- J15: value J15 TSI-Logic -> J15 PIC Test Pins; footprint Connector_PinSocket_2.54mm:PinSocket_2x05_P2.54mm_Vertical -> Connector_PinHeader_2.54mm:PinHeader_2x05_P2.54mm_Vertical
- J22: footprint Connector_PinSocket_2.54mm:PinSocket_1x04_P2.54mm_Vertical -> Connector_PinHeader_2.54mm:PinHeader_1x04_P2.54mm_Vertical
- JP4: value Testing Jumper -> MC Power Testing Jumper
- JP5: value Testing Jumper -> PC Relay Testing Jumper
- JP9: footprint Connector_PinSocket_2.54mm:PinSocket_1x02_P2.54mm_Vertical -> Connector_PinHeader_2.54mm:PinHeader_1x02_P2.54mm_Vertical
- R1, R10, R101, R102, R103, R104, R106, R107, R108, R11, R115, R116, R117, R118, R119, R12, R13, R14, R15, R16, R17, R18, R19, R20, R21, R22, R23, R24, R25, R26, R27, R28, R29, R3, R32, R33, R34, R35, R36, R37, R38, R39, R4, R40, R42, R43, R44, R45, R46, R47, R5, R52, R53, R54, R55, R56, R58, R59, R6, R61, R62, R63, R64, R65, R66, R67, R69, R7, R70, R72, R73, R74, R76, R77, R78, R8, R80, R81, R82, R83, R84, R85, R86, R87, R88, R89, R9, R90, R91, R92, R93, R94, R95, R96, R99: footprint Resistor_SMD:R_0805_2012Metric_Pad1.15x1.40mm_HandSolder -> Resistor_SMD:R_0805_2012Metric_Pad1.20x1.40mm_HandSolder
- R100: value 5K -> 10K; footprint Resistor_SMD:R_0805_2012Metric_Pad1.15x1.40mm_HandSolder -> Resistor_SMD:R_0805_2012Metric_Pad1.20x1.40mm_HandSolder
- R105: value 330 -> 2.4K; footprint Resistor_SMD:R_0805_2012Metric_Pad1.15x1.40mm_HandSolder -> Resistor_SMD:R_0805_2012Metric_Pad1.20x1.40mm_HandSolder
- R111, R112, R114, R50, R51: value 10K -> 4.7K; footprint Resistor_SMD:R_0805_2012Metric_Pad1.15x1.40mm_HandSolder -> Resistor_SMD:R_0805_2012Metric_Pad1.20x1.40mm_HandSolder
- R113: value 500 -> 4.7K; footprint Resistor_SMD:R_0805_2012Metric_Pad1.15x1.40mm_HandSolder -> Resistor_SMD:R_0805_2012Metric_Pad1.20x1.40mm_HandSolder
- R49: value 2.4K -> 10K; footprint Resistor_SMD:R_0805_2012Metric_Pad1.15x1.40mm_HandSolder -> Resistor_SMD:R_0805_2012Metric_Pad1.20x1.40mm_HandSolder
- R68: value 10K -> 100K; footprint Resistor_SMD:R_0805_2012Metric_Pad1.15x1.40mm_HandSolder -> Resistor_SMD:R_0805_2012Metric_Pad1.20x1.40mm_HandSolder
- R97: value 10K -> 1K; footprint Resistor_SMD:R_0805_2012Metric_Pad1.15x1.40mm_HandSolder -> Resistor_SMD:R_0805_2012Metric_Pad1.20x1.40mm_HandSolder
- R98: value 1K -> 10K; footprint Resistor_SMD:R_0805_2012Metric_Pad1.15x1.40mm_HandSolder -> Resistor_SMD:R_0805_2012Metric_Pad1.20x1.40mm_HandSolder
- SW1: footprint TSI_Rev_2021_Footprint_Lib:SOT95P280X145-6N -> SOT95P280X145-6N
- U16: footprint TSI_Rev_2021_Footprint_Lib:SOIC127P600X175-8N -> SOIC127P600X175-8N
- U18, U21, U26, U35, U40, U7: value MCP6004 -> TLV2464CDR; footprint TSI_Rev_2021_Footprint_Lib:SOIC127P600X175-14N -> CarMan General Footprints:SOIC127P600X175-14N
- moved C43 248.5 mm to (385.9, 115.1)
- moved R113 140.9 mm to (337.3, 124.1)
- moved R114 140.0 mm to (342.1, 124.1)
- moved C6 71.7 mm to (358.3, 118.8), turned to 0 degrees
- moved R108 4.67 mm to (218.7, 161.4), turned to 180 degrees
- moved R97 0.34 mm to (287.0, 103.2), turned to 270 degrees
- moved C25 0.23 mm to (236.0, 140.0), turned to 180 degrees
- turned R116 to 270 degrees
Connections:
- net /Throttle_Plausibility/Brake_Pressed_uC renamed /Brake_Pressed_uC
- net /Throttle_Plausibility/Throttle_PL renamed /Throttle_PL
- net /Throttle_Plausibility/Throttle_SEL renamed /Throttle_EN
- net /Throttle_Plausibility/U8_Pin12 renamed /Throttle_Plausibility/APPS1_ISO_NG
- net /Throttle_Plausibility/U8_Pin13 renamed /Throttle_Plausibility/APPS2_ISO_NS
- net /Throttle_Plausibility/U8_Pin14 renamed /Throttle_Plausibility/APPS2_ISO_NG
- net /Throttle_Plausibility/U8_Pin3 renamed /Throttle_Plausibility/APPS_WIN1
- net /Throttle_Plausibility/U8_Pin8 renamed /Throttle_Plausibility/APPS_WIN2
- net /Throttle_Plausibility/U8_Pin9 renamed /Throttle_Plausibility/APPS1_ISO_NS
- C25 pad 1: /AIRS- -> /5V
- C25 pad 2: /5V -> /AIRS-
- C43 pad 1: /IO_Ground -> /AIRS-
- C43 pad 2: /5HV -> /3.3V
- C6 pad 1: /AIRS- -> /Drive_BTN_LOGIC
- C6 pad 2: /5V -> /AIRS-
- IC1 pad 1: (no net) -> Net-(IC1-Pad1)
- IC1 pad 2: (no net) -> Net-(IC1-Pad2)
- IC2 pad 1: (no net) -> Net-(IC2-Pad1)
- IC2 pad 2: (no net) -> Net-(IC2-Pad2)
- J12 pad 8: (no net) -> Net-(J12-Pad8)
- J14 pad 4: (no net) -> Net-(J14-Pad4)
- J15 pad 1: /Cooling_CTRL -> /Test_Pin0
- J15 pad 10: (no net) -> /Test_Pin9
- J15 pad 2: /SDA -> /Test_Pin1
- J15 pad 3: /SR_CTRL -> /Test_Pin2
- J15 pad 4: /SCL -> /Test_Pin3
- J15 pad 5: /BP_CAN- -> /Test_Pin4
- J15 pad 6: /3.3V_ISO -> /Test_Pin5
- J15 pad 7: /BP_CAN+ -> /Test_Pin6
- J15 pad 8: /LOGIC_ISO_RTN -> /Test_Pin7
- J15 pad 9: /Flowrate_LOGIC -> /Test_Pin8
- J2 pad 4: (no net) -> Net-(J2-Pad4)
- J2 pad 8: (no net) -> Net-(J2-Pad8)
- J20 pad 4: /CoolTemp -> /CoolTemp_In
- J20 pad 5: /CoolTemp_In -> /AIRS-
- J20 pad 6: /AIRS- -> Net-(J20-Pad6)
- J22 pad 3: /5V -> /3.3V
- J3 pad 4: (no net) -> Net-(J3-Pad4)
- J6 pad 1: (no net) -> Net-(J6-Pad1)
- J6 pad 6: (no net) -> Net-(J6-Pad6)
- J7 pad 6: (no net) -> Net-(J7-Pad6)
- J7 pad 7: (no net) -> Net-(J7-Pad7)
- J9 pad 4: (no net) -> Net-(J9-Pad4)
- JP9 pad 2: /Relays_Cooling_Voltage_Refs/Cooling_power -> /Cooling_CTRL
- K2 pad 3: (no net) -> Net-(K2-Pad3)
- K3 pad 3: (no net) -> Net-(K3-Pad3)
- K3 pad 4: (no net) -> Net-(K3-Pad4)
- K4 pad 3: (no net) -> Net-(K4-Pad3)
- K4 pad 4: (no net) -> Net-(K4-Pad4)
- PS1 pad 4: (no net) -> Net-(PS1-Pad4)
- PS1 pad 6: (no net) -> Net-(PS1-Pad6)
- PS2 pad 2: /Relays_Cooling_Voltage_Refs/Cooling_power -> /Cooling_CTRL
- PS2 pad 6: (no net) -> Net-(PS2-Pad6)
- R111 pad 1: /5V -> /3.3V
- R111 pad 2: /SDA -> /SCL
- R112 pad 1: /SCL -> /3.3V
- R112 pad 2: /5V -> /SDA
- R113 pad 1: Net-(R113-Pad1) -> /SDA_5V
- R113 pad 2: /Flowrate -> /5V
- R114 pad 1: /LOGIC_ISO_RTN -> /5V
- R114 pad 2: /Flowrate_LOGIC -> /SCL_5V
- R32 pad 2: Net-(R32-Pad2) -> /Throttle_Plausibility/4.76V_REF
- R34 pad 1: Net-(R32-Pad2) -> /Throttle_Plausibility/4.76V_REF
- R34 pad 2: Net-(R34-Pad2) -> /Throttle_Plausibility/0.24V_REF
- R35 pad 1: Net-(R34-Pad2) -> /Throttle_Plausibility/0.24V_REF
- R68 pad 1: Net-(R68-Pad1) -> /Drive_BTN_LOGIC
- R68 pad 2: /5V -> /3.3V
- R97 pad 1: Net-(R68-Pad1) -> /Drive_BTN
- R97 pad 2: /Drive_BTN -> /Drive_BTN_LOGIC
- RV3 pad 3: (no net) -> Net-(RV3-Pad3)
- SW1 pad 1: Net-(JP1-Pad2) -> /Pedal_Out
- U18 pad 1: /Throttle_Plausibility/Pedal_Out -> /Pedal_Out
- U18 pad 10: /Throttle_Plausibility/Pedal_Out -> /Pedal_Out
- U18 pad 2: /Throttle_Plausibility/Pedal_Out -> /Pedal_Out
- U18 pad 9: Net-(R103-Pad2) -> /Throttle_Plausibility/0.24V_REF
- U19 pad 11: Net-(U19-Pad11) -> (no net)
- U19 pad 12: Net-(U19-Pad12) -> (no net)
- U19 pad 13: Net-(U19-Pad12) -> (no net)
- U19 pad 8: Net-(U19-Pad12) -> Net-(U19-Pad8)
- U25 pad 1: (no net) -> Net-(U25-Pad1)
- U25 pad 2: (no net) -> Net-(U25-Pad2)
- U25 pad 3: (no net) -> Net-(U25-Pad3)
- U25 pad 6: (no net) -> Net-(U25-Pad6)
- U27 pad 4: /5V -> /3.3V
- U30 pad 4: /5V -> /3.3V
- U32 pad 2: /LOGIC_ISO_RTN -> /PI_SHIELD_RTN
- U35 pad 4: /3.3V -> /5V
- U38 pad 6: (no net) -> Net-(U38-Pad6)
- U40 pad 5: Net-(U21-Pad13) -> Net-(RV1-Pad2)
- U40 pad 6: Net-(RV1-Pad2) -> Net-(U21-Pad13)
- U42 pad 1: Net-(U41-Pad8) -> (no net)
- U42 pad 10: /PCDC_Circuit/PC_Control -> Net-(U42-Pad10)
- U42 pad 11: /PCDC_Circuit/PC_Control -> Net-(U42-Pad10)
- U42 pad 12: Net-(U42-Pad12) -> /PCDC_Circuit/PC_Control
- U42 pad 13: Net-(U42-Pad13) -> /PCDC_Circuit/Safety_Loop_HV
- U42 pad 2: Net-(U41-Pad11) -> (no net)
- U42 pad 3: Net-(U42-Pad3) -> (no net)
- U42 pad 4: Net-(U42-Pad3) -> (no net)
- U42 pad 5: Net-(U42-Pad3) -> (no net)
- U42 pad 6: Net-(U42-Pad13) -> (no net)
- U42 pad 8: Net-(U42-Pad12) -> /PCDC_Circuit/PC_Control
- U42 pad 9: Net-(U42-Pad3) -> Net-(U19-Pad8)
- U43 pad 14: /SCL -> /SCL_5V
- U43 pad 15: /SDA -> /SDA_5V
- U43 pad 3: (no net) -> Net-(U43-Pad3)
- U43 pad 4: (no net) -> Net-(U43-Pad4)
- U43 pad 5: (no net) -> Net-(U43-Pad5)
- U43 pad 6: (no net) -> Net-(U43-Pad6)
- U43 pad 7: (no net) -> Net-(U43-Pad7)
- U43 pad 8: (no net) -> Net-(U43-Pad8)
- U5 pad 8: /5V -> /3.3V
- U7 pad 10: Net-(R32-Pad2) -> /Throttle_Plausibility/4.76V_REF
- U7 pad 13: Net-(R34-Pad2) -> /Throttle_Plausibility/0.24V_REF
- U7 pad 3: Net-(R30-Pad1) -> /Throttle_Plausibility/4.76V_REF
- U7 pad 6: Net-(R30-Pad2) -> /Throttle_Plausibility/0.24V_REF
Routing:
- net /SCL: track 367.0 -> 0.00 mm, vias 5 -> 0
- net /SDA: track 364.7 -> 0.00 mm, vias 9 -> 0
- net /5V: track 732.3 -> 445.1 mm, vias 23 -> 16
- net /LOGIC_ISO_RTN: track 276.3 -> 0.00 mm, vias 5 -> 0
- net /SR_CTRL: track 251.3 -> 0.00 mm, vias 8 -> 0
- net /PC_Ready: track 169.0 -> 4.63 mm, vias 6 -> 0
- net /Brake_Pressed_uC: track 155.4 -> 3.01 mm, vias 2 -> 0
- net /Throttle_Plausibility/AMS_FAULT: track 144.0 -> 0.00 mm, vias 4 -> 0
- net /Throttle_EN: track 138.7 -> 2.59 mm, vias 2 -> 0
- net /Throttle_Plausibility/IMD_FAULT: track 136.0 -> 0.00 mm, vias 2 -> 0
- net /Flowrate: track 133.8 -> 0.00 mm, vias 1 -> 0
- net /RTDS_CTRL: track 130.1 -> 0.00 mm, vias 2 -> 0
- net /Cooling_CTRL: track 118.5 -> 0.00 mm, vias 3 -> 0
- net /AIRS-: track 409.3 -> 292.9 mm, vias 88 -> 57
- net /AMS_FAULT_LED: track 101.3 -> 0.00 mm, vias 1 -> 0
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Other:
- board text added: "BOT & SCADA OK"
- board text added: "FW"
- board text added: "RW"
- board text removed: "AMS 24V->5V"
- board text removed: "Flowrate Iso"
- board text removed: "IMD 24V->5V"
- board text removed: "MRESET_Coil"

Commit message: Finished PCB for REV7
Parts:
- added G***: LOGO, TSI_Rev_2021_Footprint_Lib:logo_lafayette_ece_medium_24mmx9mm, F.Cu at (129.2, 104.5)
- added G***: LOGO, Lafayette_Electric_Car_Footprints:highvoltage, F.Cu at (260.2, 179.9)
- added VAL: REF, CarMan General Footprints:lafLogo, F.Cu at (250.4, 151.5)
- moved C51 197.2 mm to (241.0, 161.6)
- moved J24 180.1 mm to (226.1, 56.7), turned to 270 degrees
- moved J28 176.5 mm to (208.1, 116.3), turned to 90 degrees
- moved J27 155.0 mm to (201.0, 77.1)
- moved C53 154.0 mm to (252.3, 78.3), turned to 270 degrees
- moved C52 153.4 mm to (245.5, 79.5)
- moved J25 151.1 mm to (212.9, 64.4), turned to 180 degrees
- moved U46 148.4 mm to (251.2, 83.3)
- moved J22 145.6 mm to (269.2, 63.7)
- moved C39 132.0 mm to (260.4, 68.2), turned to 270 degrees
- moved U47 131.7 mm to (253.6, 66.0), turned to 180 degrees
- moved R122 130.1 mm to (209.5, 75.5)
- moved R123 121.6 mm to (244.9, 113.8), turned to 90 degrees
- moved C43 120.4 mm to (268.2, 89.8), turned to 0 degrees
- moved L1 110.6 mm to (258.4, 72.5)
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Routing:
- net /3.3V: track 211.7 -> 539.2 mm, vias 4 -> 23
- net /PC_Ready: track 4.63 -> 200.2 mm, vias 0 -> 12
- net /BP_CAN+: track 0.00 -> 170.4 mm, vias 0 -> 8
- net /SR_CTRL: track 0.00 -> 163.7 mm, vias 0 -> 2
- net /PI_SHIELD_RTN: track 0.00 -> 162.8 mm, vias 0 -> 2
- net /BP_CAN-: track 0.00 -> 160.9 mm, vias 0 -> 6
- net /RTDS_CTRL: track 0.00 -> 158.5 mm, vias 0 -> 8
- net /Brake_Pressed_uC: track 3.01 -> 159.3 mm, vias 0 -> 4
- net /SDA: track 0.00 -> 141.3 mm, vias 0 -> 6
- net /SCL: track 0.00 -> 139.2 mm, vias 0 -> 8
- net /Throttle_EN: track 2.59 -> 102.8 mm, vias 0 -> 8
- net /Throttle_Plausibility/APPS1_b: track 192.2 -> 101.5 mm, vias 10 -> 5
- net /Cooling_CTRL: track 0.00 -> 82.5 mm, vias 0 -> 5
- net /AIRS-: track 292.9 -> 374.8 mm, vias 57 -> 85
- net /AMS_FAULT_LED: track 0.00 -> 78.4 mm, vias 0 -> 2
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Other:
- net class Default: clearance 0.199 -> 0.225
- rule trace_clearance: 0.199 -> 0.225
- rule trace_min: 0.2 -> 0
- board text added: "AIRS- 3.3V SCL SDA"
- board text added: "CAN 120 Terminator"
- board text added: "Eli Crippen & Marwa Saleh"
- board text added: "GLV_RTN"
- board text added: "IO_Ground"
- board text added: "PC_Control"
- board text added: "PI Shield"
- board text added: "PIC Programming"
- board text added: "PIC Test Pins"
- board text added: "Pedl_Out"
- board text added: "REV 7"
- board text added: "Sfty_Loop_HV"
- board text added: "TSAL"
- board text added: "TSI Revision 7 - 3/11/22"
- board text added: "TSI Version 7 Eli Crippen, Marwa Saleh"
- board text added: "TSV_Ready"
- board text added: "UART RX TX"
- board text removed: "TSI Revision 6 - 4/27/21"
- board text removed: "TSI Version 6 John Burk, Ethan Miller, Nate Beal, Zack Martin & Troy Coleman"
- board text removed: "Zacky Bear Doesn't Like"
- board text removed: "amogus burk"
- board text removed: "zack"
