File: CarMan KiCAD Schematics/TSI/TSI_Rev.7/Sensors-Throttle.sch (KiCad schematic (older format))
At the start: 52 parts, among them IC2 TS431ILT, U21 MCP6004, U25 NCD9830DBR2G, U26 MCP6004, U4 ACPL-C870, U40 MCP6004, U5 SI8600AB-B-IS

Commit message: TSI Should be final schematic
Parts:
- removed R111, R112: 10K, Resistor_SMD:R_0805_2012Metric_Pad1.15x1.40mm_HandSolder, symbol TSI_Rev.5-rescue:R-Device
- removed U21, U26, U40: MCP6004, TSI_Rev_2021_Footprint_Lib:SOIC127P600X175-14N, symbol TSI_Rev.5-rescue:MCP6004-Amplifier_Operational
- added C50, C51: 0.1u, Capacitor_SMD:C_0805_2012Metric_Pad1.18x1.45mm_HandSolder, symbol Device:C
- added U21, U26, U40: TLV2464CDR, CarMan General Footprints:SOIC127P600X175-14N, symbol CarMan_KiCAD_Library:TLV2464CDR
Connections:
- net 5HV: now also C50.2, U21.4 (V+), U26.4 (V+)
- net 5V: no longer U5.8 (BVDD)
- net GLV_RTN: now also C51.1
- net IO_Ground: now also C50.1, U21.11 (V-), U26.11 (V-)
- net MC_Voltage: now also U21.7
- net TS_Voltage: now also U21.1
- net Throttle_HV: now also U40.8
- net at JP7.1, R53.2, R78.2: now also U26.5 (+)
- net at R93.1: now also U26.6 (-), U26.7
- net at JP8.1, R16.2, R76.2: now also U26.10 (+)
- net at R94.1, R96.1: now also U26.8, U26.9 (-)
- net at R104.2, R95.2: now also U21.5 (+)
- net at R89.1, R96.2: now also U21.6 (-)
- net at R90.1, R94.2: now also U21.2 (-)
- net at R91.2, R93.2: now also U21.3 (+)
- net at C41.2, R62.1, R64.2: now also U40.10 (+)
- net at R95.1: now also U26.13 (-), U26.14
- net at JP6.1, R6.2, R7.2: now also U26.12 (+)
- net at C40.2, R63.1, R66.2: now also U40.9 (-)
- new net 3.3V: C51.2, U5.8 (BVDD)
Other:
- note added: "From simulation- Lowpass cutoff: 268kHz"

Commit message: Pre-review_schematic
Parts:
- C20, C21, C30, C32, C35, C40, C41: footprint Capacitor_SMD:C_0805_2012Metric_Pad1.15x1.40mm_HandSolder -> Capacitor_SMD:C_0805_2012Metric_Pad1.18x1.45mm_HandSolder
- R10, R104, R13, R16, R50, R51, R53, R58, R59, R6, R62, R63, R64, R66, R7, R70, R76, R77, R78, R84, R85, R86, R87, R88, R89, R9, R90, R91, R93, R94, R95, R96: footprint Resistor_SMD:R_0805_2012Metric_Pad1.15x1.40mm_HandSolder -> Resistor_SMD:R_0805_2012Metric_Pad1.20x1.40mm_HandSolder

Commit message: TSI Post-Nadovich
Parts:
- R50, R51: value 10K -> 4.7K
Changed lines of the file:
@@
 $Descr A3 16535 11693
 encoding utf-8
-Sheet 7 7
+Sheet 6 7
 Title ""
 Date ""
@@
 P 5850 5700
 F 0 "R51" H 5920 5746 50  0000 L CNN
-F 1 "10K" H 5920 5655 50  0000 L CNN
+F 1 "4.7K" H 5920 5655 50  0000 L CNN
 F 2 "Resistor_SMD:R_0805_2012Metric_Pad1.20x1.40mm_HandSolder" V 5780 5700 50  0001 C CNN
 F 3 "~" H 5850 5700 50  0001 C CNN
@@
 P 5850 5250
 F 0 "R50" H 5780 5204 50  0000 R CNN
-F 1 "10K" H 5780 5295 50  0000 R CNN
+F 1 "4.7K" H 5780 5295 50  0000 R CNN
 F 2 "Resistor_SMD:R_0805_2012Metric_Pad1.20x1.40mm_HandSolder" V 5780 5250 50  0001 C CNN
 F 3 "~" H 5850 5250 50  0001 C CNN
