File: CarMan KiCAD Schematics/TSI/TSI_Rev.7/CAN_GLV_POWER.sch (KiCad schematic (older format))
At the start: 46 parts, among them K2 G5LE-1-E, K3 SFS2-DC24V, K4 SFS2-DC24V, U14 Bottom Left, U15 Top Left, U17 Top Right, U2 Bottom Right, U20 TLP293, U24 TLP293, U28 TLP293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

Commit message: Pre-review_schematic
Parts:
- C18, C19, C28, C29, C31, C33, C34, C36: footprint Capacitor_SMD:C_0805_2012Metric_Pad1.15x1.40mm_HandSolder -> Capacitor_SMD:C_0805_2012Metric_Pad1.18x1.45mm_HandSolder
- R25, R33, R45, R52, R54, R55, R61, R65, R80, R81, R82, R83, R92: footprint Resistor_SMD:R_0805_2012Metric_Pad1.15x1.40mm_HandSolder -> Resistor_SMD:R_0805_2012Metric_Pad1.20x1.40mm_HandSolder
Changed lines of the file:
@@
 F 0 "C34" H 1900 4900 50  0000 L CNN
 F 1 "10u" H 1850 4700 50  0000 L CNN
-F 2 "Capacitor_SMD:C_0805_2012Metric_Pad1.15x1.40mm_HandSolder" H 1850 4800 50  0001 C CNN
+F 2 "Capacitor_SMD:C_0805_2012Metric_Pad1.18x1.45mm_HandSolder" H 1850 4800 50  0001 C CNN
 F 3 "~" H 1850 4800 50  0001 C CNN
 	1    1850 4800
@@
 F 0 "C33" H 4700 5300 50  0000 L CNN
 F 1 "0.1u" H 4700 5100 50  0000 L CNN
-F 2 "Capacitor_SMD:C_0805_2012Metric_Pad1.15x1.40mm_HandSolder" H 4700 5200 50  0001 C CNN
+F 2 "Capacitor_SMD:C_0805_2012Metric_Pad1.18x1.45mm_HandSolder" H 4700 5200 50  0001 C CNN
 F 3 "~" H 4700 5200 50  0001 C CNN
 	1    4700 5200
@@
 F 0 "C31" H 5400 5550 50  0000 L CNN
 F 1 "1u" H 5400 5350 50  0000 L CNN
-F 2 "Capacitor_SMD:C_0805_2012Metric_Pad1.15x1.40mm_HandSolder" H 5350 5450 50  0001 C CNN
+F 2 "Capacitor_SMD:C_0805_2012Metric_Pad1.18x1.45mm_HandSolder" H 5350 5450 50  0001 C CNN
 F 3 "~" H 5350 5450 50  0001 C CNN
 	1    5350 5450
@@
 F 0 "C29" H 5900 5350 50  0000 L CNN
 F 1 "0.01u" H 5850 5150 50  0000 L CNN
-F 2 "Capacitor_SMD:C_0805_2012Metric_Pad1.15x1.40mm_HandSolder" H 6100 5250 50  0001 C CNN
+F 2 "Capacitor_SMD:C_0805_2012Metric_Pad1.18x1.45mm_HandSolder" H 6100 5250 50  0001 C CNN
 F 3 "~" H 6100 5250 50  0001 C CNN
 	1    6100 5250
@@
 F 0 "R92" V 13400 6425 50  0000 C CNN
 F 1 "120" V 13500 6425 50  0000 C CNN
-F 2 "Resistor_SMD:R_0805_2012Metric_Pad1.15x1.40mm_HandSolder" V 13430 6425 50  0001 C CNN
+F 2 "Resistor_SMD:R_0805_2012Metric_Pad1.20x1.40mm_HandSolder" V 13430 6425 50  0001 C CNN
 F 3 "~" H 13500 6425 50  0001 C CNN
 	1    13500 6425
@@
 F 0 "R45" V 11100 1200 50  0000 C CNN
 F 1 "2.4K" V 11200 1200 50  0000 C CNN
-F 2 "Resistor_SMD:R_0805_2012Metric_Pad1.15x1.40mm_HandSolder" V 11130 1200 50  0001 C CNN
+F 2 "Resistor_SMD:R_0805_2012Metric_Pad1.20x1.40mm_HandSolder" V 11130 1200 50  0001 C CNN
 F 3 "~" H 11200 1200 50  0001 C CNN
 	1    11200 1200
@@
 F 0 "R55" V 12250 1550 50  0000 C CNN
 F 1 "2.4K" V 12350 1550 50  0000 C CNN
-F 2 "Resistor_SMD:R_0805_2012Metric_Pad1.15x1.40mm_HandSolder" V 12280 1550 50  0001 C CNN
+F 2 "Resistor_SMD:R_0805_2012Metric_Pad1.20x1.40mm_HandSolder" V 12280 1550 50  0001 C CNN
 F 3 "~" H 12350 1550 50  0001 C CNN
 	1    12350 1550
@@
 F 0 "R52" H 14625 6275 50  0000 L CNN
 F 1 "10K" V 14575 6200 50  0000 L CNN
-F 2 "Resistor_SMD:R_0805_2012Metric_Pad1.15x1.40mm_HandSolder" V 14505 6250 50  0001 C CNN
+F 2 "Resistor_SMD:R_0805_2012Metric_Pad1.20x1.40mm_HandSolder" V 14505 6250 50  0001 C CNN
 F 3 "~" H 14575 6250 50  0001 C CNN
 	1    14575 6250
@@
 F 0 "C18" H 5890 2496 50  0000 L CNN
 F 1 "10u" H 5890 2405 50  0000 L CNN
-F 2 "Capacitor_SMD:C_0805_2012Metric_Pad1.15x1.40mm_HandSolder" H 5813 2300 50  0001 C CNN
+F 2 "Capacitor_SMD:C_0805_2012Metric_Pad1.18x1.45mm_HandSolder" H 5813 2300 50  0001 C CNN
 F 3 "~" H 5775 2450 50  0001 C CNN
 	1    5775 2450
@@
 F 0 "R25" V 11325 3325 50  0000 C CNN
 F 1 "2.4K" V 11425 3325 50  0000 C CNN
-F 2 "Resistor_SMD:R_0805_2012Metric_Pad1.15x1.40mm_HandSolder" V 11355 3325 50  0001 C CNN
+F 2 "Resistor_SMD:R_0805_2012Metric_Pad1.20x1.40mm_HandSolder" V 11355 3325 50  0001 C CNN
 F 3 "~" H 11425 3325 50  0001 C CNN
 	1    11425 3325
@@
 F 0 "R61" V 12200 3050 50  0000 L CNN
 F 1 "1.5K" V 12300 3025 50  0000 L CNN
-F 2 "Resistor_SMD:R_0805_2012Metric_Pad1.15x1.40mm_HandSolder" V 12230 3100 50  0001 C CNN
+F 2 "Resistor_SMD:R_0805_2012Metric_Pad1.20x1.40mm_HandSolder" V 12230 3100 50  0001 C CNN
 F 3 "~" H 12300 3100 50  0001 C CNN
 	1    12300 3100
@@
 F 0 "R83" V 13900 7250 50  0000 C CNN
 F 1 "1.2K" V 13975 7250 50  0000 C CNN
-F 2 "Resistor_SMD:R_0805_2012Metric_Pad1.15x1.40mm_HandSolder" V 13905 7250 50  0001 C CNN
+F 2 "Resistor_SMD:R_0805_2012Metric_Pad1.20x1.40mm_HandSolder" V 13905 7250 50  0001 C CNN
 F 3 "~" H 13975 7250 50  0001 C CNN
 	1    13975 7250
@@
 F 0 "C19" H 8700 1775 50  0000 L CNN
 F 1 "0.1u" H 8700 1575 50  0000 L CNN
-F 2 "Capacitor_SMD:C_0805_2012Metric_Pad1.15x1.40mm_HandSolder" H 8700 1675 50  0001 C CNN
+F 2 "Capacitor_SMD:C_0805_2012Metric_Pad1.18x1.45mm_HandSolder" H 8700 1675 50  0001 C CNN
 F 3 "~" H 8700 1675 50  0001 C CNN
 	1    8700 1675
@@
 F 0 "R65" H 8170 1121 50  0000 L CNN
 F 1 "2K" V 8100 1025 50  0000 L CNN
-F 2 "Resistor_SMD:R_0805_2012Metric_Pad1.15x1.40mm_HandSolder" V 8030 1075 50  0001 C CNN
+F 2 "Resistor_SMD:R_0805_2012Metric_Pad1.20x1.40mm_HandSolder" V 8030 1075 50  0001 C CNN
 F 3 "~" H 8100 1075 50  0001 C CNN
 	1    8100 1075
@@
 F 0 "R80" H 8170 1521 50  0000 L CNN
 F 1 "1.6K" V 8100 1375 50  0000 L CNN
-F 2 "Resistor_SMD:R_0805_2012Metric_Pad1.15x1.40mm_HandSolder" V 8030 1475 50  0001 C CNN
+F 2 "Resistor_SMD:R_0805_2012Metric_Pad1.20x1.40mm_HandSolder" V 8030 1475 50  0001 C CNN
 F 3 "~" H 8100 1475 50  0001 C CNN
 	1    8100 1475
@@
 F 0 "R33" V 11100 2100 50  0000 C CNN
 F 1 "2.4K" V 11200 2100 50  0000 C CNN
-F 2 "Resistor_SMD:R_0805_2012Metric_Pad1.15x1.40mm_HandSolder" V 11130 2100 50  0001 C CNN
+F 2 "Resistor_SMD:R_0805_2012Metric_Pad1.20x1.40mm_HandSolder" V 11130 2100 50  0001 C CNN
 F 3 "~" H 11200 2100 50  0001 C CNN
 	1    11200 2100
@@
 F 0 "R54" V 12250 2450 50  0000 C CNN
 F 1 "1K" V 12350 2450 50  0000 C CNN
-F 2 "Resistor_SMD:R_0805_2012Metric_Pad1.15x1.40mm_HandSolder" V 12280 2450 50  0001 C CNN
+F 2 "Resistor_SMD:R_0805_2012Metric_Pad1.20x1.40mm_HandSolder" V 12280 2450 50  0001 C CNN
 F 3 "~" H 12350 2450 50  0001 C CNN
 	1    12350 2450
@@
 F 0 "C28" H 8150 5500 50  0000 L CNN
 F 1 "10u" H 8150 5300 50  0000 L CNN
-F 2 "Capacitor_SMD:C_0805_2012Metric_Pad1.15x1.40mm_HandSolder" H 8100 5400 50  0001 C CNN
+F 2 "Capacitor_SMD:C_0805_2012Metric_Pad1.18x1.45mm_HandSolder" H 8100 5400 50  0001 C CNN
 F 3 "~" H 8100 5400 50  0001 C CNN
 	1    8100 5400
@@
 F 0 "C36" H 1350 4900 50  0000 L CNN
 F 1 "10u" H 1350 4700 50  0000 L CNN
-F 2 "Capacitor_SMD:C_0805_2012Metric_Pad1.15x1.40mm_HandSolder" H 1350 4800 50  0001 C CNN
+F 2 "Capacitor_SMD:C_0805_2012Metric_Pad1.18x1.45mm_HandSolder" H 1350 4800 50  0001 C CNN
 F 3 "~" H 1350 4800 50  0001 C CNN
 	1    1350 4800
@@
 F 0 "R81" V 2775 10225 50  0000 C CNN
 F 1 "1.2K" V 2850 10225 50  0000 C CNN
-F 2 "Resistor_SMD:R_0805_2012Metric_Pad1.15x1.40mm_HandSolder" V 2780 10225 50  0001 C CNN
+F 2 "Resistor_SMD:R_0805_2012Metric_Pad1.20x1.40mm_HandSolder" V 2780 10225 50  0001 C CNN
 F 3 "~" H 2850 10225 50  0001 C CNN
 	1    2850 10225
@@
 F 0 "R82" V 8025 10275 50  0000 C CNN
 F 1 "1.2K" V 8100 10275 50  0000 C CNN
-F 2 "Resistor_SMD:R_0805_2012Metric_Pad1.15x1.40mm_HandSolder" V 8030 10275 50  0001 C CNN
+F 2 "Resistor_SMD:R_0805_2012Metric_Pad1.20x1.40mm_HandSolder" V 8030 10275 50  0001 C CNN
 F 3 "~" H 8100 10275 50  0001 C CNN
 	1    8100 10275

Commit message: TSI Post-Nadovich
Parts:
- added R124: 1.8K, Resistor_SMD:R_0805_2012Metric_Pad1.20x1.40mm_HandSolder, symbol TSI_Rev.5-rescue:R-Device
- added R125: 3.3K, Resistor_SMD:R_0805_2012Metric_Pad1.20x1.40mm_HandSolder, symbol TSI_Rev.5-rescue:R-Device
Connections:
- net labels added: Flowrate, Flowrate_LOGIC, Flowrate_RTN
- wire segments 189 -> 197
Other:
- note added: "5V-3.3V Voltage Divider"
Changed lines of the file:
@@
 Wire Wire Line
 	3625 2450 4175 2450
-Text Notes 2825 1950 0    49   ~ 0
+Text Notes 4200 1775 0    49   ~ 0
 DC/DC Converter 24V to 12V 10A
 Text Label 2375 2750 0    49   ~ 0
@@
 Text Label 15800 2700 2    50   ~ 0
 PI_SHIELD_RTN
+Text Label 15800 3800 2    50   ~ 0
+Flowrate_LOGIC
+Text HLabel 14950 3800 0    50   Output ~ 0
+Flowrate_LOGIC
+Wire Wire Line
+	14950 3800 15800 3800
+Text Label 2700 725  0    50   ~ 0
+Flowrate
+Text Label 3300 1225 0    50   ~ 0
+Flowrate_LOGIC
+$Comp
+L TSI_Rev.5-rescue:R-Device R?
+U 1 1 633D6F1E
+P 2700 1025
+AR Path="/633D6F1E" Ref="R?"  Part="1"
+AR Path="/5FE1DE7D/633D6F1E" Ref="R124"  Part="1"
+F 0 "R124" H 2770 1071 50  0000 L CNN
+F 1 "1.8K" V 2700 950 50  0000 L CNN
+F 2 "Resistor_SMD:R_0805_2012Metric_Pad1.20x1.40mm_HandSolder" V 2630 1025 50  0001 C CNN
+F 3 "~" H 2700 1025 50  0001 C CNN
+	1    2700 1025
+	1    0    0    -1
+$EndComp
+$Comp
+L TSI_Rev.5-rescue:R-Device R?
+U 1 1 633D6F24
+P 2700 1425
+AR Path="/633D6F24" Ref="R?"  Part="1"
+AR Path="/5FE1DE7D/633D6F24" Ref="R125"  Part="1"
+F 0 "R125" H 2770 1471 50  0000 L CNN
+F 1 "3.3K" V 2700 1325 50  0000 L CNN
+F 2 "Resistor_SMD:R_0805_2012Metric_Pad1.20x1.40mm_HandSolder" V 2630 1425 50  0001 C CNN
+F 3 "~" H 2700 1425 50  0001 C CNN
+	1    2700 1425
+	1    0    0    -1
+$EndComp
+Wire Wire Line
+	2700 1275 2700 1225
+Connection ~ 2700 1225
+Wire Wire Line
+	2700 1225 2700 1175
+Wire Wire Line
+	2700 1225 3300 1225
+Wire Wire Line
+	2700 1575 2700 1725
+Text Label 2700 1725 0    50   ~ 0
+Flowrate_RTN
+Wire Wire Line
+	2700 725  2700 875
+Text Notes 3150 1525 0    50   ~ 0
+5V-3.3V Voltage Divider
+Wire Wire Line
+	14950 2800 15800 2800
+Text HLabel 14950 2800 0    50   Input ~ 0
+Flowrate
+Text Label 15800 2800 2    50   ~ 0
+Flowrate
+Wire Wire Line
+	14950 2900 15800 2900
+Text HLabel 14950 2900 0    50   Input ~ 0
+Flowrate_RTN
+Text Label 15800 2900 2    50   ~ 0
+Flowrate_RTN
 $EndSCHEMATC

Commit message: Updated Schematic and removed extra footprints from PCB. Ready to begin routing new elements in.
Parts:
- JP9: footprint Connector_PinSocket_2.54mm:PinSocket_1x02_P2.54mm_Vertical -> Connector_PinHeader_2.54mm:PinHeader_1x02_P2.54mm_Vertical
Changed lines of the file:
@@
 F 0 "JP9" H 6725 1000 50  0000 R CNN
 F 1 "If CAN_Shield & Chassis_GND need to be shorted together, weren't sure" H 7350 850 50  0001 R CNN
-F 2 "Connector_PinSocket_2.54mm:PinSocket_1x02_P2.54mm_Vertical" H 6650 850 50  0001 C CNN
+F 2 "Connector_PinHeader_2.54mm:PinHeader_1x02_P2.54mm_Vertical" H 6650 850 50  0001 C CNN
 F 3 "~" H 6650 850 50  0001 C CNN
 	1    6650 850
