File: CarMan KiCAD Schematics/TSI/TSI_Rev.7/TSI_Rev.7.sch (KiCad schematic (older format))
At the start: 41 parts, among them J1 J1 TSV, J10 J10 COOL PWR, J11 J11 GLV PWR, J12 J12 DASH/EPAL, J13 J13 BP SL, J14 J14 RSP SL, J15 J15 Testing Header, J16 J16 ROLL TSAL, J17 J17 THROTTLE PLAUS., J18 J18 BRAKES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

Commit message: TSI Should be final schematic
Parts:
- R11, R118, R119, R122, R14: footprint Resistor_SMD:R_0805_2012Metric_Pad1.15x1.40mm_HandSolder -> Resistor_SMD:R_0805_2012Metric_Pad1.20x1.40mm_HandSolder

Commit message: TSI Post-Nadovich
Other:
- moved on the sheet: J20

Commit message: TSI REV7 Final Schematic before Layout
Parts:
- renumbered J26 to J27
Connections:
- net 3.3V: now also J22.3 (Pin_3)
- net 5V: no longer J22.3 (Pin_3)
Changed lines of the file:
@@
 AIRS+
 Text Label 2725 2700 0    49   ~ 0
-5V
+3.3V
 Wire Wire Line
 	2725 2500 3175 2500
@@
 $EndComp
 $Comp
-L TSI_Rev.5-rescue:Conn_01x02-Connector_Generic J26
+L TSI_Rev.5-rescue:Conn_01x02-Connector_Generic J27
 U 1 1 62B2D611
 P 7525 1200
-F 0 "J26" H 7475 1300 50  0000 L CNN
+F 0 "J27" H 7475 1300 50  0000 L CNN
 F 1 "J16 ROLL TSAL" H 7475 1300 50  0001 L CNN
 F 2 "TSI_Rev_2021_Footprint_Lib:Molex_MiniFit-JR-5556-02A_2x01x4.20mm_Straight" H 7525 1200 50  0001 C CNN

Commit message: Updated Schematic and removed extra footprints from PCB. Ready to begin routing new elements in.
Parts:
- added J28: J28 TSAL & Pedal_Out TP, Connector_PinHeader_2.54mm:PinHeader_1x03_P2.54mm_Vertical, symbol TSI_Rev.5-rescue:Conn_01x03-Connector_Generic
- J15: value J15 Testing Header -> J15 PIC Test Pins; footprint Connector_PinSocket_2.54mm:PinSocket_2x05_P2.54mm_Vertical -> Connector_PinHeader_2.54mm:PinHeader_2x05_P2.54mm_Vertical
- J22: footprint Connector_PinSocket_2.54mm:PinSocket_1x04_P2.54mm_Vertical -> Connector_PinHeader_2.54mm:PinHeader_1x04_P2.54mm_Vertical
- J23: value J17 THROTTLE PLAUS. -> J23 Pickit Programming; footprint TSI_Rev_2021_Footprint_Lib:Molex_MiniFit-JR-5556-06A_2x03x4.20mm_Straight -> Connector_PinHeader_2.54mm:PinHeader_1x05_P2.54mm_Vertical; symbol TSI_Rev.5-rescue:Conn_01x06-Connector_Generic -> Connector_Generic:Conn_01x05
- J24: value J22 I2C -> J24 UART; footprint Connector_PinSocket_2.54mm:PinSocket_1x04_P2.54mm_Vertical -> Connector_PinHeader_2.54mm:PinHeader_1x03_P2.54mm_Vertical; symbol TSI_Rev.5-rescue:Conn_01x04-Connector_Generic -> TSI_Rev.5-rescue:Conn_01x03-Connector_Generic
- J25: value J14 RSP SL -> J25 PI SHIELD
- J27: value J16 ROLL TSAL -> CAN 120 Terminator; footprint TSI_Rev_2021_Footprint_Lib:Molex_MiniFit-JR-5556-02A_2x01x4.20mm_Straight -> Connector_PinHeader_2.54mm:PinHeader_1x02_P2.54mm_Vertical
Connections:
- net AIRS-: now also J28.3 (Pin_3)
- net TSAL: now also J28.1 (Pin_1)
- new net Pedal_Out: J28.2 (Pin_2)
- no-connect marks 13 -> 11
Other:
- note added: "PIC Testing Header"
- note added: "TSAL and Pedal_Out TP"
- note removed: "Testing Header"
- moved on the sheet: JP10, JP11, JP12, JP13, JP14, JP15, SW2, SW3
