File: CarMan KiCAD Schematics/TSI/TSI_Rev.7/PIC32.sch (KiCad schematic (older format))
At the start: 13 parts, among them U44 PIC32MZ2048EFM064-I_PT, U45 MCP2551-I_SN

Commit message: TSI Should be final schematic
Parts:
- added R111, R112: 10k, Resistor_SMD:R_0805_2012Metric_Pad1.20x1.40mm_HandSolder, symbol Device:R
- C43, C44, C45, C46, C47, C48, C49: footprint Capacitor_SMD:C_0805_2012Metric_Pad1.15x1.40mm_HandSolder -> Capacitor_SMD:C_0805_2012Metric_Pad1.18x1.45mm_HandSolder
- R120, R121, R123: footprint Resistor_SMD:R_0805_2012Metric_Pad1.15x1.40mm_HandSolder -> Resistor_SMD:R_0805_2012Metric_Pad1.20x1.40mm_HandSolder
Connections:
- net 5V: now also R111.1, R112.1
- net SCL: now also R111.2
- net SDA: now also R112.2
- net Throttle_SEL renamed Throttle_EN
Other:
- note added: "NS=Not Shorted\nNG=Not Grounded"
Changed lines of the file:
@@
 $Descr A4 11693 8268
 encoding utf-8
-Sheet 7 7
+Sheet 6 7
 Title ""
 Date ""
@@
 Wire Wire Line
 	2550 4300 2050 4300
-Wire Wire Line
-	2550 3200 2050 3200
 Text Label 6700 3200 2    39   ~ 0
 CAN_TXD
@@
 Text Label 2050 3600 0    39   ~ 0
 APPS2_ISO_NS
-Wire Wire Line
-	2550 3100 2050 3100
 Text Label 2050 3100 0    39   ~ 0
 SCL
@@
 Test_Pin9
 Text Label 6700 4100 2    39   ~ 0
-Throttle_SEL
+Throttle_EN
 Text Label 2050 2700 0    39   ~ 0
 Test_Pin6
@@
 RTDS_CTRL
 Text HLabel 8725 2675 0    39   Output ~ 0
-Throttle_SEL
+Throttle_EN
 Text HLabel 8725 2750 0    39   Output ~ 0
 Throttle_LOGIC
@@
 F 0 "R123" V 10000 4850 50  0000 C CNN
 F 1 "1K" V 9900 4850 50  0000 C CNN
-F 2 "Resistor_SMD:R_0805_2012Metric_Pad1.15x1.40mm_HandSolder" V 9830 4850 50  0001 C CNN
+F 2 "Resistor_SMD:R_0805_2012Metric_Pad1.20x1.40mm_HandSolder" V 9830 4850 50  0001 C CNN
 F 3 "~" H 9900 4850 50  0001 C CNN
 	1    9900 4850
@@
 F 0 "R121" V 2225 2300 50  0000 C CNN
 F 1 "1K" V 2300 2300 50  0000 C CNN
-F 2 "Resistor_SMD:R_0805_2012Metric_Pad1.15x1.40mm_HandSolder" V 2230 2300 50  0001 C CNN
+F 2 "Resistor_SMD:R_0805_2012Metric_Pad1.20x1.40mm_HandSolder" V 2230 2300 50  0001 C CNN
 F 3 "~" H 2300 2300 50  0001 C CNN
 	1    2300 2300
@@
 F 0 "R120" V 1925 2050 50  0000 C CNN
 F 1 "10K" V 2000 2050 50  0000 C CNN
-F 2 "Resistor_SMD:R_0805_2012Metric_Pad1.15x1.40mm_HandSolder" V 1930 2050 50  0001 C CNN
+F 2 "Resistor_SMD:R_0805_2012Metric_Pad1.20x1.40mm_HandSolder" V 1930 2050 50  0001 C CNN
 F 3 "~" H 2000 2050 50  0001 C CNN
 	1    2000 2050
@@
 F 0 "C49" V 1400 2150 50  0000 C CNN
 F 1 "0.1u" V 1400 2450 50  0000 C CNN
-F 2 "Capacitor_SMD:C_0805_2012Metric_Pad1.15x1.40mm_HandSolder" H 1500 2300 50  0001 C CNN
+F 2 "Capacitor_SMD:C_0805_2012Metric_Pad1.18x1.45mm_HandSolder" H 1500 2300 50  0001 C CNN
 F 3 "~" H 1500 2300 50  0001 C CNN
 	1    1500 2300
@@
 F 0 "C43" V 3050 1225 50  0000 C CNN
 F 1 "0.1u" V 3050 1525 50  0000 C CNN
-F 2 "Capacitor_SMD:C_0805_2012Metric_Pad1.15x1.40mm_HandSolder" H 3150 1375 50  0001 C CNN
+F 2 "Capacitor_SMD:C_0805_2012Metric_Pad1.18x1.45mm_HandSolder" H 3150 1375 50  0001 C CNN
 F 3 "~" H 3150 1375 50  0001 C CNN
 	1    3150 1375
@@
 F 0 "C44" V 3650 1225 50  0000 C CNN
 F 1 "0.1u" V 3650 1525 50  0000 C CNN
-F 2 "Capacitor_SMD:C_0805_2012Metric_Pad1.15x1.40mm_HandSolder" H 3750 1375 50  0001 C CNN
+F 2 "Capacitor_SMD:C_0805_2012Metric_Pad1.18x1.45mm_HandSolder" H 3750 1375 50  0001 C CNN
 F 3 "~" H 3750 1375 50  0001 C CNN
 	1    3750 1375
@@
 F 0 "C45" V 4250 1225 50  0000 C CNN
 F 1 "0.1u" V 4250 1525 50  0000 C CNN
-F 2 "Capacitor_SMD:C_0805_2012Metric_Pad1.15x1.40mm_HandSolder" H 4350 1375 50  0001 C CNN
+F 2 "Capacitor_SMD:C_0805_2012Metric_Pad1.18x1.45mm_HandSolder" H 4350 1375 50  0001 C CNN
 F 3 "~" H 4350 1375 50  0001 C CNN
 	1    4350 1375
@@
 F 0 "C46" V 4850 1225 50  0000 C CNN
 F 1 "0.1u" V 4850 1525 50  0000 C CNN
-F 2 "Capacitor_SMD:C_0805_2012Metric_Pad1.15x1.40mm_HandSolder" H 4950 1375 50  0001 C CNN
+F 2 "Capacitor_SMD:C_0805_2012Metric_Pad1.18x1.45mm_HandSolder" H 4950 1375 50  0001 C CNN
 F 3 "~" H 4950 1375 50  0001 C CNN
 	1    4950 1375
@@
 F 0 "C47" V 5450 1225 50  0000 C CNN
 F 1 "0.1u" V 5450 1525 50  0000 C CNN
-F 2 "Capacitor_SMD:C_0805_2012Metric_Pad1.15x1.40mm_HandSolder" H 5550 1375 50  0001 C CNN
+F 2 "Capacitor_SMD:C_0805_2012Metric_Pad1.18x1.45mm_HandSolder" H 5550 1375 50  0001 C CNN
 F 3 "~" H 5550 1375 50  0001 C CNN
 	1    5550 1375
@@
 F 0 "C48" V 6900 3700 50  0000 C CNN
 F 1 "0.1u" V 6900 4000 50  0000 C CNN
-F 2 "Capacitor_SMD:C_0805_2012Metric_Pad1.15x1.40mm_HandSolder" H 7000 3850 50  0001 C CNN
+F 2 "Capacitor_SMD:C_0805_2012Metric_Pad1.18x1.45mm_HandSolder" H 7000 3850 50  0001 C CNN
 F 3 "~" H 7000 3850 50  0001 C CNN
 	1    7000 3850
@@
 Wire Wire Line
 	4950 1625 4950 1800
+Wire Wire Line
+	1550 3100 2550 3100
+Wire Wire Line
+	1550 3200 2550 3200
+$Comp
+L Device:R R111
+U 1 1 6241050D
+P 1550 2950
+F 0 "R111" H 1620 2996 50  0000 L CNN
+F 1 "10k" H 1620 2905 50  0000 L CNN
+F 2 "Resistor_SMD:R_0805_2012Metric_Pad1.20x1.40mm_HandSolder" V 1480 2950 50  0001 C CNN
+F 3 "~" H 1550 2950 50  0001 C CNN
+	1    1550 2950
+	1    0    0    -1
+$EndComp
+Wire Wire Line
+	1550 2800 1550 2700
+Wire Wire Line
+	1550 2700 1325 2700
+$Comp
+L Device:R R112
+U 1 1 624149A2
+P 1550 3350
+F 0 "R112" H 1481 3304 50  0000 R CNN
+F 1 "10k" H 1481 3395 50  0000 R CNN
+F 2 "Resistor_SMD:R_0805_2012Metric_Pad1.20x1.40mm_HandSolder" V 1480 3350 50  0001 C CNN
+F 3 "~" H 1550 3350 50  0001 C CNN
+	1    1550 3350
+	1    0    0    1
+$EndComp
+Wire Wire Line
+	1550 3500 1550 3600
+Wire Wire Line
+	1550 3600 1325 3600
+Text Label 1325 2700 0    39   ~ 0
+5V
+Text Label 1325 3600 0    39   ~ 0
+5V
+Text Notes 1100 3900 0    50   ~ 0
+NS=Not Shorted\nNG=Not Grounded
 $EndSCHEMATC

Commit message: TSI Post-Nadovich
Parts:
- added R126: 1.8K, Resistor_SMD:R_0805_2012Metric_Pad1.20x1.40mm_HandSolder, symbol TSI_Rev.5-rescue:R-Device
- added R127: 3.3K, Resistor_SMD:R_0805_2012Metric_Pad1.20x1.40mm_HandSolder, symbol TSI_Rev.5-rescue:R-Device
- R111, R112: value 10k -> 4.7K
Connections:
- net 3.3V: now also R111.1, R112.1
- net 5V: no longer R111.1, R112.1
- net GLV_RTN: now also R127.2
- net Throttle_PL: now also R126.1; no longer U44.2 (AN16/ETXD0/PMD6/RE6)
- net APPS1_ISO_NG: no longer names the net of U44.63 (TRD3/SQID3/ERXCLK/EREFCLK/RPE3/PMD3/RE3)
- net APPS1_ISO_NS: no longer names the net of U44.62 (TRD2/SQID2/ERXDV/ECRSDV/AECRSDV/PMD2/RE2)
- net APPS2_ISO_NG: no longer names the net of U44.64 (AN18/ERXERR/PMD4/RE4)
- net APPS2_ISO_NS: no longer names the net of U44.1 (AN17/ETXEN/RPE5/PMD5/RE5)
- net APPS_WIN1: no longer names the net of U44.58 (TRD0/SQID0/ERXD1/PMD0/RE0)
- net APPS_WIN2: no longer names the net of U44.61 (TRD1/SQID1/ERXD0/PMD1/RE1)
- net Drive_BTN renamed Drive_BTN_LOGIC
- net Flowrate renamed Flowrate_LOGIC
- net Throttle_LOGIC: no longer names the net of U44.43 (AERXD0/ETXD2/RPD9/SDA1/PMCS2/PMA15/RD9)
- new net Throttle_PL_LOGIC: R126.2, R127.1, U44.2 (AN16/ETXD0/PMD6/RE6)
- no-connect marks 15 -> 22
Other:
- note added: "5V-3.3V Voltage Divider"
Changed lines of the file:
@@
 $Descr A4 11693 8268
 encoding utf-8
-Sheet 6 7
+Sheet 7 7
 Title ""
 Date ""
@@
 SDA
 Wire Wire Line
-	6200 3500 6700 3500
-Text Label 6700 3500 2    39   ~ 0
-Throttle_LOGIC
-Wire Wire Line
 	6200 3600 6700 3600
 Wire Wire Line
@@
 	2550 3500 2050 3500
 Text Label 2050 3500 0    39   ~ 0
-Throttle_PL
-Wire Wire Line
-	2550 3600 2050 3600
-Text Label 2050 3600 0    39   ~ 0
-APPS2_ISO_NS
+Throttle_PL_LOGIC
 Text Label 2050 3100 0    39   ~ 0
 SCL
 Wire Wire Line
-	6200 4700 6700 4700
-Wire Wire Line
-	6200 4800 6700 4800
-Wire Wire Line
-	6200 4900 6700 4900
-Wire Wire Line
-	6200 5000 6700 5000
-Wire Wire Line
-	2550 3700 2050 3700
-Text Label 6700 4700 2    39   ~ 0
-APPS_WIN1
-Text Label 6700 4800 2    39   ~ 0
-APPS_WIN2
-Text Label 6700 4900 2    39   ~ 0
-APPS1_ISO_NS
-Text Label 6700 5000 2    39   ~ 0
-APPS1_ISO_NG
-Text Label 2050 3700 0    39   ~ 0
-APPS2_ISO_NG
-Wire Wire Line
 	2550 4500 2050 4500
 Text Label 2050 4500 0    39   ~ 0
-Flowrate
+Flowrate_LOGIC
 Wire Wire Line
 	2550 5100 2050 5100
@@
 Safety_Loop
 Text Label 2050 5400 0    39   ~ 0
-Drive_BTN
+Drive_BTN_LOGIC
 Wire Wire Line
 	6200 3800 6700 3800
@@
 NoConn ~ 6200 4500
 NoConn ~ 6200 4600
-Text HLabel 8725 725  0    39   Input ~ 0
-APPS_WIN1
-Text HLabel 8725 800  0    39   Input ~ 0
-APPS_WIN2
-Text HLabel 8725 875  0    39   Input ~ 0
-APPS1_ISO_NS
-Text HLabel 8725 950  0    39   Input ~ 0
-APPS1_ISO_NG
-Text HLabel 8725 1025 0    39   Input ~ 0
-APPS2_ISO_NS
-Text HLabel 8725 1100 0    39   Input ~ 0
-APPS2_ISO_NG
-Text HLabel 8725 1175 0    39   Input ~ 0
-Throttle_PL
-Text HLabel 8725 1250 0    39   Input ~ 0
+Text HLabel 8725 1200 0    39   Input ~ 0
 Brake_Pressed_uC
-Text HLabel 8725 1325 0    39   Input ~ 0
-Drive_BTN
-Text HLabel 8725 1400 0    39   Input ~ 0
+Text HLabel 8725 1275 0    39   Input ~ 0
 Safety_Loop
-Text HLabel 8725 1475 0    39   Input ~ 0
+Text HLabel 8725 1350 0    39   Input ~ 0
 PC_Ready
-Text HLabel 8725 1550 0    39   Input ~ 0
-Flowrate
-Text HLabel 8725 1625 0    39   Input ~ 0
+Text HLabel 8725 1425 0    39   Input ~ 0
+Flowrate_LOGIC
+Text HLabel 8725 1500 0    39   Input ~ 0
 ~MCLR
-Text HLabel 8725 1700 0    39   Input ~ 0
+Text HLabel 8725 1575 0    39   Input ~ 0
 PGEC
-Text HLabel 8725 1775 0    39   Input ~ 0
+Text HLabel 8725 1650 0    39   Input ~ 0
 PGED
-Text HLabel 8725 1850 0    39   Input ~ 0
+Text HLabel 8725 1725 0    39   Input ~ 0
 UART_RXD
-Text HLabel 8725 1925 0    39   Input ~ 0
+Text HLabel 8725 1800 0    39   Input ~ 0
 3.3V
-Text HLabel 8725 2000 0    39   Input ~ 0
+Text HLabel 8725 1875 0    39   Input ~ 0
 GLV_RTN
 Text HLabel 8725 2450 0    39   Output ~ 0
@@
 Throttle_EN
 Text HLabel 8725 2750 0    39   Output ~ 0
-Throttle_LOGIC
+Test_Pin0
 Text HLabel 8725 2825 0    39   Output ~ 0
-Test_Pin0
+Test_Pin1
 Text HLabel 8725 2900 0    39   Output ~ 0
-Test_Pin1
+Test_Pin2
 Text HLabel 8725 2975 0    39   Output ~ 0
-Test_Pin2
+Test_Pin3
 Text HLabel 8725 3050 0    39   Output ~ 0
-Test_Pin3
+Test_Pin4
 Text HLabel 8725 3125 0    39   Output ~ 0
-Test_Pin4
+Test_Pin5
 Text HLabel 8725 3200 0    39   Output ~ 0
-Test_Pin5
+Test_Pin6
 Text HLabel 8725 3275 0    39   Output ~ 0
-Test_Pin6
+Test_Pin7
 Text HLabel 8725 3350 0    39   Output ~ 0
-Test_Pin7
+Test_Pin8
 Text HLabel 8725 3425 0    39   Output ~ 0
-Test_Pin8
+Test_Pin9
 Text HLabel 8725 3500 0    39   Output ~ 0
-Test_Pin9
-Text HLabel 8725 3650 0    39   Output ~ 0
 UART_TXD
 NoConn ~ 2550 2200
@@
 Text Label 2050 2800 0    39   ~ 0
 Test_Pin5
-Text HLabel 8725 3725 0    39   Output ~ 0
-SDA
-Text HLabel 8725 3800 0    39   Output ~ 0
-SCL
-Text HLabel 8725 2075 0    39   Input ~ 0
+Text HLabel 8725 1950 0    39   Input ~ 0
 CAN_H
-Text HLabel 8725 2150 0    39   Input ~ 0
+Text HLabel 8725 2025 0    39   Input ~ 0
 CAN_L
 $Comp
@@
 Text Label 8125 5050 0    39   ~ 0
 5V
-Text HLabel 8725 2225 0    39   Input ~ 0
+Text HLabel 8725 2100 0    39   Input ~ 0
 5V
 $Comp
@@
 P 1550 2950
 F 0 "R111" H 1620 2996 50  0000 L CNN
-F 1 "10k" H 1620 2905 50  0000 L CNN
+F 1 "4.7K" H 1620 2905 50  0000 L CNN
 F 2 "Resistor_SMD:R_0805_2012Metric_Pad1.20x1.40mm_HandSolder" V 1480 2950 50  0001 C CNN
 F 3 "~" H 1550 2950 50  0001 C CNN
@@
 P 1550 3350
 F 0 "R112" H 1481 3304 50  0000 R CNN
-F 1 "10k" H 1481 3395 50  0000 R CNN
+F 1 "4.7K" H 1481 3395 50  0000 R CNN
 F 2 "Resistor_SMD:R_0805_2012Metric_Pad1.20x1.40mm_HandSolder" V 1480 3350 50  0001 C CNN
 F 3 "~" H 1550 3350 50  0001 C CNN
@@
 	1550 3600 1325 3600
 Text Label 1325 2700 0    39   ~ 0
-5V
+3.3V
 Text Label 1325 3600 0    39   ~ 0
-5V
+3.3V
 Text Notes 1100 3900 0    50   ~ 0
 NS=Not Shorted\nNG=Not Grounded
+Text HLabel 8725 2175 0    39   Input ~ 0
+Drive_BTN_LOGIC
+Text HLabel 8725 1050 0    39   Input ~ 0
+SDA
+Text HLabel 8725 1125 0    39   Input ~ 0
+SCL
+NoConn ~ 6200 4700
+NoConn ~ 6200 4800
+NoConn ~ 6200 4900
+NoConn ~ 6200 5000
+NoConn ~ 2550 3600
+NoConn ~ 2550 3700
+Text HLabel 8725 2250 0    39   Input ~ 0
+Throttle_PL
+NoConn ~ 6200 3500
+Text Label 1125 5900 0    50   ~ 0
+Throttle_PL
+$Comp
+L TSI_Rev.5-rescue:R-Device R?
+U 1 1 63434879
+P 1125 6200
+AR Path="/63434879" Ref="R?"  Part="1"
+AR Path="/5FE1DE7D/63434879" Ref="R?"  Part="1"
+AR Path="/623B2FCE/63434879" Ref="R126"  Part="1"
+F 0 "R126" H 1195 6246 50  0000 L CNN
+F 1 "1.8K" V 1125 6125 50  0000 L CNN
+F 2 "Resistor_SMD:R_0805_2012Metric_Pad1.20x1.40mm_HandSolder" V 1055 6200 50  0001 C CNN
+F 3 "~" H 1125 6200 50  0001 C CNN
+	1    1125 6200
+	1    0    0    -1
+$EndComp
+$Comp
+L TSI_Rev.5-rescue:R-Device R?
+U 1 1 6343487F
+P 1125 6600
+AR Path="/6343487F" Ref="R?"  Part="1"
+AR Path="/5FE1DE7D/6343487F" Ref="R?"  Part="1"
+AR Path="/623B2FCE/6343487F" Ref="R127"  Part="1"
+F 0 "R127" H 1195 6646 50  0000 L CNN
+F 1 "3.3K" V 1125 6500 50  0000 L CNN
+F 2 "Resistor_SMD:R_0805_2012Metric_Pad1.20x1.40mm_HandSolder" V 1055 6600 50  0001 C CNN
+F 3 "~" H 1125 6600 50  0001 C CNN
+	1    1125 6600
+	1    0    0    -1
+$EndComp
+Wire Wire Line
+	1125 6450 1125 6400
+Connection ~ 1125 6400
+Wire Wire Line
+	1125 6400 1125 6350
+Wire Wire Line
+	1125 6400 1725 6400
+Wire Wire Line
+	1125 6750 1125 6900
+Text Label 1125 6900 0    50   ~ 0
+GLV_RTN
+Wire Wire Line
+	1125 5900 1125 6050
+Text Notes 1575 6700 0    50   ~ 0
+5V-3.3V Voltage Divider
+Text Label 1725 6400 0    50   ~ 0
+Throttle_PL_LOGIC
 $EndSCHEMATC

Commit message: TSI REV7 Final Schematic before Layout
Connections:
- net RTDS_CTRL: now also U44.58 (TRD0/SQID0/ERXD1/PMD0/RE0); no longer U44.50 (ETXERR/AETXEN/RPD2/SDA3/RD2)
Changed lines of the file:
@@
 	6200 3900 6700 3900
 Wire Wire Line
-	6200 4000 6700 4000
+	6200 4700 6700 4700
 Text Label 6700 3800 2    39   ~ 0
 Cooling_CTRL
 Text Label 6700 3900 2    39   ~ 0
 D_LED_CTRL
-Text Label 6700 4000 2    39   ~ 0
+Text Label 6700 4700 2    39   ~ 0
 RTDS_CTRL
 Wire Wire Line
@@
 Text HLabel 8725 1125 0    39   Input ~ 0
 SCL
-NoConn ~ 6200 4700
+NoConn ~ 6200 4000
 NoConn ~ 6200 4800
 NoConn ~ 6200 4900

Commit message: Finished PCB for REV7
Changed lines of the file:
@@
 Text Label 2050 3400 0    39   ~ 0
 Test_Pin0
-Text Label 2050 3200 0    39   ~ 0
+Text Label 1150 3200 0    39   ~ 0
 SDA
 Wire Wire Line
@@
 Text Label 2050 3500 0    39   ~ 0
 Throttle_PL_LOGIC
-Text Label 2050 3100 0    39   ~ 0
+Text Label 1150 3100 0    39   ~ 0
 SCL
 Wire Wire Line
@@
 Text Label 1725 6400 0    50   ~ 0
 Throttle_PL_LOGIC
+Wire Wire Line
+	1550 3200 1150 3200
+Connection ~ 1550 3200
+Wire Wire Line
+	1550 3100 1150 3100
+Connection ~ 1550 3100
 $EndSCHEMATC
